File: Schematic (KiCAD)/pcm_dac.kicad_sch (KiCad schematic)
At the start: 31 parts, among them J60 NAND_2, K100 NAND_2, K101 Reg 2 DFF-Reset N, K102 INVERT, K103 AOI_2, K104 TriBuf 8, K104(a) INVERT, K105 TriBuf 8, K105(a) INVERT, K106 NAND_2, K107 INVERT, K108 INVERT, K109,K110,K111 D-FF Set, K112 NOR_2, K113 INVERT, K114 INVERT, K96 INVERT, K99 BIGBUF

Commit message: - Started work on the pulse channels.  - Solved at least 2 of the red traces in the SVG.  - Finally realized that "Unknown 4to1" cells are actually just ordinary And-Or-Invert "AOI22" cells.
Connections:
- net at K107. (X): now also K106. (X); no longer K109,K110,K111. (/Q)
- net at K96. (X): now also J60. (X); no longer L121. (X)
- net at L134. (/Q3): now also L133. (X); no longer L135. (X)
- net at K105(a). (X): now also K105. (Y8); no longer L131. (X)
- net at L139. (/Q3): now also L138. (X); no longer L140. (X)
- net at K113. (X): now also K112. (X); no longer K114. (X)
- new net: K108. (X), K109,K110,K111. (/Q), L134. (/Q3), L139. (/Q3)
- new net: K107. (X), K109,K110,K111. (/Q)
- new net: K109,K110,K111. (/Q), K112. (X)
- new net: K96. (X), L121. (X)
- new net: K104(a). (X), K104. (Y8)
- new net: K100. (X), K106. (X)
- new net: K100. (X), K99. (X)
- new net: L134. (/Q3), L135. (X)
- new net: K105(a). (X), L131. (X)
- new net: L134. (/Q3), L136. (X)
- new net: L139. (/Q3), L140. (X)
- new net: K104. (Y8), K105. (Y8), L134. (/Q3) (x4)
- new net: L132. (X), L134. (/Q3)
- new net: L137. (X), L139. (/Q3)
- new net: L139. (/Q3), L141. (X)
- new net: K102. (X), K103. (X)
- new net: K103. (X), L121. (X)
- new net: K104. (Y8), K105. (Y8), L139. (/Q3) (x4)
- new net: K113. (X), K114. (X)

Commit message: - Pulse DAC logic is now complete.  - The 4-bit adders are verified correct using Excel.    - This revealed 1 tracing error and also 3 XNOR gates that are actually XOR in this case.  - Now including a PDF version of the schematic.
Connections:
- net at K107. (X): now also K106. (X); no longer K109,K110,K111. (/Q)
- net at K96. (X): now also J60. (X); no longer L121. (X)
- net at L134. (/Q3): now also L133. (X); no longer L135. (X)
- net at K105(a). (X): now also K105. (Y8); no longer L131. (X)
- net at L139. (/Q3): now also L138. (X); no longer L140. (X)
- net at K113. (X): now also K112. (X); no longer K114. (X)
- new net: K108. (X), K109,K110,K111. (/Q), L134. (/Q3), L139. (/Q3)
- new net: K107. (X), K109,K110,K111. (/Q)
- new net: K109,K110,K111. (/Q), K112. (X)
- new net: K96. (X), L121. (X)
- new net: K104(a). (X), K104. (Y8)
- new net: K100. (X), K106. (X)
- new net: K100. (X), K99. (X)
- new net: L134. (/Q3), L135. (X)
- new net: K105(a). (X), L131. (X)
- new net: L134. (/Q3), L136. (X)
- new net: L139. (/Q3), L140. (X)
- new net: K104. (Y8), K105. (Y8), L134. (/Q3) (x4)
- new net: L132. (X), L134. (/Q3)
- new net: L137. (X), L139. (/Q3)
- new net: L139. (/Q3), L141. (X)
- new net: K102. (X), K103. (X)
- new net: K103. (X), L121. (X)
- new net: K104. (Y8), K105. (Y8), L139. (/Q3) (x4)
- new net: K113. (X), K114. (X)
