File: Schematic (KiCAD)/pcm_dac.kicad_sch (KiCad schematic)
At the start: 31 parts, among them J60 NAND_2, K100 NAND_2, K101 Reg 2 DFF-Reset N, K102 INVERT, K103 AOI_2, K104 TriBuf 8, K104(a) INVERT, K105 TriBuf 8, K105(a) INVERT, K106 NAND_2, K107 INVERT, K108 INVERT, K109,K110,K111 D-FF Set, K112 NOR_2, K113 INVERT, K114 INVERT, K96 INVERT, K99 BIGBUF

Commit message: Tracing and schematic updates.  - Added timer to schematic.  - Added all items from artifacts sheet to the MMC5A trace.
Connections:
- net +PCM_IRQ_If_Enabled{K114} is gone; now on net /PCM_IRQ_If_Enabled{K113}: K114. (X)
- net at K107. (X): now also K106. (X); no longer K109,K110,K111. (/Q)
- net at K96. (X): now also J60. (X); no longer L121. (X)
- net at L134. (/Q3): now also L133. (X); no longer L135. (X)
- net at K105(a). (X): now also K105. (Y8); no longer L131. (X)
- net at L139. (/Q3): now also L138. (X); no longer L140. (X)
- net /PCM_IRQ_If_Enabled{K113}: now reaches K113. (X), K114. (X)
- new net: K108. (X), K109,K110,K111. (/Q), L134. (/Q3), L139. (/Q3)
- new net: K107. (X), K109,K110,K111. (/Q)
- new net: K109,K110,K111. (/Q), K112. (X)
- new net: K96. (X), L121. (X)
- new net: K104(a). (X), K104. (Y8)
- new net: K100. (X), K106. (X)
- new net: K100. (X), K99. (X)
- new net: L134. (/Q3), L135. (X)
- new net: K105(a). (X), L131. (X)
- new net: L134. (/Q3), L136. (X)
- new net: L139. (/Q3), L140. (X)
- new net: K104. (Y8), K105. (Y8), L134. (/Q3) (x4)
- new net: L132. (X), L134. (/Q3)
- new net: L137. (X), L139. (/Q3)
- new net: L139. (/Q3), L141. (X)
- new net: K102. (X), K103. (X)
- new net: K103. (X), L121. (X)
- new net: K104. (Y8), K105. (Y8), L139. (/Q3) (x4)
- new net: K112. (X), K113. (X)
- new net +PCM_IRQ_Status_Bit{K114}: K114. (X)
Changed lines of the file:
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@@
+	)
+	(junction
+		(at 167.64 167.64)
+		(diameter 0)
+		(color 0 0 0 0)
 	)
 	(junction
@@
 	(wire
 		(pts
+			(xy 167.64 162.56) (xy 168.91 162.56)
+		)
+		(stroke
+			(width 0)
+			(type default)
+		)
+	)
+	(wire
+		(pts
 			(xy 95.25 93.98) (xy 100.33 93.98)
 		)
@@
 		(pts
 			(xy 95.25 83.82) (xy 104.14 83.82)
+		)
+		(stroke
+			(width 0)
+			(type default)
+		)
+	)
+	(wire
+		(pts
+			(xy 167.64 167.64) (xy 167.64 162.56)
 		)
 		(stroke
@@
 		)
 	)
+	(global_label "{slash}PCM_IRQ_If_Enabled{K113}"
+		(shape output)
+		(at 168.91 162.56 0)
+		(fields_autoplaced yes)
+		(effects
+			(font
+				(size 1.27 1.27)
+			)
+			(justify left)
+		)
+		(property "Intersheetrefs" "${INTERSHEET_REFS}"
+			(at 198.7464 162.56 0)
+			(effects
+				(font
+					(size 1.27 1.27)
+				)
+				(justify left)
+				(hide yes)
+			)
+		)
+	)
 	(global_label "{slash}CPU_D4{L126}"
 		(shape input)
@@
 		)
 	)
-	(global_label "+PCM_IRQ_If_Enabled{K114}"
+	(global_label "+PCM_IRQ_Status_Bit{K114}"
 		(shape output)
 		(at 176.53 167.64 0)
@@
 		)
 		(property "Intersheetrefs" "${INTERSHEET_REFS}"
-			(at 206.6083 167.64 0)
+			(at 206.3665 167.64 0)
 			(effects
 				(font

Commit message: - Updated all of the various And-OR-Invert gates to have consistent names.  - Added the schematic for CL3 / SL3 GPIO pins.  There are no surprises revealed by this.  - Finished up the CPU address decoding tracing.  - Added one of the 'artifact' counters from the pulse channels
Parts:
- K103: value AOI_2 -> AOI_22
Connections:
- net at K107. (X): now also K106. (X); no longer K109,K110,K111. (/Q)
- net at K96. (X): now also J60. (X); no longer L121. (X)
- net at L134. (/Q3): now also L133. (X); no longer L135. (X)
- net at K105(a). (X): now also K105. (Y8); no longer L131. (X)
- net at L139. (/Q3): now also L138. (X); no longer L140. (X)
- new net: K108. (X), K109,K110,K111. (/Q), L134. (/Q3), L139. (/Q3)
- new net: K107. (X), K109,K110,K111. (/Q)
- new net: K109,K110,K111. (/Q), K112. (X)
- new net: K96. (X), L121. (X)
- new net: K104(a). (X), K104. (Y8)
- new net: K100. (X), K106. (X)
- new net: K100. (X), K99. (X)
- new net: L134. (/Q3), L135. (X)
- new net: K105(a). (X), L131. (X)
- new net: L134. (/Q3), L136. (X)
- new net: L139. (/Q3), L140. (X)
- new net: K104. (Y8), K105. (Y8), L134. (/Q3) (x4)
- new net: L132. (X), L134. (/Q3)
- new net: L137. (X), L139. (/Q3)
- new net: L139. (/Q3), L141. (X)
- new net: K102. (X), K103. (X)
- new net: K103. (X), L121. (X)
- new net: K104. (Y8), K105. (Y8), L139. (/Q3) (x4)
- new net: K112. (X), K113. (X)
