File: Schematic (KiCAD)/pulse_duty_envelope_volume.kicad_sch (KiCad schematic)
At the start: 70 parts, among them J65 Reg 4 D-Latch N, J68 Counter 4 Reset CL3

Commit message: - Pulse DAC logic is now complete.  - The 4-bit adders are verified correct using Excel.    - This revealed 1 tracing error and also 3 XNOR gates that are actually XOR in this case.  - Now including a PDF version of the schematic.
Connections:
- net at H90. (X): now also G94. (X); no longer H89. (X)
- net at C36. (Y): now also B103. (X)
- net at C35. (X): now also C33. (X); no longer C36. (Y)
- net at B103. (X): now also G20. (X); no longer C36. (Y)
- net at F36. (X): now also G97. (X); no longer F32. (X)
- net at B105. (X): now also C41. (Y); no longer F32. (X)
- net at C39. (X): now also C38. (X); no longer C41. (Y)
- net at E47. (X): now also F10. (X); no longer E48. (X)
- net at F15. (X): now also F16. (X); no longer G20. (X)
- net at G97. (X): now also G99. (X); no longer G98. (X)
- net at C41. (Y): now also C40. (X)
- net at F16. (X): now also F13. (X); no longer F11. (X)
- new net: E45. (X), E46. (X), E47. (X), F12. (X)
- new net: F19. (X), F23. (X)
- new net: B99. (X), C38. (X)
- new net: H89. (X), H90. (X)
- new net: G99. (X), H90. (X), H91. (X), H92. (X)
- new net: C34. (X), C36. (Y)
- new net: C35. (X), C36. (Y)
- new net: H101. (X), H105. (X)
- new net: H100. (X), H104. (X)
- new net: F20. (X), F24. (X)
- new net: F32. (X), F36. (X)
- new net: B105. (X), F32. (X)
- new net: F35. (X), G85. (/Q3)
- new net: F34. (X), G85. (/Q3)
- new net: C39. (X), C41. (Y)
- new net: E47. (X), E48. (X)
- new net: F18. (X), F22. (X)
- new net: C37. (X), C38. (X)
- new net: F15. (X), G20. (X)
- new net: G97. (X), G98. (X)
- new net: H103. (X), H107. (X)
- new net: C32. (X), C33. (X)
- new net: H102. (X), H106. (X)
- new net: F11. (X), F16. (X)
- new net: G93. (X), G97. (X)
- new net: F21. (X), F26. (X)
- new net: E68. (/Q3), F7.1. (X)
- new net: E68. (/Q3), F8. (X)
- new net: G94. (X), G97. (X)
- new net: F10. (X), F16. (X)
- new net: F12. (X), F16. (X)
- new net: B100. (X), C33. (X)
