File: Schematic (KiCAD)/chr_bank_registers.kicad_sch (KiCad schematic)
At the start: 28 parts

Commit message: - Finished up the CHR Ax bits.
Connections:
- new net: AK6. (+OE), AL6. (+OE)
- new net: AP6. (+OE), AR6. (+OE)
- new net: BF1. (+OE), BG11. (+OE)
- new net: AM6. (+OE), AN6. (+OE)

Commit message: - All cells in the left and center areas have now been added into the schematics.  - Changed naming of the PDF files; I was accidentally writing over furrtek's original with my new PDF.
Parts:
- removed AE10: Reg 2 D-Latch N, symbol MMC5:Reg_2_D-Latch_N
- removed AE11, AE12, AE13, AE14, AF3, AS39: NAND_2, symbol MMC5:NAND_2
- added AE27, AE28, AE29, AE30, AF19, AF20, AF21, AF22: INVERT, symbol MMC5:INVERT
- added AK1, AK2, AK3, AK4, AK5, AL1, AL2, AL3, AL4, AL5, AM1, AM2, AM3, AM4, AM5, AN1, AN2, AN3, AN4, AN5, AP1, AP2, AP3, AP4, AP5, AR1, AR2, AR3, AR4, AR5, BG1, BG10, BG2, BG3, BG4, BG5, BG6, BG7, BG8, BG9: BUFFER, symbol MMC5:BUFFER
Connections:
- net VSplit_CHR_Bank_$5202.0{AE26} is gone; now on net /CPU_D7{AE21}: AE26. (Q7)
- net VSplit_CHR_Bank_$5202.1{AE26} is gone; now on net /CPU_D7{AE21}: AE26. (Q7)
- net VSplit_CHR_Bank_$5202.2{AE26} is gone; now on net /CPU_D7{AE21}: AE26. (Q7)
- net VSplit_CHR_Bank_$5202.3{AE26} is gone; now on net /CPU_D7{AE21}: AE26. (Q7)
- net VSplit_CHR_Bank_$5202.4{AE26} is gone; now on net /CPU_D7{AE21}: AE26. (Q7)
- net VSplit_CHR_Bank_$5202.5{AE26} is gone; now on net /CPU_D7{AE21}: AE26. (Q7)
- net VSplit_CHR_Bank_$5202.6{AE26} is gone; now on net /CPU_D7{AE21}: AE26. (Q7)
- net VSplit_CHR_Bank_$5202.7{AE26} is gone; now on net /CPU_D7{AE21}: AE26. (Q7)
- net /CPU_D0{AE14} is gone; now on net /Reset_Detect{AE3}: AE17. (/Q1)
- net /CPU_D1{AE13} is gone; now on net /Reset_Detect{AE3}: AE17. (/Q1)
- net /CHR_REG_WRITE_D0: now also AK5. (X), AM5. (X), AP5. (X), BG1. (X); no longer AK6. (+OE), AL6. (+OE), AM6. (+OE), AN6. (+OE), AP6. (+OE), AR6. (+OE), BF1. (+OE), BG11. (+OE)
- net /CHR_REG_WRITE_D1: now also AK4. (X), AM4. (X), AP4. (X), BG2. (X); no longer AK6. (+OE), AL6. (+OE), AM6. (+OE), AN6. (+OE), AP6. (+OE), AR6. (+OE), BF1. (+OE), BG11. (+OE)
- net /CHR_REG_WRITE_D2: now also AK3. (X), AM3. (X), AP3. (X), BG3. (X); no longer AK6. (+OE), AL6. (+OE), AM6. (+OE), AN6. (+OE), AP6. (+OE), AR6. (+OE), BF1. (+OE), BG11. (+OE)
- net /CHR_REG_WRITE_D3: now also AK2. (X), AM2. (X), AP2. (X), BG4. (X); no longer AK6. (+OE), AL6. (+OE), AM6. (+OE), AN6. (+OE), AP6. (+OE), AR6. (+OE), BF1. (+OE), BG11. (+OE)
- net /CHR_REG_WRITE_D4: now also AK1. (X), AM1. (X), AP1. (X), BG5. (X); no longer AK6. (+OE), AL6. (+OE), AM6. (+OE), AN6. (+OE), AP6. (+OE), AR6. (+OE), BF1. (+OE), BG11. (+OE)
- net /CHR_REG_WRITE_D5: now also AL5. (X), AN5. (X), AR5. (X), BG6. (X); no longer AK6. (+OE), AL6. (+OE), AM6. (+OE), AN6. (+OE), AP6. (+OE), AR6. (+OE), BF1. (+OE), BG11. (+OE)
- net /CHR_REG_WRITE_D6: now also AL4. (X), AN4. (X), AR4. (X), BG7. (X); no longer AK6. (+OE), AL6. (+OE), AM6. (+OE), AN6. (+OE), AP6. (+OE), AR6. (+OE), BF1. (+OE), BG11. (+OE)
- net /CHR_REG_WRITE_D7: now also AL3. (X), AN3. (X), AR3. (X), BG8. (X); no longer AK6. (+OE), AL6. (+OE), AM6. (+OE), AN6. (+OE), AP6. (+OE), AR6. (+OE), BF1. (+OE), BG11. (+OE)
- net /CHR_REG_WRITE_D8: now also AL2. (X), AN2. (X), AR2. (X), BG9. (X); no longer AK6. (+OE), AL6. (+OE), AM6. (+OE), AN6. (+OE), AP6. (+OE), AR6. (+OE), BF1. (+OE), BG11. (+OE)
- net /CHR_REG_WRITE_D9: now also AL1. (X), AN1. (X), AR1. (X), BG10. (X); no longer AK6. (+OE), AL6. (+OE), AM6. (+OE), AN6. (+OE), AP6. (+OE), AR6. (+OE), BF1. (+OE), BG11. (+OE)
- new net: AK6. (+OE), AL6. (+OE)
- new net: AE26. (Q7), AE30. (X)
- new net: AE26. (Q7), AE27. (X)
- new net: AE26. (Q7), AF21. (X)
- new net: AE26. (Q7), AF19. (X)
- new net: AE26. (Q7), AE29. (X)
- new net: AE26. (Q7), AF22. (X)
- new net: AE26. (Q7), AE28. (X)
- new net: AE26. (Q7), AF20. (X)
- new net: AP6. (+OE), AR6. (+OE)
- new net: BF1. (+OE), BG11. (+OE)
- new net: AM6. (+OE), AN6. (+OE)
- new net +VSplit_CHR_Bank_$5202.0{AE27}: AE27. (X)
- new net +VSplit_CHR_Bank_$5202.1{AE28}: AE28. (X)
- new net +VSplit_CHR_Bank_$5202.2{AE29}: AE29. (X)
- new net +VSplit_CHR_Bank_$5202.3{AF19}: AF19. (X)
- new net +VSplit_CHR_Bank_$5202.4{AF20}: AF20. (X)
- new net +VSplit_CHR_Bank_$5202.5{AF21}: AF21. (X)
- new net +VSplit_CHR_Bank_$5202.6{AF22}: AF22. (X)
- new net +VSplit_CHR_Bank_$5202.7{AE30}: AE30. (X)
- new net 8x16_Mode_Related{AS25}: AL6. (+OE), AN6. (+OE), AR6. (+OE), BG11. (+OE)
- new net /CHR_REG_WRITE_D0{AK5}: AK5. (X), AK6. (+OE), AL6. (+OE)
- new net /CHR_REG_WRITE_D0{AM5}: AM5. (X), AM6. (+OE), AN6. (+OE)
- new net /CHR_REG_WRITE_D0{AP5}: AP5. (X), AP6. (+OE), AR6. (+OE)
- new net /CHR_REG_WRITE_D0{BG1}: BF1. (+OE), BG1. (X), BG11. (+OE)
- new net /CHR_REG_WRITE_D1{AK4}: AK4. (X), AK6. (+OE), AL6. (+OE)
- new net /CHR_REG_WRITE_D1{AM4}: AM4. (X), AM6. (+OE), AN6. (+OE)
- new net /CHR_REG_WRITE_D1{AP4}: AP4. (X), AP6. (+OE), AR6. (+OE)
- new net /CHR_REG_WRITE_D1{BG2}: BF1. (+OE), BG11. (+OE), BG2. (X)
- new net /CHR_REG_WRITE_D2{AK3}: AK3. (X), AK6. (+OE), AL6. (+OE)
- new net /CHR_REG_WRITE_D2{AM3}: AM3. (X), AM6. (+OE), AN6. (+OE)
- new net /CHR_REG_WRITE_D2{AP3}: AP3. (X), AP6. (+OE), AR6. (+OE)
- new net /CHR_REG_WRITE_D2{BG3}: BF1. (+OE), BG11. (+OE), BG3. (X)
- new net /CHR_REG_WRITE_D3{AK2}: AK2. (X), AK6. (+OE), AL6. (+OE)
- new net /CHR_REG_WRITE_D3{AM2}: AM2. (X), AM6. (+OE), AN6. (+OE)
- new net /CHR_REG_WRITE_D3{AP2}: AP2. (X), AP6. (+OE), AR6. (+OE)
- new net /CHR_REG_WRITE_D3{BG4}: BF1. (+OE), BG11. (+OE), BG4. (X)
- new net /CHR_REG_WRITE_D4{AK1}: AK1. (X), AK6. (+OE), AL6. (+OE)
- new net /CHR_REG_WRITE_D4{AM1}: AM1. (X), AM6. (+OE), AN6. (+OE)
- new net /CHR_REG_WRITE_D4{AP1}: AP1. (X), AP6. (+OE), AR6. (+OE)
- new net /CHR_REG_WRITE_D4{BG5}: BF1. (+OE), BG11. (+OE), BG5. (X)
- new net /CHR_REG_WRITE_D5{AL5}: AK6. (+OE), AL5. (X), AL6. (+OE)
- new net /CHR_REG_WRITE_D5{AN5}: AM6. (+OE), AN5. (X), AN6. (+OE)
- new net /CHR_REG_WRITE_D5{AR5}: AP6. (+OE), AR5. (X), AR6. (+OE)
- new net /CHR_REG_WRITE_D5{BG6}: BF1. (+OE), BG11. (+OE), BG6. (X)
- new net /CHR_REG_WRITE_D6{AL4}: AK6. (+OE), AL4. (X), AL6. (+OE)
- new net /CHR_REG_WRITE_D6{AN4}: AM6. (+OE), AN4. (X), AN6. (+OE)
- new net /CHR_REG_WRITE_D6{AR4}: AP6. (+OE), AR4. (X), AR6. (+OE)
- new net /CHR_REG_WRITE_D6{BG7}: BF1. (+OE), BG11. (+OE), BG7. (X)
- new net /CHR_REG_WRITE_D7{AL3}: AK6. (+OE), AL3. (X), AL6. (+OE)
- new net /CHR_REG_WRITE_D7{AN3}: AM6. (+OE), AN3. (X), AN6. (+OE)
- new net /CHR_REG_WRITE_D7{AR3}: AP6. (+OE), AR3. (X), AR6. (+OE)
- new net /CHR_REG_WRITE_D7{BG8}: BF1. (+OE), BG11. (+OE), BG8. (X)
- new net /CHR_REG_WRITE_D8{AL2}: AK6. (+OE), AL2. (X), AL6. (+OE)
- new net /CHR_REG_WRITE_D8{AN2}: AM6. (+OE), AN2. (X), AN6. (+OE)
- new net /CHR_REG_WRITE_D8{AR2}: AP6. (+OE), AR2. (X), AR6. (+OE)
- new net /CHR_REG_WRITE_D8{BG9}: BF1. (+OE), BG11. (+OE), BG9. (X)
- new net /CHR_REG_WRITE_D9{AL1}: AK6. (+OE), AL1. (X), AL6. (+OE)
- new net /CHR_REG_WRITE_D9{AN1}: AM6. (+OE), AN1. (X), AN6. (+OE)
- new net /CHR_REG_WRITE_D9{AR1}: AP6. (+OE), AR1. (X), AR6. (+OE)
- new net /CHR_REG_WRITE_D9{BG10}: BF1. (+OE), BG10. (X), BG11. (+OE)
- new net /CPU_D0{AE16}: AE17. (/Q1)
- new net /CPU_D1{AE15}: AE17. (/Q1)
Other:
- note added: "CHR Reg Write Buffering"
- note added: "Note: Reg 10 might have +OE input and /OE output, not sure."
- note removed: "$5101 Register CHR Mode"
- note removed: "Why did AF3 and AS39 not use simpler logic?"
- moved on the sheet: AE17, AE26, AF4, AF5, AF6, AF7, AG1, AG2, AG3, AH1, AH2, AJ1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
