File: Schematic (KiCAD)/chr_bank_registers.kicad_sch (KiCad schematic)
At the start: 69 parts

Commit message: - Updated all of the various And-OR-Invert gates to have consistent names.  - Added the schematic for CL3 / SL3 GPIO pins.  There are no surprises revealed by this.  - Finished up the CPU address decoding tracing.  - Added one of the 'artifact' counters from the pulse channels
Connections:
- new net: AK6. (+OE), AL6. (+OE)
- new net: AE26. (Q7), AE30. (X)
- new net: AE26. (Q7), AE27. (X)
- new net: AE26. (Q7), AF21. (X)
- new net: AE26. (Q7), AF19. (X)
- new net: AE26. (Q7), AE29. (X)
- new net: AE26. (Q7), AF22. (X)
- new net: AE26. (Q7), AE28. (X)
- new net: AE26. (Q7), AF20. (X)
- new net: AP6. (+OE), AR6. (+OE)
- new net: BF1. (+OE), BG11. (+OE)
- new net: AM6. (+OE), AN6. (+OE)
Changed lines of the file:
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@@
 	)
 	(symbol
-		(lib_name "BUFFER_31")
+		(lib_name "BUFFER_33")
 		(lib_id "MMC5:BUFFER")
 		(at 379.73 152.4 0)
@@
 	)
 	(symbol
-		(lib_name "BUFFER_33")
+		(lib_name "BUFFER_29")
 		(lib_id "MMC5:BUFFER")
 		(at 379.73 144.78 0)
@@
 	)
 	(symbol
+		(lib_name "Reg_10_D-Latch_OE_2")
 		(lib_id "MMC5:Reg_10_D-Latch_OE")
 		(at 46.99 219.71 0)
@@
 	)
 	(symbol
-		(lib_name "INVERT_12")
+		(lib_name "INVERT_8")
 		(lib_id "MMC5:INVERT")
 		(at 306.07 55.88 0)
@@
 	)
 	(symbol
+		(lib_name "TriBuf_1N_1")
 		(lib_id "MMC5:TriBuf_1N")
 		(at 59.69 34.29 0)
@@
 	)
 	(symbol
-		(lib_name "BUFFER_24")
+		(lib_name "BUFFER_21")
 		(lib_id "MMC5:BUFFER")
 		(at 379.73 95.25 0)
@@
 	)
 	(symbol
-		(lib_name "BUFFER_15")
+		(lib_name "BUFFER_14")
 		(lib_id "MMC5:BUFFER")
 		(at 379.73 45.72 0)
@@
 	)
 	(symbol
-		(lib_name "BUFFER_5")
+		(lib_name "BUFFER_6")
 		(lib_id "MMC5:BUFFER")
 		(at 379.73 123.19 0)
@@
 	)
 	(symbol
-		(lib_name "BUFFER_29")
+		(lib_name "BUFFER_30")
 		(lib_id "MMC5:BUFFER")
 		(at 379.73 132.08 0)
@@
 	)
 	(symbol
-		(lib_name "BUFFER_13")
+		(lib_name "BUFFER_15")
 		(lib_id "MMC5:BUFFER")
 		(at 379.73 53.34 0)
@@
 	)
 	(symbol
-		(lib_name "TriBuf_1N_1")
 		(lib_id "MMC5:TriBuf_1N")
 		(at 59.69 26.67 0)
@@
 	)
 	(symbol
-		(lib_name "BUFFER_25")
+		(lib_name "BUFFER_26")
 		(lib_id "MMC5:BUFFER")
 		(at 379.73 119.38 0)
@@
 	)
 	(symbol
-		(lib_name "BUFFER_32")
+		(lib_name "BUFFER_31")
 		(lib_id "MMC5:BUFFER")
 		(at 379.73 148.59 0)
@@
 	)
 	(symbol
+		(lib_name "Reg_10_D-Latch_N_2")
 		(lib_id "MMC5:Reg_10_D-Latch_N")
 		(at 46.99 106.68 0)
@@
 	)
 	(symbol
-		(lib_name "BUFFER_3")
+		(lib_name "BUFFER_4")
 		(lib_id "MMC5:BUFFER")
 		(at 379.73 90.17 0)
@@
 	)
 	(symbol
-		(lib_name "BUFFER_38")
+		(lib_name "BUFFER_39")
 		(lib_id "MMC5:BUFFER")
 		(at 379.73 181.61 0)
@@
 	)
 	(symbol
-		(lib_name "Reg_10_D-Latch_OE_5")
+		(lib_name "Reg_10_D-Latch_OE_6")
 		(lib_id "MMC5:Reg_10_D-Latch_OE")
 		(at 208.28 176.53 0)
@@
 	)
 	(symbol
-		(lib_name "Reg_10_D-Latch_OE_4")
+		(lib_name "Reg_10_D-Latch_OE_3")
 		(lib_id "MMC5:Reg_10_D-Latch_OE")
 		(at 208.28 219.71 0)
@@
 	)
 	(symbol
-		(lib_name "BUFFER_18")
+		(lib_name "BUFFER_17")
 		(lib_id "MMC5:BUFFER")
 		(at 379.73 62.23 0)
@@
 	)
 	(symbol
-		(lib_name "Reg_10_D-Latch_OE_6")
+		(lib_name "Reg_10_D-Latch_OE_1")
 		(lib_id "MMC5:Reg_10_D-Latch_OE")
 		(at 289.56 219.71 0)
@@
 	)
 	(symbol
-		(lib_name "BUFFER_20")
+		(lib_name "BUFFER_19")
 		(lib_id "MMC5:BUFFER")
 		(at 379.73 82.55 0)
@@
 	)
 	(symbol
-		(lib_name "Reg_10_D-Latch_OE_2")
 		(lib_id "MMC5:Reg_10_D-Latch_OE")
 		(at 127 219.71 0)
@@
 	)
 	(symbol
-		(lib_name "BUFFER_30")
+		(lib_name "BUFFER_32")
 		(lib_id "MMC5:BUFFER")
 		(at 379.73 128.27 0)
@@
 	)
 	(symbol
-		(lib_name "BUFFER_34")
+		(lib_name "BUFFER_36")
 		(lib_id "MMC5:BUFFER")
 		(at 379.73 168.91 0)
@@
 	)
 	(symbol
-		(lib_name "Reg_10_D-Latch_OE_1")
+		(lib_name "Reg_10_D-Latch_OE_4")
 		(lib_id "MMC5:Reg_10_D-Latch_OE")
 		(at 46.99 176.53 0)
@@
 	)
 	(symbol
-		(lib_name "BUFFER_35")
+		(lib_name "BUFFER_37")
 		(lib_id "MMC5:BUFFER")
 		(at 379.73 165.1 0)
@@
 	)
 	(symbol
-		(lib_name "Reg_10_D-Latch_OE_7")
+		(lib_name "Reg_10_D-Latch_OE_5")
 		(lib_id "MMC5:Reg_10_D-Latch_OE")
 		(at 289.56 176.53 0)
@@
 	)
 	(symbol
-		(lib_name "BUFFER_37")
+		(lib_name "BUFFER_34")
 		(lib_id "MMC5:BUFFER")
 		(at 379.73 185.42 0)
@@
 	)
 	(symbol
-		(lib_name "BUFFER_6")
+		(lib_name "BUFFER_2")
 		(lib_id "MMC5:BUFFER")
 		(at 379.73 139.7 0)
@@
 	)
 	(symbol
-		(lib_name "BUFFER_23")
+		(lib_name "BUFFER_25")
 		(lib_id "MMC5:BUFFER")
 		(at 379.73 99.06 0)
@@
 	)
 	(symbol
-		(lib_name "BUFFER_22")
+		(lib_name "BUFFER_23")
 		(lib_id "MMC5:BUFFER")
 		(at 379.73 102.87 0)
@@
 	)
 	(symbol
-		(lib_name "INVERT_5")
+		(lib_name "INVERT_2")
 		(lib_id "MMC5:INVERT")
 		(at 299.72 29.21 0)
@@
 	)
 	(symbol
-		(lib_name "TriBuf_9N_1")
 		(lib_id "MMC5:TriBuf_9N")
 		(at 214.63 41.91 0)
@@
 	)
 	(symbol
-		(lib_name "BUFFER_27")
+		(lib_name "BUFFER_22")
 		(lib_id "MMC5:BUFFER")
 		(at 379.73 111.76 0)
@@
 	)
 	(symbol
-		(lib_name "INVERT_10")
+		(lib_name "INVERT_5")
 		(lib_id "MMC5:INVERT")
 		(at 306.07 48.26 0)
@@
 	)
 	(symbol
-		(lib_name "BUFFER_17")
+		(lib_name "BUFFER_16")
 		(lib_id "MMC5:BUFFER")
 		(at 379.73 66.04 0)
@@
 	)
 	(symbol
-		(lib_name "INVERT_8")
+		(lib_name "INVERT_4")
 		(lib_id "MMC5:INVERT")
 		(at 306.07 40.64 0)
@@
 	)
 	(symbol
-		(lib_name "INVERT_7")
+		(lib_name "INVERT_3")
 		(lib_id "MMC5:INVERT")
 		(at 299.72 36.83 0)
@@
 	)
 	(symbol
-		(lib_name "INVERT_9")
+		(lib_name "INVERT_7")
 		(lib_id "MMC5:INVERT")
 		(at 299.72 52.07 0)
@@
 	)
 	(symbol
-		(lib_name "INVERT_6")
+		(lib_name "INVERT_1")
 		(lib_id "MMC5:INVERT")
 		(at 306.07 33.02 0)
@@
 	)
 	(symbol
-		(lib_name "Reg_10_D-Latch_N_2")
+		(lib_name "Reg_10_D-Latch_N_3")
 		(lib_id "MMC5:Reg_10_D-Latch_N")
 		(at 289.56 106.68 0)
@@
 	)
 	(symbol
-		(lib_name "BUFFER_26")
+		(lib_name "BUFFER_27")
 		(lib_id "MMC5:BUFFER")
 		(at 379.73 115.57 0)
@@
 	)
 	(symbol
+		(lib_name "BUFFER_3")
 		(lib_id "MMC5:BUFFER")
 		(at 379.73 40.64 0)
@@
 	)
 	(symbol
-		(lib_name "BUFFER_39")
+		(lib_name "BUFFER_35")
 		(lib_id "MMC5:BUFFER")
 		(at 379.73 177.8 0)
@@
 	)
 	(symbol
-		(lib_name "BUFFER_1")
 		(lib_id "MMC5:BUFFER")
 		(at 379.73 57.15 0)
@@
 	)
 	(symbol
+		(lib_name "TriBuf_9N_1")
 		(lib_id "MMC5:TriBuf_9N")
 		(at 162.56 41.91 0)
@@
 	)
 	(symbol
-		(lib_name "BUFFER_21")
+		(lib_name "BUFFER_20")
 		(lib_id "MMC5:BUFFER")
 		(at 379.73 78.74 0)
@@
 	)
 	(symbol
-		(lib_name "BUFFER_12")
+		(lib_name "BUFFER_13")
 		(lib_id "MMC5:BUFFER")
 		(at 379.73 29.21 0)
@@
 	)
 	(symbol
-		(lib_name "BUFFER_14")
+		(lib_name "BUFFER_18")
 		(lib_id "MMC5:BUFFER")
 		(at 379.73 49.53 0)
@@
 	)
 	(symbol
-		(lib_name "BUFFER_2")
+		(lib_name "BUFFER_5")
 		(lib_id "MMC5:BUFFER")
 		(at 379.73 73.66 0)
@@
 	)
 	(symbol
-		(lib_name "BUFFER_36")
+		(lib_name "BUFFER_38")
 		(lib_id "MMC5:BUFFER")
 		(at 379.73 161.29 0)
@@
 	)
 	(symbol
-		(lib_name "BUFFER_16")
+		(lib_name "BUFFER_12")
 		(lib_id "MMC5:BUFFER")
 		(at 379.73 69.85 0)
@@
 	)
 	(symbol
-		(lib_name "BUFFER_19")
+		(lib_name "BUFFER_24")
 		(lib_id "MMC5:BUFFER")
 		(at 379.73 86.36 0)
@@
 	)
 	(symbol
-		(lib_name "BUFFER_4")
+		(lib_name "BUFFER_1")
 		(lib_id "MMC5:BUFFER")
 		(at 379.73 106.68 0)
@@
 	)
 	(symbol
-		(lib_name "Reg_10_D-Latch_OE_3")
+		(lib_name "Reg_10_D-Latch_OE_7")
 		(lib_id "MMC5:Reg_10_D-Latch_OE")
 		(at 127 176.53 0)
@@
 	)
 	(symbol
-		(lib_name "Reg_10_D-Latch_N_3")
 		(lib_id "MMC5:Reg_10_D-Latch_N")
 		(at 208.28 106.68 0)
@@
 	)
 	(symbol
-		(lib_name "INVERT_11")
+		(lib_name "INVERT_6")
 		(lib_id "MMC5:INVERT")
 		(at 299.72 44.45 0)
