File: Schematic (KiCAD)/artifacts.kicad_sch (KiCad schematic)
At the start: 61 parts, among them J14 NAND_2, J15 NAND_3, J3 BIGBUF, J56 INVERT, J57 INVERT, J58 INVERT, J61 INVERT, J62 INVERT, J63 NOR_3, J64 NOR_3, J67 INVERT, J69 INVERT, K23 INVERT, K24 NAND_2, K61 NAND_3, K62 INVERT

Commit message: - Lots of additional comments and signal name improvements.  - "Don't know what this is yet but it is important" section of the pulse channels:    - I worked out the logic and it is a 4-bit binary up-counter with preload, made from gates and D-latches instead of T-flip-flops.    - It is extremely similar to the envelope counter, but takes twice the die space and much more traces.    - None of its outputs go anywhere else, so I believe that it has no actual function.    - It seems to be a previous attempt at making the envelope counter and it got disconnected and left in.    - Each pulse channel has its own copy and I moved both of them to the "Artifacts" sheet.    - The wasted space amounts to about half of one of the large columns on the left side of the die.  - A couple of "OAI2" cells that noted "unclear order": I determined the correct order of the inputs based on several others which were known.  - Deduced the purpose of the 2 separate methods of scanline detection:    - The one looking for 3 consecutive reads finds the start of a scanline.    - The one counting PPU /RD to find PPU cycle 336, finds the end of the scanline.    - I moved these beside each other on the same sheet for clarity.  - A66.5 Changed from Nand to Nor in order to make sense.  - Basic test mode:    - Pin 92: Active low, enables test mode.    - Pin 29: In test mode, it gives external control of "Scanline Start Detection", which is normally done with the familiar 3 matching PPU reads.  When not in test mode, the pin has no function.    - Pin 30: In test mode, it gives external control of "Scanline End Detection", which is normally done by counting PPU /RD to find PPU cycle 336.  It also gives control of "Pulse Length Clock" when in test mode.  When not in test mode, the pin has no function.    - Pin 98/SL3: In test mode, it gives external control of "Pulse Timer Clock".  Whether or not in test mode, this pin low makes the MMC5 pretend $5104 had not yet been written since reset, probably as a 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
Parts:
- added G29, G30, G32, G34, G36, G38, G40, G42, G44, G45, G47, G50, G52, G55, G57, G59, G61, G63, G65, G66, G67, G68, G82, H38, H39, H41, H43, H45, H47, H49, H51, H52, H54, H56, H58, H60, H63, H65, H67, H68, H71, H73, H75, H76, H78: INVERT, symbol MMC5:INVERT
- added G31, G33, G35, G37, G39, H40, H42, H44, H46, H48: NAND_2, symbol MMC5:NAND_2
- added G41, H50: NOR_2, symbol MMC5:NOR_2
- added G43, G48, G54, H64, H69, H77: NAND_4, symbol MMC5:NAND_4
- added G46, H72: NAND_5, symbol MMC5:NAND_5
- added G49, G53, G56, G60, G62, H53, H55, H61, H62, H70: NAND_3, symbol MMC5:NAND_3
- added G51, G58, G64, H57, H66, H74: NOR_3, symbol MMC5:NOR_3
- added G69, H80: Reg 4 D-Latch N, symbol MMC5:Reg_4_D-Latch_N
Connections:
- net Pulse_Timer_Clock{A61} is gone; now on net Pulse_Timer_Clock_Fast{A61}: B91. (X), B95. (X)
- net at L61. (X): now also J15. (X); no longer L60. (X)
- net at J15. (X): now also L19. (X); no longer L61. (X)
- net at J62. (X): now also J63. (X); no longer J61. (X)
- net at G96. (X): now also F25. (X); no longer G86. (X)
- net at B36. (X): now also B35. (X); no longer B37. (X)
- net at C4. (X): now also C3. (X); no longer C5. (X)
- net at B32. (X): now also B31. (X); no longer B33. (X)
- net at B27. (X): now also B28. (X); no longer B26. (X)
- net at L20. (X): now also J58. (X); no longer K23. (X)
- net at J58. (X): now also J57. (X); no longer L20. (X)
- net at B93. (X): now also B69. (X); no longer A76. (X)
- net at H59. (X): now also J69. (X); no longer H81. (X)
- net at J56. (X): now also K62. (X); no longer J57. (X)
- net at K62. (X): now also K61. (X); no longer J56. (X)
- net at A20. (X): now also A21. (X); no longer A19. (X)
- net at B96. (X): now also B95. (X); no longer B97. (X)
- net at E32. (X): now also E31. (X); no longer E33. (X)
- net at J63. (X): now also J64. (X); no longer J62. (X)
- net at C29. (X): now also B69. (X); no longer C30. (X)
- net Pulse_Timer_Clock_Fast{A61}: now reaches B91. (X)
- net at B28. (X): now also B29. (X); no longer B27. (X)
- net at E66. (X): now also D43. (X); no longer E54. (X)
- net at K24. (X): now also K23. (X); no longer J14. (X)
- net at B35. (X): now also B34. (X); no longer B36. (X)
- new net: H44. (X), H45. (X)
- new net: H45. (X), H66. (X)
- new net: L60. (X), L61. (X)
- new net: G47. (X), G51. (X)
- new net: G46. (X), G47. (X)
- new net: H38. (X), H48. (X), H53. (X), H55. (X), H61. (X), H62. (X), H64. (X), H69. (X), H70. (X), H72. (X)
- new net: H70. (X), H71. (X)
- new net: H69. (X), H70. (X)
- new net: H38. (X), H39. (X), H40. (X), H42. (X), H44. (X), H46. (X)
- new net: G62. (X), G63. (X)
- new net: G63. (X), G64. (X)
- new net: H71. (X), H74. (X)
- new net: H73. (X), H74. (X)
- new net: H47. (X), H74. (X)
- new net: H74. (X), H75. (X)
- new net: G34. (X), G58. (X)
- new net: G58. (X), G59. (X)
- new net: G55. (X), G58. (X)
- new net: G57. (X), G58. (X)
- new net: H57. (X), H58. (X)
- new net: H58. (X), H80. (/Q3)
- new net: J61. (X), J62. (X)
- new net: G86. (X), G96. (X)
- new net: F25. (X), G96. (X)
- new net: H43. (X), H57. (X)
- new net: H42. (X), H43. (X)
- new net: B36. (X), B37. (X)
- new net: C4. (X), C5. (X)
- new net: G33. (X), G34. (X)
- new net: G30. (X), G39. (X), G46. (X), G48. (X), G49. (X), G53. (X), G54. (X), G56. (X), G60. (X), G62. (X)
- new net: G39. (X), G40. (X)
- new net: H61. (X), H62. (X)
- new net: H62. (X), H63. (X)
- new net: H48. (X), H49. (X)
- new net: B32. (X), B33. (X)
- new net: B26. (X), B27. (X)
- new net: H41. (X), H50. (X)
- new net: H49. (X), H50. (X)
- new net: H50. (X), H51. (X)
- new net: K23. (X), L20. (X)
- new net: A76. (X), B93. (X)
- new net: G37. (X), G38. (X)
- new net: G38. (X), G41. (X)
- new net: G49. (X), G50. (X)
- new net: G48. (X), G49. (X)
- new net: H59. (X), H81. (X)
- new net: J56. (X), J57. (X)
- new net: A19. (X), A20. (X)
- new net: A20. (X), A21. (X)
- new net: B96. (X), B97. (X)
- new net: G50. (X), G51. (X)
- new net: G51. (X), G52. (X)
- new net: G32. (X), G51. (X)
- new net: G53. (X), G56. (X)
- new net: H54. (X), H57. (X)
- new net: H56. (X), H57. (X)
- new net: H46. (X), H47. (X)
- new net: E32. (X), E33. (X)
- new net: G29. (X), G30. (X), G31. (X), G33. (X), G35. (X), G37. (X)
- new net: G35. (X), G36. (X)
- new net: G36. (X), G64. (X)
- new net: H55. (X), H56. (X)
- new net: E31. (X), F6.1. (X)
- new net: H40. (X), H41. (X)
- new net: H75. (X), H80. (/Q3)
- new net: H51. (X), H80. (/Q3)
- new net: H67. (X), H80. (/Q3)
- new net: J63. (X), J64. (X)
- new net: J3. (X), L19. (X)
- new net: C29. (X), C30. (X)
- new net: G43. (X), G44. (X)
- new net: C2. (X), C3. (X)
- new net: G60. (X), G61. (X)
- new net: H53. (X), H54. (X)
- new net: E54. (X), E66. (X)
- new net: D43. (X), E66. (X)
- new net: J14. (X), K24. (X)
- new net: B28. (X), B29. (X)
- new net: H72. (X), H73. (X)
- new net: G56. (X), G57. (X)
- new net: G61. (X), G64. (X)
- new net: G64. (X), G65. (X)
- new net: G31. (X), G32. (X)
- new net: G52. (X), G69. (/Q3)
- new net: H77. (X), H78. (X)
- new net: D44. (X), J69. (X)
- new net: H65. (X), H66. (X)
- new net: H66. (X), H67. (X)
- new net: H63. (X), H66. (X)
- new net: G59. (X), G69. (/Q3)
- new net: G42. (X), G69. (/Q3)
- new net: G65. (X), G69. (/Q3)
- new net: H64. (X), H65. (X)
- new net: G54. (X), G55. (X)
- new net: G41. (X), G42. (X)
- new net: G40. (X), G41. (X)
- new net +Pulse_1_Counter.0{H52}: H52. (X), H55. (X), H61. (X), H64. (X), H69. (X), H72. (X), H77. (X)
- new net +Pulse_1_Counter.0{H80}: H80. (/Q3)
- new net +Pulse_1_Counter.1{H60}: H60. (X), H61. (X), H64. (X), H69. (X), H72. (X), H77. (X)
- new net +Pulse_1_Counter.1{H80}: H53. (X), H80. (/Q3)
- new net +Pulse_1_Counter.2{H68}: H68. (X), H69. (X), H72. (X), H77. (X)
- new net +Pulse_1_Counter.2{H80}: H62. (X), H80. (/Q3)
- new net +Pulse_1_Counter.3{H76}: H76. (X), H77. (X)
- new net +Pulse_1_Counter.3{H80}: H70. (X), H80. (/Q3)
- new net +Pulse_1_Counter=$F{H78}: H78. (X)
- new net +Pulse_2_Counter.0{G68}: G43. (X), G46. (X), G48. (X), G53. (X), G54. (X), G60. (X), G68. (X)
- new net +Pulse_2_Counter.0{G69}: G69. (/Q3)
- new net +Pulse_2_Counter.1{G67}: G43. (X), G46. (X), G48. (X), G53. (X), G54. (X), G67. (X)
- new net +Pulse_2_Counter.1{G69}: G69. (/Q3)
- new net +Pulse_2_Counter.1{G82}: G62. (X), G82. (X)
- new net +Pulse_2_Counter.2{G66}: G43. (X), G46. (X), G48. (X), G66. (X)
- new net +Pulse_2_Counter.2{G69}: G56. (X), G69. (/Q3)
- new net +Pulse_2_Counter.3{G45}: G43. (X), G45. (X)
- new net +Pulse_2_Counter.3{G69}: G49. (X), G69. (/Q3)
- new net +Pulse_2_Counter=$F{G44}: G44. (X)
- new net /$5000.0_Vol.0{J65}: H40. (X)
- new net /$5000.1_Vol.1{J65}: H42. (X)
- new net /$5000.2_Vol.2{J65}: H44. (X)
- new net /$5000.3_Vol.3{J65}: H46. (X)
- new net /$5004.0_Vol.0{F37}: G37. (X)
- new net /$5004.1_Vol.1{F37}: G35. (X)
- new net /$5004.2_Vol.2{F37}: G33. (X)
- new net /$5004.3_Vol.3{F37}: G31. (X)
- new net /Pulse_1_Counter.0{H80}: H48. (X), H52. (X), H53. (X), H80. (/Q3)
- new net /Pulse_1_Counter.1{H80}: H55. (X), H60. (X), H80. (/Q3)
- new net /Pulse_1_Counter.2{H80}: H64. (X), H68. (X), H80. (/Q3)
- new net /Pulse_1_Counter.3{H80}: H72. (X), H76. (X), H80. (/Q3)
- new net /Pulse_1_Counter_Preload{H82(a).2}: H39. (X)
- new net /Pulse_2_Counter.0{G69}: G39. (X), G62. (X), G68. (X), G69. (/Q3)
- new net /Pulse_2_Counter.1{G69}: G60. (X), G67. (X), G69. (/Q3), G82. (X)
- new net /Pulse_2_Counter.2{G69}: G54. (X), G66. (X), G69. (/Q3)
- new net /Pulse_2_Counter.3{G69}: G45. (X), G46. (X), G69. (/Q3)
- new net /Pulse_2_Counter_Preload{E34(b).2}: G29. (X)
- new net /Pulse_Timer_Clock_SL3{E51}: G69. (/Q3)
- new net /Pulse_Timer_Clock_SL3{H87}: H80. (/Q3)
Other:
- note added: "241.08Hz"
- note added: "Pulse 1 Unused 4-bit Binary Up-Counter With Preload"
- note added: "Pulse 2 Unused 4-bit Binary Up-Counter With Preload"
- note added: "The only output that goes elsewhere is H78, which gets latched by H82(a), coming directly back here as /Pulse_1_Counter_Preload; all self-contained. It does not appear to provide any other external signals, so I don't think it actually does anything. It seems like an abandoned envelope counter that was left in. It latches the 4-bit pulse volume, then counts up at a rate of 240 Hz. Nothing stops i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"

Commit message: - Improved "Identification of Cells" document for NAND, NOR, and XNOR/XOR gates.  - Gate S16 is a NAND-8 gate; it was shown as NOR-8 before.
Connections:
- net at H45. (X): now also H66. (X); no longer H44. (X)
- net at H66. (X): now also H63. (X); no longer H45. (X)
- net at L61. (X): now also J15. (X); no longer L60. (X)
- net at J15. (X): now also L19. (X); no longer L61. (X)
- net at G47. (X): now also G46. (X); no longer G51. (X)
- net at H71. (X): now also H74. (X); no longer H70. (X)
- net at G63. (X): now also G64. (X); no longer G62. (X)
- net at G64. (X): now also G65. (X); no longer G63. (X)
- net at H74. (X): now also H75. (X); no longer H71. (X)
- net at H73. (X): now also H72. (X); no longer H74. (X)
- net at H47. (X): now also H46. (X); no longer H74. (X)
- net at H75. (X): now also H80. (/Q3); no longer H74. (X)
- net at G58. (X): now also G57. (X); no longer G34. (X)
- net at G59. (X): now also G69. (/Q3); no longer G58. (X)
- net at G55. (X): now also G54. (X); no longer G58. (X)
- net at G57. (X): now also G56. (X); no longer G58. (X)
- net at H58. (X): now also H80. (/Q3); no longer H57. (X)
- net at J62. (X): now also J63. (X); no longer J61. (X)
- net at G96. (X): now also F25. (X); no longer G86. (X)
- net at H43. (X): now also H42. (X); no longer H57. (X)
- net at B36. (X): now also B35. (X); no longer B37. (X)
- net at C4. (X): now also C3. (X); no longer C5. (X)
- net at G40. (X): now also G41. (X); no longer G39. (X)
- net at H49. (X): now also H50. (X); no longer H48. (X)
- net at B32. (X): now also B31. (X); no longer B33. (X)
- net at B27. (X): now also B28. (X); no longer B26. (X)
- net at H50. (X): now also H51. (X); no longer H41. (X)
- net at H51. (X): now also H80. (/Q3); no longer H50. (X)
- net at L20. (X): now also J58. (X); no longer K23. (X)
- net at J58. (X): now also J57. (X); no longer L20. (X)
- net at B93. (X): now also B69. (X); no longer A76. (X)
- net at G38. (X): now also G41. (X); no longer G37. (X)
- net at G50. (X): now also G51. (X); no longer G49. (X)
- net at H59. (X): now also J69. (X); no longer H81. (X)
- net at J56. (X): now also K62. (X); no longer J57. (X)
- net at K62. (X): now also K61. (X); no longer J56. (X)
- net at A20. (X): now also A21. (X); no longer A19. (X)
- net at B96. (X): now also B95. (X); no longer B97. (X)
- net at G51. (X): now also G32. (X); no longer G50. (X)
- net at G52. (X): now also G69. (/Q3); no longer G51. (X)
- net at G32. (X): now also G31. (X); no longer G51. (X)
- net at H57. (X): now also H56. (X); no longer H54. (X)
- net at H56. (X): now also H55. (X); no longer H57. (X)
- net at E32. (X): now also E31. (X); no longer E33. (X)
- net at G36. (X): now also G64. (X); no longer G35. (X)
- net at H67. (X): now also H66. (X); no longer H80. (/Q3)
- net at J63. (X): now also J64. (X); no longer J62. (X)
- net at C29. (X): now also B69. (X); no longer C30. (X)
- net at G61. (X): now also G64. (X); no longer G60. (X)
- net at B28. (X): now also B29. (X); no longer B27. (X)
- net at E66. (X): now also D43. (X); no longer E54. (X)
- net at K24. (X): now also K23. (X); no longer J14. (X)
- net at G65. (X): now also G69. (/Q3); no longer G64. (X)
- net at H65. (X): now also H64. (X); no longer H66. (X)
- net at G42. (X): now also G41. (X); no longer G69. (/Q3)
- net at B35. (X): now also B34. (X); no longer B36. (X)
- new net: H44. (X), H45. (X)
- new net: L60. (X), L61. (X)
- new net: G47. (X), G51. (X)
- new net: H38. (X), H48. (X), H53. (X), H55. (X), H61. (X), H62. (X), H64. (X), H69. (X), H70. (X), H72. (X)
- new net: H70. (X), H71. (X)
- new net: H69. (X), H70. (X)
- new net: H38. (X), H39. (X), H40. (X), H42. (X), H44. (X), H46. (X)
- new net: G62. (X), G63. (X)
- new net: H73. (X), H74. (X)
- new net: H47. (X), H74. (X)
- new net: G34. (X), G58. (X)
- new net: G58. (X), G59. (X)
- new net: G55. (X), G58. (X)
- new net: H57. (X), H58. (X)
- new net: J61. (X), J62. (X)
- new net: G86. (X), G96. (X)
- new net: F25. (X), G96. (X)
- new net: H43. (X), H57. (X)
- new net: B36. (X), B37. (X)
- new net: C4. (X), C5. (X)
- new net: G30. (X), G39. (X), G46. (X), G48. (X), G49. (X), G53. (X), G54. (X), G56. (X), G60. (X), G62. (X)
- new net: G39. (X), G40. (X)
- new net: H61. (X), H62. (X)
- new net: H62. (X), H63. (X)
- new net: H48. (X), H49. (X)
- new net: B32. (X), B33. (X)
- new net: B26. (X), B27. (X)
- new net: H41. (X), H50. (X)
- new net: K23. (X), L20. (X)
- new net: A76. (X), B93. (X)
- new net: G37. (X), G38. (X)
- new net: G49. (X), G50. (X)
- new net: G48. (X), G49. (X)
- new net: H59. (X), H81. (X)
- new net: J56. (X), J57. (X)
- new net: A19. (X), A20. (X)
- new net: A20. (X), A21. (X)
- new net: B96. (X), B97. (X)
- new net: G51. (X), G52. (X)
- new net: G53. (X), G56. (X)
- new net: H54. (X), H57. (X)
- new net: E32. (X), E33. (X)
- new net: G29. (X), G30. (X), G31. (X), G33. (X), G35. (X), G37. (X)
- new net: G35. (X), G36. (X)
- new net: E31. (X), F6.1. (X)
- new net: H67. (X), H80. (/Q3)
- new net: J63. (X), J64. (X)
- new net: J3. (X), L19. (X)
- new net: C29. (X), C30. (X)
- new net: G43. (X), G44. (X)
- new net: C2. (X), C3. (X)
- new net: G60. (X), G61. (X)
- new net: E54. (X), E66. (X)
- new net: D43. (X), E66. (X)
- new net: J14. (X), K24. (X)
- new net: B28. (X), B29. (X)
- new net: H77. (X), H78. (X)
- new net: D44. (X), J69. (X)
- new net: H65. (X), H66. (X)
- new net: G42. (X), G69. (/Q3)

Commit message: - I have fixed all of the problems I was having in the $2006 section, and things are all going places that make sense now.  - I am making good progress on the timer as well.  - I pulled a couple changes back into the letterless SVG and updated the schematic.
Parts:
- removed J15: NAND_3, symbol MMC5:NAND_3
- added J15: NOR_3, symbol MMC5:NOR_3
Connections:
- net at H45. (X): now also H66. (X); no longer H44. (X)
- net at H66. (X): now also H63. (X); no longer H45. (X)
- net at L61. (X): now also J15. (X); no longer L60. (X)
- net at G47. (X): now also G46. (X); no longer G51. (X)
- net at H71. (X): now also H74. (X); no longer H70. (X)
- net at G63. (X): now also G64. (X); no longer G62. (X)
- net at G64. (X): now also G65. (X); no longer G63. (X)
- net at H74. (X): now also H75. (X); no longer H71. (X)
- net at H73. (X): now also H72. (X); no longer H74. (X)
- net at H47. (X): now also H46. (X); no longer H74. (X)
- net at H75. (X): now also H80. (/Q3); no longer H74. (X)
- net at G58. (X): now also G57. (X); no longer G34. (X)
- net at G59. (X): now also G69. (/Q3); no longer G58. (X)
- net at G55. (X): now also G54. (X); no longer G58. (X)
- net at G57. (X): now also G56. (X); no longer G58. (X)
- net at H58. (X): now also H80. (/Q3); no longer H57. (X)
- net at J62. (X): now also J63. (X); no longer J61. (X)
- net at G96. (X): now also F25. (X); no longer G86. (X)
- net at H43. (X): now also H42. (X); no longer H57. (X)
- net at B36. (X): now also B35. (X); no longer B37. (X)
- net at C4. (X): now also C3. (X); no longer C5. (X)
- net at G40. (X): now also G41. (X); no longer G39. (X)
- net at H49. (X): now also H50. (X); no longer H48. (X)
- net at B32. (X): now also B31. (X); no longer B33. (X)
- net at B27. (X): now also B28. (X); no longer B26. (X)
- net at H50. (X): now also H51. (X); no longer H41. (X)
- net at H51. (X): now also H80. (/Q3); no longer H50. (X)
- net at L20. (X): now also J58. (X); no longer K23. (X)
- net at J58. (X): now also J57. (X); no longer L20. (X)
- net at B93. (X): now also B69. (X); no longer A76. (X)
- net at G38. (X): now also G41. (X); no longer G37. (X)
- net at G50. (X): now also G51. (X); no longer G49. (X)
- net at H59. (X): now also J69. (X); no longer H81. (X)
- net at J56. (X): now also K62. (X); no longer J57. (X)
- net at K62. (X): now also K61. (X); no longer J56. (X)
- net at A20. (X): now also A21. (X); no longer A19. (X)
- net at B96. (X): now also B95. (X); no longer B97. (X)
- net at G51. (X): now also G32. (X); no longer G50. (X)
- net at G52. (X): now also G69. (/Q3); no longer G51. (X)
- net at G32. (X): now also G31. (X); no longer G51. (X)
- net at H57. (X): now also H56. (X); no longer H54. (X)
- net at H56. (X): now also H55. (X); no longer H57. (X)
- net at E32. (X): now also E31. (X); no longer E33. (X)
- net at G36. (X): now also G64. (X); no longer G35. (X)
- net at H67. (X): now also H66. (X); no longer H80. (/Q3)
- net at J63. (X): now also J64. (X); no longer J62. (X)
- net at C29. (X): now also B69. (X); no longer C30. (X)
- net at G61. (X): now also G64. (X); no longer G60. (X)
- net at B28. (X): now also B29. (X); no longer B27. (X)
- net at E66. (X): now also D43. (X); no longer E54. (X)
- net at K24. (X): now also K23. (X); no longer J14. (X)
- net at G65. (X): now also G69. (/Q3); no longer G64. (X)
- net at H65. (X): now also H64. (X); no longer H66. (X)
- net at G42. (X): now also G41. (X); no longer G69. (/Q3)
- net at B35. (X): now also B34. (X); no longer B36. (X)
- new net: H44. (X), H45. (X)
- new net: L60. (X), L61. (X)
- new net: G47. (X), G51. (X)
- new net: H38. (X), H48. (X), H53. (X), H55. (X), H61. (X), H62. (X), H64. (X), H69. (X), H70. (X), H72. (X)
- new net: H70. (X), H71. (X)
- new net: H69. (X), H70. (X)
- new net: H38. (X), H39. (X), H40. (X), H42. (X), H44. (X), H46. (X)
- new net: G62. (X), G63. (X)
- new net: H73. (X), H74. (X)
- new net: H47. (X), H74. (X)
- new net: G34. (X), G58. (X)
- new net: G58. (X), G59. (X)
- new net: G55. (X), G58. (X)
- new net: H57. (X), H58. (X)
- new net: J61. (X), J62. (X)
- new net: G86. (X), G96. (X)
- new net: F25. (X), G96. (X)
- new net: H43. (X), H57. (X)
- new net: B36. (X), B37. (X)
- new net: C4. (X), C5. (X)
- new net: G30. (X), G39. (X), G46. (X), G48. (X), G49. (X), G53. (X), G54. (X), G56. (X), G60. (X), G62. (X)
- new net: G39. (X), G40. (X)
- new net: H61. (X), H62. (X)
- new net: H62. (X), H63. (X)
- new net: H48. (X), H49. (X)
- new net: B32. (X), B33. (X)
- new net: B26. (X), B27. (X)
- new net: H41. (X), H50. (X)
- new net: K23. (X), L20. (X)
- new net: A76. (X), B93. (X)
- new net: G37. (X), G38. (X)
- new net: G49. (X), G50. (X)
- new net: G48. (X), G49. (X)
- new net: H59. (X), H81. (X)
- new net: J56. (X), J57. (X)
- new net: A19. (X), A20. (X)
- new net: A20. (X), A21. (X)
- new net: B96. (X), B97. (X)
- new net: G51. (X), G52. (X)
- new net: G53. (X), G56. (X)
- new net: H54. (X), H57. (X)
- new net: E32. (X), E33. (X)
- new net: G29. (X), G30. (X), G31. (X), G33. (X), G35. (X), G37. (X)
- new net: J15. (X), L19. (X)
- new net: G35. (X), G36. (X)
- new net: E31. (X), F6.1. (X)
- new net: H67. (X), H80. (/Q3)
- new net: J63. (X), J64. (X)
- new net: C29. (X), C30. (X)
- new net: G43. (X), G44. (X)
- new net: C2. (X), C3. (X)
- new net: G60. (X), G61. (X)
- new net: E54. (X), E66. (X)
- new net: D43. (X), E66. (X)
- new net: J14. (X), K24. (X)
- new net: B28. (X), B29. (X)
- new net: H77. (X), H78. (X)
- new net: D44. (X), J69. (X)
- new net: H65. (X), H66. (X)
- new net: G42. (X), G69. (/Q3)
Changed lines of the file:
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@@
 	)
 	(symbol
+		(lib_name "NOR_3_21")
+		(lib_id "MMC5:NOR_3")
+		(at 67.31 193.04 0)
+		(unit 1)
+		(exclude_from_sim no)
+		(in_bom yes)
+		(on_board yes)
+		(dnp no)
+		(fields_autoplaced yes)
+		(property "Reference" "J15"
+			(at 67.31 188.214 0)
+			(do_not_autoplace yes)
+			(effects
+				(font
+					(size 1.27 1.27)
+				)
+				(justify top)
+			)
+		)
+		(property "Value" "NOR_3"
+			(at 67.31 193.04 0)
+			(do_not_autoplace yes)
+			(effects
+				(font
+					(size 0.635 0.635)
+				)
+			)
+		)
+		(property "Footprint" ""
+			(at 67.31 193.04 0)
+			(effects
+				(font
+					(size 1.27 1.27)
+				)
+				(hide yes)
+			)
+		)
+		(property "Datasheet" ""
+			(at 67.31 193.04 0)
+			(effects
+				(font
+					(size 1.27 1.27)
+				)
+				(hide yes)
+			)
+		)
+		(property "Description" ""
+			(at 67.31 193.04 0)
+			(effects
+				(font
+					(size 1.27 1.27)
+				)
+				(hide yes)
+			)
+		)
+		(pin ""
+		)
+		(pin ""
+		)
+		(pin ""
+		)
+		(pin ""
+		)
+		(instances
+			(project "MMC5"
+				(path "/46093bf6-f83e-4237-9ece-7350a682aff0/f2339e17-4f55-43f8-b207-f65123403db0"
+					(reference "J15")
+					(unit 1)
+				)
+			)
+		)
+	)
+	(symbol
 		(lib_name "INVERT_63")
 		(lib_id "MMC5:INVERT")
@@
 					(unit 1)
 				)
-			)
-		)
-	)
-	(symbol
-		(lib_name "NAND_3_11")
-		(lib_id "MMC5:NAND_3")
-		(at 67.31 193.04 0)
-		(unit 1)
-		(exclude_from_sim no)
-		(in_bom yes)
-		(on_board yes)
-		(dnp no)
-		(property "Reference" "J15"
-			(at 67.31 188.214 0)
-			(do_not_autoplace yes)
-			(effects
-				(font
-					(size 1.27 1.27)
-				)
-				(justify top)
-			)
-		)
-		(property "Value" "NAND_3"
-			(at 67.31 193.04 0)
-			(do_not_autoplace yes)
-			(effects
-				(font
-					(size 0.635 0.635)
-				)
-			)
-		)
-		(property "Footprint" ""
-			(at 67.31 193.04 0)
-			(effects
-				(font
-					(size 1.27 1.27)
-				)
-				(hide yes)
-			)
-		)
-		(property "Datasheet" ""
-			(at 67.31 193.04 0)
-			(effects
-				(font
-					(size 1.27 1.27)
-				)
-				(hide yes)
-			)
-		)
-		(property "Description" ""
-			(at 67.31 193.04 0)
-			(effects
-				(font
-					(size 1.27 1.27)
-				)
-				(hide yes)
-			)
-		)
-		(pin ""
-		)
-		(pin ""
-		)
-		(pin ""
-		)
-		(pin ""
-		)
-		(instances
-			(project "MMC5"
-				(path "/46093bf6-f83e-4237-9ece-7350a682aff0/f2339e17-4f55-43f8-b207-f65123403db0"
-					(reference "J15")
-					(unit 1)
-				)
