File: Schematic (KiCAD)/chr_address_bus_15_to_19.kicad_sch (KiCad schematic)
At the start: 85 parts

Commit message: - Lots of additional comments and signal name improvements.  - "Don't know what this is yet but it is important" section of the pulse channels:    - I worked out the logic and it is a 4-bit binary up-counter with preload, made from gates and D-latches instead of T-flip-flops.    - It is extremely similar to the envelope counter, but takes twice the die space and much more traces.    - None of its outputs go anywhere else, so I believe that it has no actual function.    - It seems to be a previous attempt at making the envelope counter and it got disconnected and left in.    - Each pulse channel has its own copy and I moved both of them to the "Artifacts" sheet.    - The wasted space amounts to about half of one of the large columns on the left side of the die.  - A couple of "OAI2" cells that noted "unclear order": I determined the correct order of the inputs based on several others which were known.  - Deduced the purpose of the 2 separate methods of scanline detection:    - The one looking for 3 consecutive reads finds the start of a scanline.    - The one counting PPU /RD to find PPU cycle 336, finds the end of the scanline.    - I moved these beside each other on the same sheet for clarity.  - A66.5 Changed from Nand to Nor in order to make sense.  - Basic test mode:    - Pin 92: Active low, enables test mode.    - Pin 29: In test mode, it gives external control of "Scanline Start Detection", which is normally done with the familiar 3 matching PPU reads.  When not in test mode, the pin has no function.    - Pin 30: In test mode, it gives external control of "Scanline End Detection", which is normally done by counting PPU /RD to find PPU cycle 336.  It also gives control of "Pulse Length Clock" when in test mode.  When not in test mode, the pin has no function.    - Pin 98/SL3: In test mode, it gives external control of "Pulse Timer Clock".  Whether or not in test mode, this pin low makes the MMC5 pretend $5104 had not yet been written since reset, probably as a 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
Connections:
- net at BD9. (X): now also BD12. (X); no longer BD17. (X)
- net at BD8. (X): now also BD5. (X); no longer BD9. (X)
- net at BD4. (X): now also BD2. (X); no longer BD9. (X)
- net at BD12. (X): now also BD13. (X); no longer BD9. (X)
- net at BD14. (X): now also BD15. (X); no longer BD13. (X)
- net at BC14. (X): now also BC15. (X); no longer BC16. (X)
- net at BC13. (X): now also BC12. (X); no longer BC14. (X)
- net at BC12. (X): now also BC11. (X); no longer BC13. (X)
- net at BB4. (X): now also BB1. (X); no longer BB3. (X)
- net at BC4. (X): now also BC3. (X); no longer BC2. (X)
- net at BA8. (X): now also BA9. (X); no longer BA6. (X)
- net at BE14. (X): now also BE15. (X); no longer BE16. (X)
- net at BE13. (X): now also BE12. (X); no longer BE14. (X)
- net at BE8. (X): now also BE6. (X); no longer BE5. (X)
- net at BC9. (X): now also BC12. (X); no longer BC17. (X)
- net at BE4. (X): now also BE1. (X); no longer BE2. (X)
- net at BE9. (X): now also BE12. (X); no longer BE4. (X)
- net at BB8. (X): now also BB5. (X); no longer BB7. (X)
- net at BA12. (X): now also BA10. (X); no longer BA9. (X)
- net at BA13. (X): now also BA14. (X); no longer BA12. (X)
- net at BA9. (X): now also BA17. (X); no longer BA8. (X)
- net at BB12. (X): now also BB10. (X); no longer BB9. (X)
- net at BB13. (X): now also BB14. (X); no longer BB12. (X)
- net at BB9. (X): now also BB4. (X); no longer BB8. (X)
- net at BA4. (X): now also BA2. (X); no longer BA3. (X)
- net at BC8. (X): now also BC7. (X); no longer BC5. (X)
- new net: BD17. (X), BD9. (X)
- new net: BD8. (X), BD9. (X)
- new net: BD4. (X), BD9. (X)
- new net: BD13. (X), BD14. (X)
- new net: BD14. (X), BD16. (X)
- new net: BC14. (X), BC16. (X)
- new net: BC13. (X), BC14. (X)
- new net: BB3. (X), BB4. (X)
- new net: BC2. (X), BC4. (X)
- new net: BD3. (X), BD4. (X)
- new net: BA6. (X), BA8. (X)
- new net: BD7. (X), BD8. (X)
- new net: BA5. (X), BA8. (X)
- new net: BE14. (X), BE16. (X)
- new net: BE13. (X), BE14. (X)
- new net: BE5. (X), BE8. (X)
- new net: BC17. (X), BC9. (X)
- new net: BE2. (X), BE4. (X)
- new net: BE4. (X), BE9. (X)
- new net: BE3. (X), BE4. (X)
- new net: BB7. (X), BB8. (X)
- new net: BB2. (X), BB4. (X)
- new net: BA12. (X), BA9. (X)
- new net: BA11. (X), BA12. (X)
- new net: BA12. (X), BA13. (X)
- new net: BD1. (X), BD4. (X)
- new net: BD11. (X), BD12. (X)
- new net: BA7. (X), BA8. (X)
- new net: BB12. (X), BB9. (X)
- new net: BB12. (X), BB13. (X)
- new net: BB11. (X), BB12. (X)
- new net: BC10. (X), BC12. (X)
- new net: BB8. (X), BB9. (X)
- new net: BB17. (X), BB9. (X)
- new net: BB14. (X), BB15. (X)
- new net: BB14. (X), BB16. (X)
- new net: BB6. (X), BB8. (X)
- new net: BD10. (X), BD12. (X)
- new net: BD6. (X), BD8. (X)
- new net: BA14. (X), BA15. (X)
- new net: BA14. (X), BA16. (X)
- new net: BA3. (X), BA4. (X)
- new net: BC5. (X), BC8. (X)
- new net: BC8. (X), BC9. (X)
- new net: BC4. (X), BC9. (X)
- new net: BA4. (X), BA9. (X)
- new net: BA1. (X), BA4. (X)
- new net: BC6. (X), BC8. (X)
- new net: BE11. (X), BE12. (X)
- new net: BE8. (X), BE9. (X)
- new net: BE7. (X), BE8. (X)
- new net: BC1. (X), BC4. (X)
- new net: BE10. (X), BE12. (X)
- new net: BE17. (X), BE9. (X)

Commit message: - Improved "Identification of Cells" document for NAND, NOR, and XNOR/XOR gates.  - Gate S16 is a NAND-8 gate; it was shown as NOR-8 before.
Connections:
- net at BD9. (X): now also BD12. (X); no longer BD17. (X)
- net at BD8. (X): now also BD5. (X); no longer BD9. (X)
- net at BD4. (X): now also BD2. (X); no longer BD9. (X)
- net at BD12. (X): now also BD13. (X); no longer BD9. (X)
- net at BD14. (X): now also BD15. (X); no longer BD13. (X)
- net at BC14. (X): now also BC15. (X); no longer BC16. (X)
- net at BC13. (X): now also BC12. (X); no longer BC14. (X)
- net at BC12. (X): now also BC11. (X); no longer BC13. (X)
- net at BB4. (X): now also BB1. (X); no longer BB3. (X)
- net at BC4. (X): now also BC3. (X); no longer BC2. (X)
- net at BA8. (X): now also BA9. (X); no longer BA6. (X)
- net at BE14. (X): now also BE15. (X); no longer BE16. (X)
- net at BE13. (X): now also BE12. (X); no longer BE14. (X)
- net at BE8. (X): now also BE6. (X); no longer BE5. (X)
- net at BC9. (X): now also BC12. (X); no longer BC17. (X)
- net at BE4. (X): now also BE1. (X); no longer BE2. (X)
- net at BE9. (X): now also BE12. (X); no longer BE4. (X)
- net at BB8. (X): now also BB5. (X); no longer BB7. (X)
- net at BA12. (X): now also BA10. (X); no longer BA9. (X)
- net at BA13. (X): now also BA14. (X); no longer BA12. (X)
- net at BA9. (X): now also BA17. (X); no longer BA8. (X)
- net at BB12. (X): now also BB10. (X); no longer BB9. (X)
- net at BB13. (X): now also BB14. (X); no longer BB12. (X)
- net at BB9. (X): now also BB4. (X); no longer BB8. (X)
- net at BA4. (X): now also BA2. (X); no longer BA3. (X)
- net at BC8. (X): now also BC7. (X); no longer BC5. (X)
- new net: BD17. (X), BD9. (X)
- new net: BD8. (X), BD9. (X)
- new net: BD4. (X), BD9. (X)
- new net: BD13. (X), BD14. (X)
- new net: BD14. (X), BD16. (X)
- new net: BC14. (X), BC16. (X)
- new net: BC13. (X), BC14. (X)
- new net: BB3. (X), BB4. (X)
- new net: BC2. (X), BC4. (X)
- new net: BD3. (X), BD4. (X)
- new net: BA6. (X), BA8. (X)
- new net: BD7. (X), BD8. (X)
- new net: BA5. (X), BA8. (X)
- new net: BE14. (X), BE16. (X)
- new net: BE13. (X), BE14. (X)
- new net: BE5. (X), BE8. (X)
- new net: BC17. (X), BC9. (X)
- new net: BE2. (X), BE4. (X)
- new net: BE4. (X), BE9. (X)
- new net: BE3. (X), BE4. (X)
- new net: BB7. (X), BB8. (X)
- new net: BB2. (X), BB4. (X)
- new net: BA12. (X), BA9. (X)
- new net: BA11. (X), BA12. (X)
- new net: BA12. (X), BA13. (X)
- new net: BD1. (X), BD4. (X)
- new net: BD11. (X), BD12. (X)
- new net: BA7. (X), BA8. (X)
- new net: BB12. (X), BB9. (X)
- new net: BB12. (X), BB13. (X)
- new net: BB11. (X), BB12. (X)
- new net: BC10. (X), BC12. (X)
- new net: BB8. (X), BB9. (X)
- new net: BB17. (X), BB9. (X)
- new net: BB14. (X), BB15. (X)
- new net: BB14. (X), BB16. (X)
- new net: BB6. (X), BB8. (X)
- new net: BD10. (X), BD12. (X)
- new net: BD6. (X), BD8. (X)
- new net: BA14. (X), BA15. (X)
- new net: BA14. (X), BA16. (X)
- new net: BA3. (X), BA4. (X)
- new net: BC5. (X), BC8. (X)
- new net: BC8. (X), BC9. (X)
- new net: BC4. (X), BC9. (X)
- new net: BA4. (X), BA9. (X)
- new net: BA1. (X), BA4. (X)
- new net: BC6. (X), BC8. (X)
- new net: BE11. (X), BE12. (X)
- new net: BE8. (X), BE9. (X)
- new net: BE7. (X), BE8. (X)
- new net: BC1. (X), BC4. (X)
- new net: BE10. (X), BE12. (X)
- new net: BE17. (X), BE9. (X)

Commit message: - I have fixed all of the problems I was having in the $2006 section, and things are all going places that make sense now.  - I am making good progress on the timer as well.  - I pulled a couple changes back into the letterless SVG and updated the schematic.
Connections:
- net at BD9. (X): now also BD12. (X); no longer BD17. (X)
- net at BD8. (X): now also BD5. (X); no longer BD9. (X)
- net at BD4. (X): now also BD2. (X); no longer BD9. (X)
- net at BD12. (X): now also BD13. (X); no longer BD9. (X)
- net at BD14. (X): now also BD15. (X); no longer BD13. (X)
- net at BC14. (X): now also BC15. (X); no longer BC16. (X)
- net at BC13. (X): now also BC12. (X); no longer BC14. (X)
- net at BC12. (X): now also BC11. (X); no longer BC13. (X)
- net at BB4. (X): now also BB1. (X); no longer BB3. (X)
- net at BC4. (X): now also BC3. (X); no longer BC2. (X)
- net at BA8. (X): now also BA9. (X); no longer BA6. (X)
- net at BE14. (X): now also BE15. (X); no longer BE16. (X)
- net at BE13. (X): now also BE12. (X); no longer BE14. (X)
- net at BE8. (X): now also BE6. (X); no longer BE5. (X)
- net at BC9. (X): now also BC12. (X); no longer BC17. (X)
- net at BE4. (X): now also BE1. (X); no longer BE2. (X)
- net at BE9. (X): now also BE12. (X); no longer BE4. (X)
- net at BB8. (X): now also BB5. (X); no longer BB7. (X)
- net at BA12. (X): now also BA10. (X); no longer BA9. (X)
- net at BA13. (X): now also BA14. (X); no longer BA12. (X)
- net at BA9. (X): now also BA17. (X); no longer BA8. (X)
- net at BB12. (X): now also BB10. (X); no longer BB9. (X)
- net at BB13. (X): now also BB14. (X); no longer BB12. (X)
- net at BB9. (X): now also BB4. (X); no longer BB8. (X)
- net at BA4. (X): now also BA2. (X); no longer BA3. (X)
- net at BC8. (X): now also BC7. (X); no longer BC5. (X)
- new net: BD17. (X), BD9. (X)
- new net: BD8. (X), BD9. (X)
- new net: BD4. (X), BD9. (X)
- new net: BD13. (X), BD14. (X)
- new net: BD14. (X), BD16. (X)
- new net: BC14. (X), BC16. (X)
- new net: BC13. (X), BC14. (X)
- new net: BB3. (X), BB4. (X)
- new net: BC2. (X), BC4. (X)
- new net: BD3. (X), BD4. (X)
- new net: BA6. (X), BA8. (X)
- new net: BD7. (X), BD8. (X)
- new net: BA5. (X), BA8. (X)
- new net: BE14. (X), BE16. (X)
- new net: BE13. (X), BE14. (X)
- new net: BE5. (X), BE8. (X)
- new net: BC17. (X), BC9. (X)
- new net: BE2. (X), BE4. (X)
- new net: BE4. (X), BE9. (X)
- new net: BE3. (X), BE4. (X)
- new net: BB7. (X), BB8. (X)
- new net: BB2. (X), BB4. (X)
- new net: BA12. (X), BA9. (X)
- new net: BA11. (X), BA12. (X)
- new net: BA12. (X), BA13. (X)
- new net: BD1. (X), BD4. (X)
- new net: BD11. (X), BD12. (X)
- new net: BA7. (X), BA8. (X)
- new net: BB12. (X), BB9. (X)
- new net: BB12. (X), BB13. (X)
- new net: BB11. (X), BB12. (X)
- new net: BC10. (X), BC12. (X)
- new net: BB8. (X), BB9. (X)
- new net: BB17. (X), BB9. (X)
- new net: BB14. (X), BB15. (X)
- new net: BB14. (X), BB16. (X)
- new net: BB6. (X), BB8. (X)
- new net: BD10. (X), BD12. (X)
- new net: BD6. (X), BD8. (X)
- new net: BA14. (X), BA15. (X)
- new net: BA14. (X), BA16. (X)
- new net: BA3. (X), BA4. (X)
- new net: BC5. (X), BC8. (X)
- new net: BC8. (X), BC9. (X)
- new net: BC4. (X), BC9. (X)
- new net: BA4. (X), BA9. (X)
- new net: BA1. (X), BA4. (X)
- new net: BC6. (X), BC8. (X)
- new net: BE11. (X), BE12. (X)
- new net: BE8. (X), BE9. (X)
- new net: BE7. (X), BE8. (X)
- new net: BC1. (X), BC4. (X)
- new net: BE10. (X), BE12. (X)
- new net: BE17. (X), BE9. (X)

Commit message: I fixed 2 errors in the letterless MMC5 tracing:
1. BK5 is a NAND-4 gate.  It was thought to be NAND-3 before.
2.  BL83 and BL96 signals got swapped here before.  They actually cross each other:

BL83 = "PPU_RW_Mode_%0x_Access"
BL96 = "+ExRAM_Mode_$0x"

This propagated out to several changes in the schematic.
Connections:
- net at BD9. (X): now also BD12. (X); no longer BD17. (X)
- net at BD8. (X): now also BD5. (X); no longer BD9. (X)
- net at BD4. (X): now also BD2. (X); no longer BD9. (X)
- net at BD12. (X): now also BD13. (X); no longer BD9. (X)
- net at BD14. (X): now also BD15. (X); no longer BD13. (X)
- net at BC14. (X): now also BC15. (X); no longer BC16. (X)
- net at BC13. (X): now also BC12. (X); no longer BC14. (X)
- net at BC12. (X): now also BC11. (X); no longer BC13. (X)
- net at BB4. (X): now also BB1. (X); no longer BB3. (X)
- net at BC4. (X): now also BC3. (X); no longer BC2. (X)
- net at BA8. (X): now also BA9. (X); no longer BA6. (X)
- net at BE14. (X): now also BE15. (X); no longer BE16. (X)
- net at BE13. (X): now also BE12. (X); no longer BE14. (X)
- net at BE8. (X): now also BE6. (X); no longer BE5. (X)
- net at BC9. (X): now also BC12. (X); no longer BC17. (X)
- net at BE4. (X): now also BE1. (X); no longer BE2. (X)
- net at BE9. (X): now also BE12. (X); no longer BE4. (X)
- net at BB8. (X): now also BB5. (X); no longer BB7. (X)
- net at BA12. (X): now also BA10. (X); no longer BA9. (X)
- net at BA13. (X): now also BA14. (X); no longer BA12. (X)
- net at BA9. (X): now also BA17. (X); no longer BA8. (X)
- net at BB12. (X): now also BB10. (X); no longer BB9. (X)
- net at BB13. (X): now also BB14. (X); no longer BB12. (X)
- net at BB9. (X): now also BB4. (X); no longer BB8. (X)
- net at BA4. (X): now also BA2. (X); no longer BA3. (X)
- net at BC8. (X): now also BC7. (X); no longer BC5. (X)
- new net: BD17. (X), BD9. (X)
- new net: BD8. (X), BD9. (X)
- new net: BD4. (X), BD9. (X)
- new net: BD13. (X), BD14. (X)
- new net: BD14. (X), BD16. (X)
- new net: BC14. (X), BC16. (X)
- new net: BC13. (X), BC14. (X)
- new net: BB3. (X), BB4. (X)
- new net: BC2. (X), BC4. (X)
- new net: BD3. (X), BD4. (X)
- new net: BA6. (X), BA8. (X)
- new net: BD7. (X), BD8. (X)
- new net: BA5. (X), BA8. (X)
- new net: BE14. (X), BE16. (X)
- new net: BE13. (X), BE14. (X)
- new net: BE5. (X), BE8. (X)
- new net: BC17. (X), BC9. (X)
- new net: BE2. (X), BE4. (X)
- new net: BE4. (X), BE9. (X)
- new net: BE3. (X), BE4. (X)
- new net: BB7. (X), BB8. (X)
- new net: BB2. (X), BB4. (X)
- new net: BA12. (X), BA9. (X)
- new net: BA11. (X), BA12. (X)
- new net: BA12. (X), BA13. (X)
- new net: BD1. (X), BD4. (X)
- new net: BD11. (X), BD12. (X)
- new net: BA7. (X), BA8. (X)
- new net: BB12. (X), BB9. (X)
- new net: BB12. (X), BB13. (X)
- new net: BB11. (X), BB12. (X)
- new net: BC10. (X), BC12. (X)
- new net: BB8. (X), BB9. (X)
- new net: BB17. (X), BB9. (X)
- new net: BB14. (X), BB15. (X)
- new net: BB14. (X), BB16. (X)
- new net: BB6. (X), BB8. (X)
- new net: BD10. (X), BD12. (X)
- new net: BD6. (X), BD8. (X)
- new net: BA14. (X), BA15. (X)
- new net: BA14. (X), BA16. (X)
- new net: BA3. (X), BA4. (X)
- new net: BC5. (X), BC8. (X)
- new net: BC8. (X), BC9. (X)
- new net: BC4. (X), BC9. (X)
- new net: BA4. (X), BA9. (X)
- new net: BA1. (X), BA4. (X)
- new net: BC6. (X), BC8. (X)
- new net: BE11. (X), BE12. (X)
- new net: BE8. (X), BE9. (X)
- new net: BE7. (X), BE8. (X)
- new net: BC1. (X), BC4. (X)
- new net: BE10. (X), BE12. (X)
- new net: BE17. (X), BE9. (X)

Commit message: Schematic and SVG Updates
Connections:
- net at BD9. (X): now also BD12. (X); no longer BD17. (X)
- net at BD8. (X): now also BD5. (X); no longer BD9. (X)
- net at BD4. (X): now also BD2. (X); no longer BD9. (X)
- net at BD12. (X): now also BD13. (X); no longer BD9. (X)
- net at BD14. (X): now also BD15. (X); no longer BD13. (X)
- net at BC14. (X): now also BC15. (X); no longer BC16. (X)
- net at BC13. (X): now also BC12. (X); no longer BC14. (X)
- net at BC12. (X): now also BC11. (X); no longer BC13. (X)
- net at BB4. (X): now also BB1. (X); no longer BB3. (X)
- net at BC4. (X): now also BC3. (X); no longer BC2. (X)
- net at BA8. (X): now also BA9. (X); no longer BA6. (X)
- net at BE14. (X): now also BE15. (X); no longer BE16. (X)
- net at BE13. (X): now also BE12. (X); no longer BE14. (X)
- net at BE8. (X): now also BE6. (X); no longer BE5. (X)
- net at BC9. (X): now also BC12. (X); no longer BC17. (X)
- net at BE4. (X): now also BE1. (X); no longer BE2. (X)
- net at BE9. (X): now also BE12. (X); no longer BE4. (X)
- net at BB8. (X): now also BB5. (X); no longer BB7. (X)
- net at BA12. (X): now also BA10. (X); no longer BA9. (X)
- net at BA13. (X): now also BA14. (X); no longer BA12. (X)
- net at BA9. (X): now also BA17. (X); no longer BA8. (X)
- net at BB12. (X): now also BB10. (X); no longer BB9. (X)
- net at BB13. (X): now also BB14. (X); no longer BB12. (X)
- net at BB9. (X): now also BB4. (X); no longer BB8. (X)
- net at BA4. (X): now also BA2. (X); no longer BA3. (X)
- net at BC8. (X): now also BC7. (X); no longer BC5. (X)
- new net: BD17. (X), BD9. (X)
- new net: BD8. (X), BD9. (X)
- new net: BD4. (X), BD9. (X)
- new net: BD13. (X), BD14. (X)
- new net: BD14. (X), BD16. (X)
- new net: BC14. (X), BC16. (X)
- new net: BC13. (X), BC14. (X)
- new net: BB3. (X), BB4. (X)
- new net: BC2. (X), BC4. (X)
- new net: BD3. (X), BD4. (X)
- new net: BA6. (X), BA8. (X)
- new net: BD7. (X), BD8. (X)
- new net: BA5. (X), BA8. (X)
- new net: BE14. (X), BE16. (X)
- new net: BE13. (X), BE14. (X)
- new net: BE5. (X), BE8. (X)
- new net: BC17. (X), BC9. (X)
- new net: BE2. (X), BE4. (X)
- new net: BE4. (X), BE9. (X)
- new net: BE3. (X), BE4. (X)
- new net: BB7. (X), BB8. (X)
- new net: BB2. (X), BB4. (X)
- new net: BA12. (X), BA9. (X)
- new net: BA11. (X), BA12. (X)
- new net: BA12. (X), BA13. (X)
- new net: BD1. (X), BD4. (X)
- new net: BD11. (X), BD12. (X)
- new net: BA7. (X), BA8. (X)
- new net: BB12. (X), BB9. (X)
- new net: BB12. (X), BB13. (X)
- new net: BB11. (X), BB12. (X)
- new net: BC10. (X), BC12. (X)
- new net: BB8. (X), BB9. (X)
- new net: BB17. (X), BB9. (X)
- new net: BB14. (X), BB15. (X)
- new net: BB14. (X), BB16. (X)
- new net: BB6. (X), BB8. (X)
- new net: BD10. (X), BD12. (X)
- new net: BD6. (X), BD8. (X)
- new net: BA14. (X), BA15. (X)
- new net: BA14. (X), BA16. (X)
- new net: BA3. (X), BA4. (X)
- new net: BC5. (X), BC8. (X)
- new net: BC8. (X), BC9. (X)
- new net: BC4. (X), BC9. (X)
- new net: BA4. (X), BA9. (X)
- new net: BA1. (X), BA4. (X)
- new net: BC6. (X), BC8. (X)
- new net: BE11. (X), BE12. (X)
- new net: BE8. (X), BE9. (X)
- new net: BE7. (X), BE8. (X)
- new net: BC1. (X), BC4. (X)
- new net: BE10. (X), BE12. (X)
- new net: BE17. (X), BE9. (X)

Commit message: Schematic and SVG Updates
Connections:
- net at BD9. (X): now also BD12. (X); no longer BD17. (X)
- net at BD8. (X): now also BD5. (X); no longer BD9. (X)
- net at BD4. (X): now also BD2. (X); no longer BD9. (X)
- net at BD12. (X): now also BD13. (X); no longer BD9. (X)
- net at BD14. (X): now also BD15. (X); no longer BD13. (X)
- net at BC14. (X): now also BC15. (X); no longer BC16. (X)
- net at BC13. (X): now also BC12. (X); no longer BC14. (X)
- net at BC12. (X): now also BC11. (X); no longer BC13. (X)
- net at BB4. (X): now also BB1. (X); no longer BB3. (X)
- net at BC4. (X): now also BC3. (X); no longer BC2. (X)
- net at BA8. (X): now also BA9. (X); no longer BA6. (X)
- net at BE14. (X): now also BE15. (X); no longer BE16. (X)
- net at BE13. (X): now also BE12. (X); no longer BE14. (X)
- net at BE8. (X): now also BE6. (X); no longer BE5. (X)
- net at BC9. (X): now also BC12. (X); no longer BC17. (X)
- net at BE4. (X): now also BE1. (X); no longer BE2. (X)
- net at BE9. (X): now also BE12. (X); no longer BE4. (X)
- net at BB8. (X): now also BB5. (X); no longer BB7. (X)
- net at BA12. (X): now also BA10. (X); no longer BA9. (X)
- net at BA13. (X): now also BA14. (X); no longer BA12. (X)
- net at BA9. (X): now also BA17. (X); no longer BA8. (X)
- net at BB12. (X): now also BB10. (X); no longer BB9. (X)
- net at BB13. (X): now also BB14. (X); no longer BB12. (X)
- net at BB9. (X): now also BB4. (X); no longer BB8. (X)
- net at BA4. (X): now also BA2. (X); no longer BA3. (X)
- net at BC8. (X): now also BC7. (X); no longer BC5. (X)
- new net: BD17. (X), BD9. (X)
- new net: BD8. (X), BD9. (X)
- new net: BD4. (X), BD9. (X)
- new net: BD13. (X), BD14. (X)
- new net: BD14. (X), BD16. (X)
- new net: BC14. (X), BC16. (X)
- new net: BC13. (X), BC14. (X)
- new net: BB3. (X), BB4. (X)
- new net: BC2. (X), BC4. (X)
- new net: BD3. (X), BD4. (X)
- new net: BA6. (X), BA8. (X)
- new net: BD7. (X), BD8. (X)
- new net: BA5. (X), BA8. (X)
- new net: BE14. (X), BE16. (X)
- new net: BE13. (X), BE14. (X)
- new net: BE5. (X), BE8. (X)
- new net: BC17. (X), BC9. (X)
- new net: BE2. (X), BE4. (X)
- new net: BE4. (X), BE9. (X)
- new net: BE3. (X), BE4. (X)
- new net: BB7. (X), BB8. (X)
- new net: BB2. (X), BB4. (X)
- new net: BA12. (X), BA9. (X)
- new net: BA11. (X), BA12. (X)
- new net: BA12. (X), BA13. (X)
- new net: BD1. (X), BD4. (X)
- new net: BD11. (X), BD12. (X)
- new net: BA7. (X), BA8. (X)
- new net: BB12. (X), BB9. (X)
- new net: BB12. (X), BB13. (X)
- new net: BB11. (X), BB12. (X)
- new net: BC10. (X), BC12. (X)
- new net: BB8. (X), BB9. (X)
- new net: BB17. (X), BB9. (X)
- new net: BB14. (X), BB15. (X)
- new net: BB14. (X), BB16. (X)
- new net: BB6. (X), BB8. (X)
- new net: BD10. (X), BD12. (X)
- new net: BD6. (X), BD8. (X)
- new net: BA14. (X), BA15. (X)
- new net: BA14. (X), BA16. (X)
- new net: BA3. (X), BA4. (X)
- new net: BC5. (X), BC8. (X)
- new net: BC8. (X), BC9. (X)
- new net: BC4. (X), BC9. (X)
- new net: BA4. (X), BA9. (X)
- new net: BA1. (X), BA4. (X)
- new net: BC6. (X), BC8. (X)
- new net: BE11. (X), BE12. (X)
- new net: BE8. (X), BE9. (X)
- new net: BE7. (X), BE8. (X)
- new net: BC1. (X), BC4. (X)
- new net: BE10. (X), BE12. (X)
- new net: BE17. (X), BE9. (X)
