File: Schematic (KiCAD)/chr_address_bus_15_to_19.kicad_sch (KiCad schematic)
At the start: 85 parts

Commit message: Tracing and schematic updates.  - Added timer to schematic.  - Added all items from artifacts sheet to the MMC5A trace.
Connections:
- net at BD9. (X): now also BD12. (X); no longer BD17. (X)
- net at BD8. (X): now also BD5. (X); no longer BD9. (X)
- net at BD4. (X): now also BD2. (X); no longer BD9. (X)
- net at BD12. (X): now also BD13. (X); no longer BD9. (X)
- net at BD14. (X): now also BD15. (X); no longer BD13. (X)
- net at BC14. (X): now also BC15. (X); no longer BC16. (X)
- net at BC13. (X): now also BC12. (X); no longer BC14. (X)
- net at BC12. (X): now also BC11. (X); no longer BC13. (X)
- net at BB4. (X): now also BB1. (X); no longer BB3. (X)
- net at BC4. (X): now also BC3. (X); no longer BC2. (X)
- net at BA8. (X): now also BA9. (X); no longer BA6. (X)
- net at BE14. (X): now also BE15. (X); no longer BE16. (X)
- net at BE13. (X): now also BE12. (X); no longer BE14. (X)
- net at BE8. (X): now also BE6. (X); no longer BE5. (X)
- net at BC9. (X): now also BC12. (X); no longer BC17. (X)
- net at BE4. (X): now also BE1. (X); no longer BE2. (X)
- net at BE9. (X): now also BE12. (X); no longer BE4. (X)
- net at BB8. (X): now also BB5. (X); no longer BB7. (X)
- net at BA12. (X): now also BA10. (X); no longer BA9. (X)
- net at BA13. (X): now also BA14. (X); no longer BA12. (X)
- net at BA9. (X): now also BA17. (X); no longer BA8. (X)
- net at BB12. (X): now also BB10. (X); no longer BB9. (X)
- net at BB13. (X): now also BB14. (X); no longer BB12. (X)
- net at BB9. (X): now also BB4. (X); no longer BB8. (X)
- net at BA4. (X): now also BA2. (X); no longer BA3. (X)
- net at BC8. (X): now also BC7. (X); no longer BC5. (X)
- new net: BD17. (X), BD9. (X)
- new net: BD8. (X), BD9. (X)
- new net: BD4. (X), BD9. (X)
- new net: BD13. (X), BD14. (X)
- new net: BD14. (X), BD16. (X)
- new net: BC14. (X), BC16. (X)
- new net: BC13. (X), BC14. (X)
- new net: BB3. (X), BB4. (X)
- new net: BC2. (X), BC4. (X)
- new net: BD3. (X), BD4. (X)
- new net: BA6. (X), BA8. (X)
- new net: BD7. (X), BD8. (X)
- new net: BA5. (X), BA8. (X)
- new net: BE14. (X), BE16. (X)
- new net: BE13. (X), BE14. (X)
- new net: BE5. (X), BE8. (X)
- new net: BC17. (X), BC9. (X)
- new net: BE2. (X), BE4. (X)
- new net: BE4. (X), BE9. (X)
- new net: BE3. (X), BE4. (X)
- new net: BB7. (X), BB8. (X)
- new net: BB2. (X), BB4. (X)
- new net: BA12. (X), BA9. (X)
- new net: BA11. (X), BA12. (X)
- new net: BA12. (X), BA13. (X)
- new net: BD1. (X), BD4. (X)
- new net: BD11. (X), BD12. (X)
- new net: BA7. (X), BA8. (X)
- new net: BB12. (X), BB9. (X)
- new net: BB12. (X), BB13. (X)
- new net: BB11. (X), BB12. (X)
- new net: BC10. (X), BC12. (X)
- new net: BB8. (X), BB9. (X)
- new net: BB17. (X), BB9. (X)
- new net: BB14. (X), BB15. (X)
- new net: BB14. (X), BB16. (X)
- new net: BB6. (X), BB8. (X)
- new net: BD10. (X), BD12. (X)
- new net: BD6. (X), BD8. (X)
- new net: BA14. (X), BA15. (X)
- new net: BA14. (X), BA16. (X)
- new net: BA3. (X), BA4. (X)
- new net: BC5. (X), BC8. (X)
- new net: BC8. (X), BC9. (X)
- new net: BC4. (X), BC9. (X)
- new net: BA4. (X), BA9. (X)
- new net: BA1. (X), BA4. (X)
- new net: BC6. (X), BC8. (X)
- new net: BE11. (X), BE12. (X)
- new net: BE8. (X), BE9. (X)
- new net: BE7. (X), BE8. (X)
- new net: BC1. (X), BC4. (X)
- new net: BE10. (X), BE12. (X)
- new net: BE17. (X), BE9. (X)

Commit message: Added the new MMC5A read-register bits in the schematic. Additional MMC5A tracing work.
Connections:
- net at BD9. (X): now also BD12. (X); no longer BD17. (X)
- net at BD8. (X): now also BD5. (X); no longer BD9. (X)
- net at BD4. (X): now also BD2. (X); no longer BD9. (X)
- net at BD12. (X): now also BD13. (X); no longer BD9. (X)
- net at BD14. (X): now also BD15. (X); no longer BD13. (X)
- net at BC14. (X): now also BC15. (X); no longer BC16. (X)
- net at BC13. (X): now also BC12. (X); no longer BC14. (X)
- net at BC12. (X): now also BC11. (X); no longer BC13. (X)
- net at BB4. (X): now also BB1. (X); no longer BB3. (X)
- net at BC4. (X): now also BC3. (X); no longer BC2. (X)
- net at BA8. (X): now also BA9. (X); no longer BA6. (X)
- net at BE14. (X): now also BE15. (X); no longer BE16. (X)
- net at BE13. (X): now also BE12. (X); no longer BE14. (X)
- net at BE8. (X): now also BE6. (X); no longer BE5. (X)
- net at BC9. (X): now also BC12. (X); no longer BC17. (X)
- net at BE4. (X): now also BE1. (X); no longer BE2. (X)
- net at BE9. (X): now also BE12. (X); no longer BE4. (X)
- net at BB8. (X): now also BB5. (X); no longer BB7. (X)
- net at BA12. (X): now also BA10. (X); no longer BA9. (X)
- net at BA13. (X): now also BA14. (X); no longer BA12. (X)
- net at BA9. (X): now also BA17. (X); no longer BA8. (X)
- net at BB12. (X): now also BB10. (X); no longer BB9. (X)
- net at BB13. (X): now also BB14. (X); no longer BB12. (X)
- net at BB9. (X): now also BB4. (X); no longer BB8. (X)
- net at BA4. (X): now also BA2. (X); no longer BA3. (X)
- net at BC8. (X): now also BC7. (X); no longer BC5. (X)
- new net: BD17. (X), BD9. (X)
- new net: BD8. (X), BD9. (X)
- new net: BD4. (X), BD9. (X)
- new net: BD13. (X), BD14. (X)
- new net: BD14. (X), BD16. (X)
- new net: BC14. (X), BC16. (X)
- new net: BC13. (X), BC14. (X)
- new net: BB3. (X), BB4. (X)
- new net: BC2. (X), BC4. (X)
- new net: BD3. (X), BD4. (X)
- new net: BA6. (X), BA8. (X)
- new net: BD7. (X), BD8. (X)
- new net: BA5. (X), BA8. (X)
- new net: BE14. (X), BE16. (X)
- new net: BE13. (X), BE14. (X)
- new net: BE5. (X), BE8. (X)
- new net: BC17. (X), BC9. (X)
- new net: BE2. (X), BE4. (X)
- new net: BE4. (X), BE9. (X)
- new net: BE3. (X), BE4. (X)
- new net: BB7. (X), BB8. (X)
- new net: BB2. (X), BB4. (X)
- new net: BA12. (X), BA9. (X)
- new net: BA11. (X), BA12. (X)
- new net: BA12. (X), BA13. (X)
- new net: BD1. (X), BD4. (X)
- new net: BD11. (X), BD12. (X)
- new net: BA7. (X), BA8. (X)
- new net: BB12. (X), BB9. (X)
- new net: BB12. (X), BB13. (X)
- new net: BB11. (X), BB12. (X)
- new net: BC10. (X), BC12. (X)
- new net: BB8. (X), BB9. (X)
- new net: BB17. (X), BB9. (X)
- new net: BB14. (X), BB15. (X)
- new net: BB14. (X), BB16. (X)
- new net: BB6. (X), BB8. (X)
- new net: BD10. (X), BD12. (X)
- new net: BD6. (X), BD8. (X)
- new net: BA14. (X), BA15. (X)
- new net: BA14. (X), BA16. (X)
- new net: BA3. (X), BA4. (X)
- new net: BC5. (X), BC8. (X)
- new net: BC8. (X), BC9. (X)
- new net: BC4. (X), BC9. (X)
- new net: BA4. (X), BA9. (X)
- new net: BA1. (X), BA4. (X)
- new net: BC6. (X), BC8. (X)
- new net: BE11. (X), BE12. (X)
- new net: BE8. (X), BE9. (X)
- new net: BE7. (X), BE8. (X)
- new net: BC1. (X), BC4. (X)
- new net: BE10. (X), BE12. (X)
- new net: BE17. (X), BE9. (X)

Commit message: - Fixed the register read bit schematic errors noted by Joe in the Nesdev forum.
Connections:
- net at BD9. (X): now also BD12. (X); no longer BD17. (X)
- net at BD8. (X): now also BD5. (X); no longer BD9. (X)
- net at BD4. (X): now also BD2. (X); no longer BD9. (X)
- net at BD12. (X): now also BD13. (X); no longer BD9. (X)
- net at BD14. (X): now also BD15. (X); no longer BD13. (X)
- net at BC14. (X): now also BC15. (X); no longer BC16. (X)
- net at BC13. (X): now also BC12. (X); no longer BC14. (X)
- net at BC12. (X): now also BC11. (X); no longer BC13. (X)
- net at BB4. (X): now also BB1. (X); no longer BB3. (X)
- net at BC4. (X): now also BC3. (X); no longer BC2. (X)
- net at BA8. (X): now also BA9. (X); no longer BA6. (X)
- net at BE14. (X): now also BE15. (X); no longer BE16. (X)
- net at BE13. (X): now also BE12. (X); no longer BE14. (X)
- net at BE8. (X): now also BE6. (X); no longer BE5. (X)
- net at BC9. (X): now also BC12. (X); no longer BC17. (X)
- net at BE4. (X): now also BE1. (X); no longer BE2. (X)
- net at BE9. (X): now also BE12. (X); no longer BE4. (X)
- net at BB8. (X): now also BB5. (X); no longer BB7. (X)
- net at BA12. (X): now also BA10. (X); no longer BA9. (X)
- net at BA13. (X): now also BA14. (X); no longer BA12. (X)
- net at BA9. (X): now also BA17. (X); no longer BA8. (X)
- net at BB12. (X): now also BB10. (X); no longer BB9. (X)
- net at BB13. (X): now also BB14. (X); no longer BB12. (X)
- net at BB9. (X): now also BB4. (X); no longer BB8. (X)
- net at BA4. (X): now also BA2. (X); no longer BA3. (X)
- net at BC8. (X): now also BC7. (X); no longer BC5. (X)
- new net: BD17. (X), BD9. (X)
- new net: BD8. (X), BD9. (X)
- new net: BD4. (X), BD9. (X)
- new net: BD13. (X), BD14. (X)
- new net: BD14. (X), BD16. (X)
- new net: BC14. (X), BC16. (X)
- new net: BC13. (X), BC14. (X)
- new net: BB3. (X), BB4. (X)
- new net: BC2. (X), BC4. (X)
- new net: BD3. (X), BD4. (X)
- new net: BA6. (X), BA8. (X)
- new net: BD7. (X), BD8. (X)
- new net: BA5. (X), BA8. (X)
- new net: BE14. (X), BE16. (X)
- new net: BE13. (X), BE14. (X)
- new net: BE5. (X), BE8. (X)
- new net: BC17. (X), BC9. (X)
- new net: BE2. (X), BE4. (X)
- new net: BE4. (X), BE9. (X)
- new net: BE3. (X), BE4. (X)
- new net: BB7. (X), BB8. (X)
- new net: BB2. (X), BB4. (X)
- new net: BA12. (X), BA9. (X)
- new net: BA11. (X), BA12. (X)
- new net: BA12. (X), BA13. (X)
- new net: BD1. (X), BD4. (X)
- new net: BD11. (X), BD12. (X)
- new net: BA7. (X), BA8. (X)
- new net: BB12. (X), BB9. (X)
- new net: BB12. (X), BB13. (X)
- new net: BB11. (X), BB12. (X)
- new net: BC10. (X), BC12. (X)
- new net: BB8. (X), BB9. (X)
- new net: BB17. (X), BB9. (X)
- new net: BB14. (X), BB15. (X)
- new net: BB14. (X), BB16. (X)
- new net: BB6. (X), BB8. (X)
- new net: BD10. (X), BD12. (X)
- new net: BD6. (X), BD8. (X)
- new net: BA14. (X), BA15. (X)
- new net: BA14. (X), BA16. (X)
- new net: BA3. (X), BA4. (X)
- new net: BC5. (X), BC8. (X)
- new net: BC8. (X), BC9. (X)
- new net: BC4. (X), BC9. (X)
- new net: BA4. (X), BA9. (X)
- new net: BA1. (X), BA4. (X)
- new net: BC6. (X), BC8. (X)
- new net: BE11. (X), BE12. (X)
- new net: BE8. (X), BE9. (X)
- new net: BE7. (X), BE8. (X)
- new net: BC1. (X), BC4. (X)
- new net: BE10. (X), BE12. (X)
- new net: BE17. (X), BE9. (X)

Commit message: - Updated all of the various And-OR-Invert gates to have consistent names.  - Added the schematic for CL3 / SL3 GPIO pins.  There are no surprises revealed by this.  - Finished up the CPU address decoding tracing.  - Added one of the 'artifact' counters from the pulse channels
Connections:
- net at BD9. (X): now also BD12. (X); no longer BD17. (X)
- net at BD8. (X): now also BD5. (X); no longer BD9. (X)
- net at BD4. (X): now also BD2. (X); no longer BD9. (X)
- net at BD12. (X): now also BD13. (X); no longer BD9. (X)
- net at BD14. (X): now also BD15. (X); no longer BD13. (X)
- net at BC14. (X): now also BC15. (X); no longer BC16. (X)
- net at BC13. (X): now also BC12. (X); no longer BC14. (X)
- net at BC12. (X): now also BC11. (X); no longer BC13. (X)
- net at BB4. (X): now also BB1. (X); no longer BB3. (X)
- net at BC4. (X): now also BC3. (X); no longer BC2. (X)
- net at BA8. (X): now also BA9. (X); no longer BA6. (X)
- net at BE14. (X): now also BE15. (X); no longer BE16. (X)
- net at BE13. (X): now also BE12. (X); no longer BE14. (X)
- net at BE8. (X): now also BE6. (X); no longer BE5. (X)
- net at BC9. (X): now also BC12. (X); no longer BC17. (X)
- net at BE4. (X): now also BE1. (X); no longer BE2. (X)
- net at BE9. (X): now also BE12. (X); no longer BE4. (X)
- net at BB8. (X): now also BB5. (X); no longer BB7. (X)
- net at BA12. (X): now also BA10. (X); no longer BA9. (X)
- net at BA13. (X): now also BA14. (X); no longer BA12. (X)
- net at BA9. (X): now also BA17. (X); no longer BA8. (X)
- net at BB12. (X): now also BB10. (X); no longer BB9. (X)
- net at BB13. (X): now also BB14. (X); no longer BB12. (X)
- net at BB9. (X): now also BB4. (X); no longer BB8. (X)
- net at BA4. (X): now also BA2. (X); no longer BA3. (X)
- net at BC8. (X): now also BC7. (X); no longer BC5. (X)
- new net: BD17. (X), BD9. (X)
- new net: BD8. (X), BD9. (X)
- new net: BD4. (X), BD9. (X)
- new net: BD13. (X), BD14. (X)
- new net: BD14. (X), BD16. (X)
- new net: BC14. (X), BC16. (X)
- new net: BC13. (X), BC14. (X)
- new net: BB3. (X), BB4. (X)
- new net: BC2. (X), BC4. (X)
- new net: BD3. (X), BD4. (X)
- new net: BA6. (X), BA8. (X)
- new net: BD7. (X), BD8. (X)
- new net: BA5. (X), BA8. (X)
- new net: BE14. (X), BE16. (X)
- new net: BE13. (X), BE14. (X)
- new net: BE5. (X), BE8. (X)
- new net: BC17. (X), BC9. (X)
- new net: BE2. (X), BE4. (X)
- new net: BE4. (X), BE9. (X)
- new net: BE3. (X), BE4. (X)
- new net: BB7. (X), BB8. (X)
- new net: BB2. (X), BB4. (X)
- new net: BA12. (X), BA9. (X)
- new net: BA11. (X), BA12. (X)
- new net: BA12. (X), BA13. (X)
- new net: BD1. (X), BD4. (X)
- new net: BD11. (X), BD12. (X)
- new net: BA7. (X), BA8. (X)
- new net: BB12. (X), BB9. (X)
- new net: BB12. (X), BB13. (X)
- new net: BB11. (X), BB12. (X)
- new net: BC10. (X), BC12. (X)
- new net: BB8. (X), BB9. (X)
- new net: BB17. (X), BB9. (X)
- new net: BB14. (X), BB15. (X)
- new net: BB14. (X), BB16. (X)
- new net: BB6. (X), BB8. (X)
- new net: BD10. (X), BD12. (X)
- new net: BD6. (X), BD8. (X)
- new net: BA14. (X), BA15. (X)
- new net: BA14. (X), BA16. (X)
- new net: BA3. (X), BA4. (X)
- new net: BC5. (X), BC8. (X)
- new net: BC8. (X), BC9. (X)
- new net: BC4. (X), BC9. (X)
- new net: BA4. (X), BA9. (X)
- new net: BA1. (X), BA4. (X)
- new net: BC6. (X), BC8. (X)
- new net: BE11. (X), BE12. (X)
- new net: BE8. (X), BE9. (X)
- new net: BE7. (X), BE8. (X)
- new net: BC1. (X), BC4. (X)
- new net: BE10. (X), BE12. (X)
- new net: BE17. (X), BE9. (X)
