File: Schematic (KiCAD)/multiplier.kicad_sch (KiCad schematic)
At the start: 37 parts

Commit message: - Lots of additional comments and signal name improvements.  - "Don't know what this is yet but it is important" section of the pulse channels:    - I worked out the logic and it is a 4-bit binary up-counter with preload, made from gates and D-latches instead of T-flip-flops.    - It is extremely similar to the envelope counter, but takes twice the die space and much more traces.    - None of its outputs go anywhere else, so I believe that it has no actual function.    - It seems to be a previous attempt at making the envelope counter and it got disconnected and left in.    - Each pulse channel has its own copy and I moved both of them to the "Artifacts" sheet.    - The wasted space amounts to about half of one of the large columns on the left side of the die.  - A couple of "OAI2" cells that noted "unclear order": I determined the correct order of the inputs based on several others which were known.  - Deduced the purpose of the 2 separate methods of scanline detection:    - The one looking for 3 consecutive reads finds the start of a scanline.    - The one counting PPU /RD to find PPU cycle 336, finds the end of the scanline.    - I moved these beside each other on the same sheet for clarity.  - A66.5 Changed from Nand to Nor in order to make sense.  - Basic test mode:    - Pin 92: Active low, enables test mode.    - Pin 29: In test mode, it gives external control of "Scanline Start Detection", which is normally done with the familiar 3 matching PPU reads.  When not in test mode, the pin has no function.    - Pin 30: In test mode, it gives external control of "Scanline End Detection", which is normally done by counting PPU /RD to find PPU cycle 336.  It also gives control of "Pulse Length Clock" when in test mode.  When not in test mode, the pin has no function.    - Pin 98/SL3: In test mode, it gives external control of "Pulse Timer Clock".  Whether or not in test mode, this pin low makes the MMC5 pretend $5104 had not yet been written since reset, probably as a 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
Connections:
- net at MUL7. (X): now also BL77. (X); no longer MULTIPLIER. (Y15)
- net at MUL14. (X): now also MULTIPLIER. (Y15); no longer BL68. (X)
- net at MULTIPLIER. (Y15): now also MUL16. (X); no longer MUL14. (X)
- net at MUL6. (X): now also BL76. (X); no longer MULTIPLIER. (Y15)
- net at MUL10. (X): now also MULTIPLIER. (Y15); no longer BL72. (X)
- net at MUL13. (X): now also MULTIPLIER. (Y15); no longer BL67. (X)
- net at MUL11. (X): now also MULTIPLIER. (Y15); no longer BL65. (X)
- net at MUL2. (X): now also MULTIPLIER. (Y15); no longer BL64. (X)
- net at MUL3. (X): now also BL73. (X); no longer MULTIPLIER. (Y15)
- net at MUL4. (X): now also BL74. (X); no longer MULTIPLIER. (Y15)
- net at MUL1. (X): now also BL63. (X); no longer MULTIPLIER. (Y15)
- net at MUL9. (X): now also BL71. (X); no longer MULTIPLIER. (Y15)
- net at MUL15. (X): now also BL69. (X); no longer MULTIPLIER. (Y15)
- net at MUL5. (X): now also BL75. (X); no longer MULTIPLIER. (Y15)
- net at MUL8. (X): now also BL78. (X); no longer MULTIPLIER. (Y15)
- net at MUL12. (X): now also BL66. (X); no longer MULTIPLIER. (Y15)
- net at MUL16. (X): now also BL70. (X); no longer MULTIPLIER. (Y15)
- new net: MUL7. (X), MULTIPLIER. (Y15)
- new net: BL68. (X), MUL14. (X)
- new net: MUL17. (X), MUL27. (/Q7)
- new net: MUL6. (X), MULTIPLIER. (Y15)
- new net: BL72. (X), MUL10. (X)
- new net: BL67. (X), MUL13. (X)
- new net: BL65. (X), MUL11. (X)
- new net: MUL18. (/Q7), MUL28. (X)
- new net: BL64. (X), MUL2. (X)
- new net: MUL3. (X), MULTIPLIER. (Y15)
- new net: MUL4. (X), MULTIPLIER. (Y15)
- new net: MUL27. (/Q7), MULTIPLIER. (Y15) (x8)
- new net: MUL1. (X), MULTIPLIER. (Y15)
- new net: MUL9. (X), MULTIPLIER. (Y15)
- new net: MUL15. (X), MULTIPLIER. (Y15)
- new net: MUL5. (X), MULTIPLIER. (Y15)
- new net: MUL8. (X), MULTIPLIER. (Y15)
- new net: MUL18. (/Q7), MULTIPLIER. (Y15) (x8)
- new net: MUL12. (X), MULTIPLIER. (Y15)

Commit message: - Improved "Identification of Cells" document for NAND, NOR, and XNOR/XOR gates.  - Gate S16 is a NAND-8 gate; it was shown as NOR-8 before.
Connections:
- net at MUL7. (X): now also BL77. (X); no longer MULTIPLIER. (Y15)
- net at MUL14. (X): now also MULTIPLIER. (Y15); no longer BL68. (X)
- net at MULTIPLIER. (Y15): now also MUL16. (X); no longer MUL14. (X)
- net at MUL6. (X): now also BL76. (X); no longer MULTIPLIER. (Y15)
- net at MUL10. (X): now also MULTIPLIER. (Y15); no longer BL72. (X)
- net at MUL13. (X): now also MULTIPLIER. (Y15); no longer BL67. (X)
- net at MUL11. (X): now also MULTIPLIER. (Y15); no longer BL65. (X)
- net at MUL2. (X): now also MULTIPLIER. (Y15); no longer BL64. (X)
- net at MUL3. (X): now also BL73. (X); no longer MULTIPLIER. (Y15)
- net at MUL4. (X): now also BL74. (X); no longer MULTIPLIER. (Y15)
- net at MUL1. (X): now also BL63. (X); no longer MULTIPLIER. (Y15)
- net at MUL9. (X): now also BL71. (X); no longer MULTIPLIER. (Y15)
- net at MUL15. (X): now also BL69. (X); no longer MULTIPLIER. (Y15)
- net at MUL5. (X): now also BL75. (X); no longer MULTIPLIER. (Y15)
- net at MUL8. (X): now also BL78. (X); no longer MULTIPLIER. (Y15)
- net at MUL12. (X): now also BL66. (X); no longer MULTIPLIER. (Y15)
- net at MUL16. (X): now also BL70. (X); no longer MULTIPLIER. (Y15)
- new net: MUL7. (X), MULTIPLIER. (Y15)
- new net: BL68. (X), MUL14. (X)
- new net: MUL17. (X), MUL27. (/Q7)
- new net: MUL6. (X), MULTIPLIER. (Y15)
- new net: BL72. (X), MUL10. (X)
- new net: BL67. (X), MUL13. (X)
- new net: BL65. (X), MUL11. (X)
- new net: MUL18. (/Q7), MUL28. (X)
- new net: BL64. (X), MUL2. (X)
- new net: MUL3. (X), MULTIPLIER. (Y15)
- new net: MUL4. (X), MULTIPLIER. (Y15)
- new net: MUL27. (/Q7), MULTIPLIER. (Y15) (x8)
- new net: MUL1. (X), MULTIPLIER. (Y15)
- new net: MUL9. (X), MULTIPLIER. (Y15)
- new net: MUL15. (X), MULTIPLIER. (Y15)
- new net: MUL5. (X), MULTIPLIER. (Y15)
- new net: MUL8. (X), MULTIPLIER. (Y15)
- new net: MUL18. (/Q7), MULTIPLIER. (Y15) (x8)
- new net: MUL12. (X), MULTIPLIER. (Y15)

Commit message: - I have fixed all of the problems I was having in the $2006 section, and things are all going places that make sense now.  - I am making good progress on the timer as well.  - I pulled a couple changes back into the letterless SVG and updated the schematic.
Connections:
- net at MUL7. (X): now also BL77. (X); no longer MULTIPLIER. (Y15)
- net at MUL14. (X): now also MULTIPLIER. (Y15); no longer BL68. (X)
- net at MULTIPLIER. (Y15): now also MUL16. (X); no longer MUL14. (X)
- net at MUL6. (X): now also BL76. (X); no longer MULTIPLIER. (Y15)
- net at MUL10. (X): now also MULTIPLIER. (Y15); no longer BL72. (X)
- net at MUL13. (X): now also MULTIPLIER. (Y15); no longer BL67. (X)
- net at MUL11. (X): now also MULTIPLIER. (Y15); no longer BL65. (X)
- net at MUL2. (X): now also MULTIPLIER. (Y15); no longer BL64. (X)
- net at MUL3. (X): now also BL73. (X); no longer MULTIPLIER. (Y15)
- net at MUL4. (X): now also BL74. (X); no longer MULTIPLIER. (Y15)
- net at MUL1. (X): now also BL63. (X); no longer MULTIPLIER. (Y15)
- net at MUL9. (X): now also BL71. (X); no longer MULTIPLIER. (Y15)
- net at MUL15. (X): now also BL69. (X); no longer MULTIPLIER. (Y15)
- net at MUL5. (X): now also BL75. (X); no longer MULTIPLIER. (Y15)
- net at MUL8. (X): now also BL78. (X); no longer MULTIPLIER. (Y15)
- net at MUL12. (X): now also BL66. (X); no longer MULTIPLIER. (Y15)
- net at MUL16. (X): now also BL70. (X); no longer MULTIPLIER. (Y15)
- new net: MUL7. (X), MULTIPLIER. (Y15)
- new net: BL68. (X), MUL14. (X)
- new net: MUL17. (X), MUL27. (/Q7)
- new net: MUL6. (X), MULTIPLIER. (Y15)
- new net: BL72. (X), MUL10. (X)
- new net: BL67. (X), MUL13. (X)
- new net: BL65. (X), MUL11. (X)
- new net: MUL18. (/Q7), MUL28. (X)
- new net: BL64. (X), MUL2. (X)
- new net: MUL3. (X), MULTIPLIER. (Y15)
- new net: MUL4. (X), MULTIPLIER. (Y15)
- new net: MUL27. (/Q7), MULTIPLIER. (Y15) (x8)
- new net: MUL1. (X), MULTIPLIER. (Y15)
- new net: MUL9. (X), MULTIPLIER. (Y15)
- new net: MUL15. (X), MULTIPLIER. (Y15)
- new net: MUL5. (X), MULTIPLIER. (Y15)
- new net: MUL8. (X), MULTIPLIER. (Y15)
- new net: MUL18. (/Q7), MULTIPLIER. (Y15) (x8)
- new net: MUL12. (X), MULTIPLIER. (Y15)

Commit message: I fixed 2 errors in the letterless MMC5 tracing:
1. BK5 is a NAND-4 gate.  It was thought to be NAND-3 before.
2.  BL83 and BL96 signals got swapped here before.  They actually cross each other:

BL83 = "PPU_RW_Mode_%0x_Access"
BL96 = "+ExRAM_Mode_$0x"

This propagated out to several changes in the schematic.
Connections:
- net at MUL7. (X): now also BL77. (X); no longer MULTIPLIER. (Y15)
- net at MUL14. (X): now also MULTIPLIER. (Y15); no longer BL68. (X)
- net at MULTIPLIER. (Y15): now also MUL16. (X); no longer MUL14. (X)
- net at MUL6. (X): now also BL76. (X); no longer MULTIPLIER. (Y15)
- net at MUL10. (X): now also MULTIPLIER. (Y15); no longer BL72. (X)
- net at MUL13. (X): now also MULTIPLIER. (Y15); no longer BL67. (X)
- net at MUL11. (X): now also MULTIPLIER. (Y15); no longer BL65. (X)
- net at MUL2. (X): now also MULTIPLIER. (Y15); no longer BL64. (X)
- net at MUL3. (X): now also BL73. (X); no longer MULTIPLIER. (Y15)
- net at MUL4. (X): now also BL74. (X); no longer MULTIPLIER. (Y15)
- net at MUL1. (X): now also BL63. (X); no longer MULTIPLIER. (Y15)
- net at MUL9. (X): now also BL71. (X); no longer MULTIPLIER. (Y15)
- net at MUL15. (X): now also BL69. (X); no longer MULTIPLIER. (Y15)
- net at MUL5. (X): now also BL75. (X); no longer MULTIPLIER. (Y15)
- net at MUL8. (X): now also BL78. (X); no longer MULTIPLIER. (Y15)
- net at MUL12. (X): now also BL66. (X); no longer MULTIPLIER. (Y15)
- net at MUL16. (X): now also BL70. (X); no longer MULTIPLIER. (Y15)
- new net: MUL7. (X), MULTIPLIER. (Y15)
- new net: BL68. (X), MUL14. (X)
- new net: MUL17. (X), MUL27. (/Q7)
- new net: MUL6. (X), MULTIPLIER. (Y15)
- new net: BL72. (X), MUL10. (X)
- new net: BL67. (X), MUL13. (X)
- new net: BL65. (X), MUL11. (X)
- new net: MUL18. (/Q7), MUL28. (X)
- new net: BL64. (X), MUL2. (X)
- new net: MUL3. (X), MULTIPLIER. (Y15)
- new net: MUL4. (X), MULTIPLIER. (Y15)
- new net: MUL27. (/Q7), MULTIPLIER. (Y15) (x8)
- new net: MUL1. (X), MULTIPLIER. (Y15)
- new net: MUL9. (X), MULTIPLIER. (Y15)
- new net: MUL15. (X), MULTIPLIER. (Y15)
- new net: MUL5. (X), MULTIPLIER. (Y15)
- new net: MUL8. (X), MULTIPLIER. (Y15)
- new net: MUL18. (/Q7), MULTIPLIER. (Y15) (x8)
- new net: MUL12. (X), MULTIPLIER. (Y15)

Commit message: Schematic and SVG Updates
Connections:
- net at MUL7. (X): now also BL77. (X); no longer MULTIPLIER. (Y15)
- net at MUL14. (X): now also MULTIPLIER. (Y15); no longer BL68. (X)
- net at MULTIPLIER. (Y15): now also MUL16. (X); no longer MUL14. (X)
- net at MUL6. (X): now also BL76. (X); no longer MULTIPLIER. (Y15)
- net at MUL10. (X): now also MULTIPLIER. (Y15); no longer BL72. (X)
- net at MUL13. (X): now also MULTIPLIER. (Y15); no longer BL67. (X)
- net at MUL11. (X): now also MULTIPLIER. (Y15); no longer BL65. (X)
- net at MUL2. (X): now also MULTIPLIER. (Y15); no longer BL64. (X)
- net at MUL3. (X): now also BL73. (X); no longer MULTIPLIER. (Y15)
- net at MUL4. (X): now also BL74. (X); no longer MULTIPLIER. (Y15)
- net at MUL1. (X): now also BL63. (X); no longer MULTIPLIER. (Y15)
- net at MUL9. (X): now also BL71. (X); no longer MULTIPLIER. (Y15)
- net at MUL15. (X): now also BL69. (X); no longer MULTIPLIER. (Y15)
- net at MUL5. (X): now also BL75. (X); no longer MULTIPLIER. (Y15)
- net at MUL8. (X): now also BL78. (X); no longer MULTIPLIER. (Y15)
- net at MUL12. (X): now also BL66. (X); no longer MULTIPLIER. (Y15)
- net at MUL16. (X): now also BL70. (X); no longer MULTIPLIER. (Y15)
- new net: MUL7. (X), MULTIPLIER. (Y15)
- new net: BL68. (X), MUL14. (X)
- new net: MUL17. (X), MUL27. (/Q7)
- new net: MUL6. (X), MULTIPLIER. (Y15)
- new net: BL72. (X), MUL10. (X)
- new net: BL67. (X), MUL13. (X)
- new net: BL65. (X), MUL11. (X)
- new net: MUL18. (/Q7), MUL28. (X)
- new net: BL64. (X), MUL2. (X)
- new net: MUL3. (X), MULTIPLIER. (Y15)
- new net: MUL4. (X), MULTIPLIER. (Y15)
- new net: MUL27. (/Q7), MULTIPLIER. (Y15) (x8)
- new net: MUL1. (X), MULTIPLIER. (Y15)
- new net: MUL9. (X), MULTIPLIER. (Y15)
- new net: MUL15. (X), MULTIPLIER. (Y15)
- new net: MUL5. (X), MULTIPLIER. (Y15)
- new net: MUL8. (X), MULTIPLIER. (Y15)
- new net: MUL18. (/Q7), MULTIPLIER. (Y15) (x8)
- new net: MUL12. (X), MULTIPLIER. (Y15)

Commit message: Schematic and SVG Updates
Connections:
- net at MUL7. (X): now also BL77. (X); no longer MULTIPLIER. (Y15)
- net at MUL14. (X): now also MULTIPLIER. (Y15); no longer BL68. (X)
- net at MULTIPLIER. (Y15): now also MUL16. (X); no longer MUL14. (X)
- net at MUL6. (X): now also BL76. (X); no longer MULTIPLIER. (Y15)
- net at MUL10. (X): now also MULTIPLIER. (Y15); no longer BL72. (X)
- net at MUL13. (X): now also MULTIPLIER. (Y15); no longer BL67. (X)
- net at MUL11. (X): now also MULTIPLIER. (Y15); no longer BL65. (X)
- net at MUL2. (X): now also MULTIPLIER. (Y15); no longer BL64. (X)
- net at MUL3. (X): now also BL73. (X); no longer MULTIPLIER. (Y15)
- net at MUL4. (X): now also BL74. (X); no longer MULTIPLIER. (Y15)
- net at MUL1. (X): now also BL63. (X); no longer MULTIPLIER. (Y15)
- net at MUL9. (X): now also BL71. (X); no longer MULTIPLIER. (Y15)
- net at MUL15. (X): now also BL69. (X); no longer MULTIPLIER. (Y15)
- net at MUL5. (X): now also BL75. (X); no longer MULTIPLIER. (Y15)
- net at MUL8. (X): now also BL78. (X); no longer MULTIPLIER. (Y15)
- net at MUL12. (X): now also BL66. (X); no longer MULTIPLIER. (Y15)
- net at MUL16. (X): now also BL70. (X); no longer MULTIPLIER. (Y15)
- new net: MUL7. (X), MULTIPLIER. (Y15)
- new net: BL68. (X), MUL14. (X)
- new net: MUL17. (X), MUL27. (/Q7)
- new net: MUL6. (X), MULTIPLIER. (Y15)
- new net: BL72. (X), MUL10. (X)
- new net: BL67. (X), MUL13. (X)
- new net: BL65. (X), MUL11. (X)
- new net: MUL18. (/Q7), MUL28. (X)
- new net: BL64. (X), MUL2. (X)
- new net: MUL3. (X), MULTIPLIER. (Y15)
- new net: MUL4. (X), MULTIPLIER. (Y15)
- new net: MUL27. (/Q7), MULTIPLIER. (Y15) (x8)
- new net: MUL1. (X), MULTIPLIER. (Y15)
- new net: MUL9. (X), MULTIPLIER. (Y15)
- new net: MUL15. (X), MULTIPLIER. (Y15)
- new net: MUL5. (X), MULTIPLIER. (Y15)
- new net: MUL8. (X), MULTIPLIER. (Y15)
- new net: MUL18. (/Q7), MULTIPLIER. (Y15) (x8)
- new net: MUL12. (X), MULTIPLIER. (Y15)

Commit message: Tracing and schematic updates.  - Added timer to schematic.  - Added all items from artifacts sheet to the MMC5A trace.
Connections:
- net at MUL7. (X): now also BL77. (X); no longer MULTIPLIER. (Y15)
- net at MUL14. (X): now also MULTIPLIER. (Y15); no longer BL68. (X)
- net at MULTIPLIER. (Y15): now also MUL16. (X); no longer MUL14. (X)
- net at MUL6. (X): now also BL76. (X); no longer MULTIPLIER. (Y15)
- net at MUL10. (X): now also MULTIPLIER. (Y15); no longer BL72. (X)
- net at MUL13. (X): now also MULTIPLIER. (Y15); no longer BL67. (X)
- net at MUL11. (X): now also MULTIPLIER. (Y15); no longer BL65. (X)
- net at MUL2. (X): now also MULTIPLIER. (Y15); no longer BL64. (X)
- net at MUL3. (X): now also BL73. (X); no longer MULTIPLIER. (Y15)
- net at MUL4. (X): now also BL74. (X); no longer MULTIPLIER. (Y15)
- net at MUL1. (X): now also BL63. (X); no longer MULTIPLIER. (Y15)
- net at MUL9. (X): now also BL71. (X); no longer MULTIPLIER. (Y15)
- net at MUL15. (X): now also BL69. (X); no longer MULTIPLIER. (Y15)
- net at MUL5. (X): now also BL75. (X); no longer MULTIPLIER. (Y15)
- net at MUL8. (X): now also BL78. (X); no longer MULTIPLIER. (Y15)
- net at MUL12. (X): now also BL66. (X); no longer MULTIPLIER. (Y15)
- net at MUL16. (X): now also BL70. (X); no longer MULTIPLIER. (Y15)
- new net: MUL7. (X), MULTIPLIER. (Y15)
- new net: BL68. (X), MUL14. (X)
- new net: MUL17. (X), MUL27. (/Q7)
- new net: MUL6. (X), MULTIPLIER. (Y15)
- new net: BL72. (X), MUL10. (X)
- new net: BL67. (X), MUL13. (X)
- new net: BL65. (X), MUL11. (X)
- new net: MUL18. (/Q7), MUL28. (X)
- new net: BL64. (X), MUL2. (X)
- new net: MUL3. (X), MULTIPLIER. (Y15)
- new net: MUL4. (X), MULTIPLIER. (Y15)
- new net: MUL27. (/Q7), MULTIPLIER. (Y15) (x8)
- new net: MUL1. (X), MULTIPLIER. (Y15)
- new net: MUL9. (X), MULTIPLIER. (Y15)
- new net: MUL15. (X), MULTIPLIER. (Y15)
- new net: MUL5. (X), MULTIPLIER. (Y15)
- new net: MUL8. (X), MULTIPLIER. (Y15)
- new net: MUL18. (/Q7), MULTIPLIER. (Y15) (x8)
- new net: MUL12. (X), MULTIPLIER. (Y15)

Commit message: Added the new MMC5A read-register bits in the schematic. Additional MMC5A tracing work.
Connections:
- net at MUL7. (X): now also BL77. (X); no longer MULTIPLIER. (Y15)
- net at MUL14. (X): now also MULTIPLIER. (Y15); no longer BL68. (X)
- net at MULTIPLIER. (Y15): now also MUL16. (X); no longer MUL14. (X)
- net at MUL6. (X): now also BL76. (X); no longer MULTIPLIER. (Y15)
- net at MUL10. (X): now also MULTIPLIER. (Y15); no longer BL72. (X)
- net at MUL13. (X): now also MULTIPLIER. (Y15); no longer BL67. (X)
- net at MUL11. (X): now also MULTIPLIER. (Y15); no longer BL65. (X)
- net at MUL2. (X): now also MULTIPLIER. (Y15); no longer BL64. (X)
- net at MUL3. (X): now also BL73. (X); no longer MULTIPLIER. (Y15)
- net at MUL4. (X): now also BL74. (X); no longer MULTIPLIER. (Y15)
- net at MUL1. (X): now also BL63. (X); no longer MULTIPLIER. (Y15)
- net at MUL9. (X): now also BL71. (X); no longer MULTIPLIER. (Y15)
- net at MUL15. (X): now also BL69. (X); no longer MULTIPLIER. (Y15)
- net at MUL5. (X): now also BL75. (X); no longer MULTIPLIER. (Y15)
- net at MUL8. (X): now also BL78. (X); no longer MULTIPLIER. (Y15)
- net at MUL12. (X): now also BL66. (X); no longer MULTIPLIER. (Y15)
- net at MUL16. (X): now also BL70. (X); no longer MULTIPLIER. (Y15)
- new net: MUL7. (X), MULTIPLIER. (Y15)
- new net: BL68. (X), MUL14. (X)
- new net: MUL17. (X), MUL27. (/Q7)
- new net: MUL6. (X), MULTIPLIER. (Y15)
- new net: BL72. (X), MUL10. (X)
- new net: BL67. (X), MUL13. (X)
- new net: BL65. (X), MUL11. (X)
- new net: MUL18. (/Q7), MUL28. (X)
- new net: BL64. (X), MUL2. (X)
- new net: MUL3. (X), MULTIPLIER. (Y15)
- new net: MUL4. (X), MULTIPLIER. (Y15)
- new net: MUL27. (/Q7), MULTIPLIER. (Y15) (x8)
- new net: MUL1. (X), MULTIPLIER. (Y15)
- new net: MUL9. (X), MULTIPLIER. (Y15)
- new net: MUL15. (X), MULTIPLIER. (Y15)
- new net: MUL5. (X), MULTIPLIER. (Y15)
- new net: MUL8. (X), MULTIPLIER. (Y15)
- new net: MUL18. (/Q7), MULTIPLIER. (Y15) (x8)
- new net: MUL12. (X), MULTIPLIER. (Y15)
