File: Schematic (KiCAD)/multiplier.kicad_sch (KiCad schematic)
At the start: 37 parts

Commit message: - Fixed the register read bit schematic errors noted by Joe in the Nesdev forum.
Connections:
- net at MUL7. (X): now also BL77. (X); no longer MULTIPLIER. (Y15)
- net at MUL14. (X): now also MULTIPLIER. (Y15); no longer BL68. (X)
- net at MULTIPLIER. (Y15): now also MUL16. (X); no longer MUL14. (X)
- net at MUL6. (X): now also BL76. (X); no longer MULTIPLIER. (Y15)
- net at MUL10. (X): now also MULTIPLIER. (Y15); no longer BL72. (X)
- net at MUL13. (X): now also MULTIPLIER. (Y15); no longer BL67. (X)
- net at MUL11. (X): now also MULTIPLIER. (Y15); no longer BL65. (X)
- net at MUL2. (X): now also MULTIPLIER. (Y15); no longer BL64. (X)
- net at MUL3. (X): now also BL73. (X); no longer MULTIPLIER. (Y15)
- net at MUL4. (X): now also BL74. (X); no longer MULTIPLIER. (Y15)
- net at MUL1. (X): now also BL63. (X); no longer MULTIPLIER. (Y15)
- net at MUL9. (X): now also BL71. (X); no longer MULTIPLIER. (Y15)
- net at MUL15. (X): now also BL69. (X); no longer MULTIPLIER. (Y15)
- net at MUL5. (X): now also BL75. (X); no longer MULTIPLIER. (Y15)
- net at MUL8. (X): now also BL78. (X); no longer MULTIPLIER. (Y15)
- net at MUL12. (X): now also BL66. (X); no longer MULTIPLIER. (Y15)
- net at MUL16. (X): now also BL70. (X); no longer MULTIPLIER. (Y15)
- new net: MUL7. (X), MULTIPLIER. (Y15)
- new net: BL68. (X), MUL14. (X)
- new net: MUL17. (X), MUL27. (/Q7)
- new net: MUL6. (X), MULTIPLIER. (Y15)
- new net: BL72. (X), MUL10. (X)
- new net: BL67. (X), MUL13. (X)
- new net: BL65. (X), MUL11. (X)
- new net: MUL18. (/Q7), MUL28. (X)
- new net: BL64. (X), MUL2. (X)
- new net: MUL3. (X), MULTIPLIER. (Y15)
- new net: MUL4. (X), MULTIPLIER. (Y15)
- new net: MUL27. (/Q7), MULTIPLIER. (Y15) (x8)
- new net: MUL1. (X), MULTIPLIER. (Y15)
- new net: MUL9. (X), MULTIPLIER. (Y15)
- new net: MUL15. (X), MULTIPLIER. (Y15)
- new net: MUL5. (X), MULTIPLIER. (Y15)
- new net: MUL8. (X), MULTIPLIER. (Y15)
- new net: MUL18. (/Q7), MULTIPLIER. (Y15) (x8)
- new net: MUL12. (X), MULTIPLIER. (Y15)

Commit message: - Updated all of the various And-OR-Invert gates to have consistent names.  - Added the schematic for CL3 / SL3 GPIO pins.  There are no surprises revealed by this.  - Finished up the CPU address decoding tracing.  - Added one of the 'artifact' counters from the pulse channels
Connections:
- net at MUL7. (X): now also BL77. (X); no longer MULTIPLIER. (Y15)
- net at MUL14. (X): now also MULTIPLIER. (Y15); no longer BL68. (X)
- net at MULTIPLIER. (Y15): now also MUL16. (X); no longer MUL14. (X)
- net at MUL6. (X): now also BL76. (X); no longer MULTIPLIER. (Y15)
- net at MUL10. (X): now also MULTIPLIER. (Y15); no longer BL72. (X)
- net at MUL13. (X): now also MULTIPLIER. (Y15); no longer BL67. (X)
- net at MUL11. (X): now also MULTIPLIER. (Y15); no longer BL65. (X)
- net at MUL2. (X): now also MULTIPLIER. (Y15); no longer BL64. (X)
- net at MUL3. (X): now also BL73. (X); no longer MULTIPLIER. (Y15)
- net at MUL4. (X): now also BL74. (X); no longer MULTIPLIER. (Y15)
- net at MUL1. (X): now also BL63. (X); no longer MULTIPLIER. (Y15)
- net at MUL9. (X): now also BL71. (X); no longer MULTIPLIER. (Y15)
- net at MUL15. (X): now also BL69. (X); no longer MULTIPLIER. (Y15)
- net at MUL5. (X): now also BL75. (X); no longer MULTIPLIER. (Y15)
- net at MUL8. (X): now also BL78. (X); no longer MULTIPLIER. (Y15)
- net at MUL12. (X): now also BL66. (X); no longer MULTIPLIER. (Y15)
- net at MUL16. (X): now also BL70. (X); no longer MULTIPLIER. (Y15)
- new net: MUL7. (X), MULTIPLIER. (Y15)
- new net: BL68. (X), MUL14. (X)
- new net: MUL17. (X), MUL27. (/Q7)
- new net: MUL6. (X), MULTIPLIER. (Y15)
- new net: BL72. (X), MUL10. (X)
- new net: BL67. (X), MUL13. (X)
- new net: BL65. (X), MUL11. (X)
- new net: MUL18. (/Q7), MUL28. (X)
- new net: BL64. (X), MUL2. (X)
- new net: MUL3. (X), MULTIPLIER. (Y15)
- new net: MUL4. (X), MULTIPLIER. (Y15)
- new net: MUL27. (/Q7), MULTIPLIER. (Y15) (x8)
- new net: MUL1. (X), MULTIPLIER. (Y15)
- new net: MUL9. (X), MULTIPLIER. (Y15)
- new net: MUL15. (X), MULTIPLIER. (Y15)
- new net: MUL5. (X), MULTIPLIER. (Y15)
- new net: MUL8. (X), MULTIPLIER. (Y15)
- new net: MUL18. (/Q7), MULTIPLIER. (Y15) (x8)
- new net: MUL12. (X), MULTIPLIER. (Y15)
Changed lines of the file:
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@@
 	)
 	(symbol
-		(lib_name "BUFFER_8")
+		(lib_name "BUFFER_12")
 		(lib_id "MMC5:BUFFER")
 		(at 201.93 124.46 0)
@@
 	)
 	(symbol
-		(lib_name "BUFFER_13")
+		(lib_name "BUFFER_15")
 		(lib_id "MMC5:BUFFER")
 		(at 201.93 78.74 0)
@@
 	)
 	(symbol
+		(lib_name "BUFFER_1")
 		(lib_id "MMC5:BUFFER")
 		(at 72.39 107.95 0)
@@
 	)
 	(symbol
-		(lib_name "BUFFER_9")
+		(lib_name "BUFFER_7")
 		(lib_id "MMC5:BUFFER")
 		(at 201.93 130.81 0)
@@
 	)
 	(symbol
-		(lib_name "BUFFER_27")
+		(lib_name "BUFFER_33")
 		(lib_id "MMC5:BUFFER")
 		(at 210.82 104.14 0)
@@
 	)
 	(symbol
-		(lib_name "BUFFER_23")
+		(lib_name "BUFFER_29")
 		(lib_id "MMC5:BUFFER")
 		(at 210.82 78.74 0)
@@
 	)
 	(symbol
-		(lib_name "BUFFER_22")
+		(lib_name "BUFFER_31")
 		(lib_id "MMC5:BUFFER")
 		(at 210.82 85.09 0)
@@
 	)
 	(symbol
-		(lib_name "BUFFER_20")
+		(lib_name "BUFFER_25")
 		(lib_id "MMC5:BUFFER")
 		(at 210.82 97.79 0)
@@
 	)
 	(symbol
-		(lib_name "BUFFER_1")
 		(lib_id "MMC5:BUFFER")
 		(at 72.39 166.37 0)
@@
 	)
 	(symbol
-		(lib_name "BUFFER_19")
+		(lib_name "BUFFER_22")
 		(lib_id "MMC5:BUFFER")
 		(at 210.82 156.21 0)
@@
 	)
 	(symbol
-		(lib_name "BUFFER_4")
+		(lib_name "BUFFER_10")
 		(lib_id "MMC5:BUFFER")
 		(at 201.93 149.86 0)
@@
 	)
 	(symbol
-		(lib_name "BUFFER_5")
+		(lib_name "BUFFER_11")
 		(lib_id "MMC5:BUFFER")
 		(at 201.93 143.51 0)
@@
 	)
 	(symbol
-		(lib_name "BUFFER_14")
+		(lib_name "BUFFER_4")
 		(lib_id "MMC5:BUFFER")
 		(at 201.93 97.79 0)
@@
 	)
 	(symbol
-		(lib_name "BUFFER_26")
+		(lib_name "BUFFER_24")
 		(lib_id "MMC5:BUFFER")
 		(at 210.82 110.49 0)
@@
 	)
 	(symbol
+		(lib_name "Reg_8_D-Latch_N_1")
 		(lib_id "MMC5:Reg_8_D-Latch_N")
 		(at 87.63 64.77 0)
@@
 	)
 	(symbol
-		(lib_name "BUFFER_2")
+		(lib_name "BUFFER_3")
 		(lib_id "MMC5:BUFFER")
 		(at 201.93 162.56 0)
@@
 	)
 	(symbol
-		(lib_name "BUFFER_32")
+		(lib_name "BUFFER_27")
 		(lib_id "MMC5:BUFFER")
 		(at 210.82 124.46 0)
@@
 	)
 	(symbol
-		(lib_name "BUFFER_11")
+		(lib_name "BUFFER_13")
 		(lib_id "MMC5:BUFFER")
 		(at 201.93 110.49 0)
@@
 	)
 	(symbol
-		(lib_name "BUFFER_28")
+		(lib_name "BUFFER_23")
 		(lib_id "MMC5:BUFFER")
 		(at 210.82 149.86 0)
@@
 	)
 	(symbol
-		(lib_name "BUFFER_30")
+		(lib_name "BUFFER_20")
 		(lib_id "MMC5:BUFFER")
 		(at 210.82 137.16 0)
@@
 	)
 	(symbol
-		(lib_name "BUFFER_25")
+		(lib_name "BUFFER_21")
 		(lib_id "MMC5:BUFFER")
 		(at 210.82 66.04 0)
@@
 	)
 	(symbol
-		(lib_name "BUFFER_10")
+		(lib_name "BUFFER_9")
 		(lib_id "MMC5:BUFFER")
 		(at 201.93 72.39 0)
@@
 	)
 	(symbol
-		(lib_name "BUFFER_31")
+		(lib_name "BUFFER_32")
 		(lib_id "MMC5:BUFFER")
 		(at 210.82 130.81 0)
@@
 	)
 	(symbol
-		(lib_name "BUFFER_12")
+		(lib_name "BUFFER_8")
 		(lib_id "MMC5:BUFFER")
 		(at 201.93 85.09 0)
@@
 	)
 	(symbol
-		(lib_name "BUFFER_24")
+		(lib_name "BUFFER_18")
 		(lib_id "MMC5:BUFFER")
 		(at 210.82 72.39 0)
@@
 	)
 	(symbol
-		(lib_name "BUFFER_33")
+		(lib_name "BUFFER_28")
 		(lib_id "MMC5:BUFFER")
 		(at 210.82 118.11 0)
@@
 	)
 	(symbol
-		(lib_name "BUFFER_21")
+		(lib_name "BUFFER_30")
 		(lib_id "MMC5:BUFFER")
 		(at 210.82 91.44 0)
@@
 	)
 	(symbol
-		(lib_name "BUFFER_3")
+		(lib_name "BUFFER_14")
 		(lib_id "MMC5:BUFFER")
 		(at 201.93 156.21 0)
@@
 	)
 	(symbol
-		(lib_name "BUFFER_18")
+		(lib_name "BUFFER_19")
 		(lib_id "MMC5:BUFFER")
 		(at 210.82 162.56 0)
@@
 	)
 	(symbol
-		(lib_name "BUFFER_29")
+		(lib_name "BUFFER_26")
 		(lib_id "MMC5:BUFFER")
 		(at 210.82 143.51 0)
@@
 	)
 	(symbol
-		(lib_name "BUFFER_7")
+		(lib_name "BUFFER_5")
 		(lib_id "MMC5:BUFFER")
 		(at 201.93 137.16 0)
@@
 	)
 	(symbol
-		(lib_name "Reg_8_D-Latch_N_1")
 		(lib_id "MMC5:Reg_8_D-Latch_N")
 		(at 87.63 123.19 0)
@@
 	)
 	(symbol
-		(lib_name "BUFFER_15")
+		(lib_name "BUFFER_2")
 		(lib_id "MMC5:BUFFER")
 		(at 201.93 91.44 0)
