File: Schematic (KiCAD)/MMC5.kicad_sch (KiCad schematic)
At the start: 6 parts, among them K115 NAND_2, K115 NAND_3, K116 INVERT

Commit message: - Updated all of the various And-OR-Invert gates to have consistent names.  - Added the schematic for CL3 / SL3 GPIO pins.  There are no surprises revealed by this.  - Finished up the CPU address decoding tracing.  - Added one of the 'artifact' counters from the pulse channels
Connections:
- new net: K115. (X), K115. (X), K116. (X)
Other:
- added sheet MMC5A CL3 SL3 GPIO (mmc5a_cl3_sl3_gpio.kicad_sch)
