File: Schematic (KiCAD)/chr_a0_a1_a2.kicad_sch (KiCad schematic)
At the start: 60 parts, among them J72 NAND_4, J73 NOR_2, J74 NAND_2, P10 NAND_2, P11 NAND_2, P12,13,18,19,25,26 Reg 3 DFF-Reset, P14 INVERT, P15 T-FF Preload, P16 NAND_2, P17 NAND_2, P20 INVERT, P21 T-FF Preload, P22 BUFFER, P23 NAND_2, P24 NAND_2, P27 INVERT, P28 BUFFER, P8 INVERT, P9 T-FF Preload

Commit message: - Updated all of the various And-OR-Invert gates to have consistent names.  - Added the schematic for CL3 / SL3 GPIO pins.  There are no surprises revealed by this.  - Finished up the CPU address decoding tracing.  - Added one of the 'artifact' counters from the pulse channels
Parts:
- DISCH15: value AOI_2 -> AOI_22
Connections:
- net at R27. (/Q): now also R26. (X)
- net at R26. (X): now also R29. (X); no longer R27. (/Q)
- net at R15. (X): now also R16. (X); no longer R3. (X)
- net at P28. (X): now also R26. (X); no longer P12,13,18,19,25,26. (Q2)
- net at N7. (X): now also N8. (X); no longer N6. (X)
- net at BL44. (X): now also BL43. (X); no longer BL47. (X)
- net at DISCH12. (X): now also DISCH13. (X); no longer DISCH1,2,3. (Q1)
- net at DISCH14. (X): now also DISCH11. (X); no longer DISCH13. (X)
- new net: DISCH11. (X), DISCH14. (X), DISCH4. (X), DISCH5. (X), DISCH7. (X), DISCH9. (X)
- new net: DISCH5. (X), DISCH6. (X)
- new net: R27. (/Q), R28. (X)
- new net: R27. (/Q), R29. (X)
- new net: DISCH7. (X), DISCH8. (X)
- new net: R15. (X), R16. (X), R17,18,19,20,21,22,23. (/Q2)
- new net: R15. (X), R3. (X)
- new net: P10. (X), P11. (X), P9. (/Q)
- new net: P27. (X), R25. (X)
- new net: P12,13,18,19,25,26. (Q2), P28. (X)
- new net: P12,13,18,19,25,26. (Q2), P17. (X)
- new net: P11. (X), P12,13,18,19,25,26. (Q2)
- new net: P12,13,18,19,25,26. (Q2), P24. (X)
- new net: P14. (X), P15. (/Q), P9. (/Q)
- new net: P8. (X), P9. (/Q)
- new net: P21. (/Q), P22. (X)
- new net: DISCH10. (X), DISCH9. (X)
- new net: N11,12,13. (/Q1), N14. (X)
- new net: N10. (X), N11,12,13. (/Q1), N8. (X)
- new net: N6. (X), N7. (X)
- new net: P15. (/Q), P16. (X), P17. (X)
- new net: DISCH15. (X), DISCH16. (X), DISCH17. (X)
- new net: DISCH15. (X), DISCH4. (X)
- new net: P21. (/Q), P23. (X), P24. (X)
- new net: BL44. (X), BL47. (X)
- new net: N26. (X), N28. (X)
- new net: P15. (/Q), P20. (X), P21. (/Q)
- new net: N18,19,20,21,24,25,27,29,32,34,36,37. (Y3), N23. (X)
- new net: N17. (X), N18,19,20,21,24,25,27,29,32,34,36,37. (Y3)
- new net: N18,19,20,21,24,25,27,29,32,34,36,37. (Y3), N30. (X)
- new net: DISCH1,2,3. (Q1), DISCH12. (X)
- new net: DISCH13. (X), DISCH14. (X)
Changed lines of the file:
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@@
 	)
 	(symbol
-		(lib_name "NAND_2_11")
+		(lib_name "NAND_2_20")
 		(lib_id "MMC5:NAND_2")
 		(at 307.34 104.14 0)
@@
 	)
 	(symbol
-		(lib_name "BUFFER_2")
+		(lib_name "BUFFER_3")
 		(lib_id "MMC5:BUFFER")
 		(at 231.14 198.12 0)
@@
 	)
 	(symbol
-		(lib_name "NAND_2_12")
+		(lib_name "NAND_2_18")
 		(lib_id "MMC5:NAND_2")
 		(at 307.34 95.25 0)
@@
 	)
 	(symbol
-		(lib_name "NAND_2_4")
+		(lib_name "NAND_2_5")
 		(lib_id "MMC5:NAND_2")
 		(at 72.39 93.98 0)
@@
 	)
 	(symbol
-		(lib_name "NAND_2_32")
+		(lib_name "NAND_2_10")
 		(lib_id "MMC5:NAND_2")
 		(at 312.42 193.04 0)
@@
 	)
 	(symbol
-		(lib_name "INVERT_3")
+		(lib_name "INVERT_10")
 		(lib_id "MMC5:INVERT")
 		(at 146.05 87.63 0)
@@
 	)
 	(symbol
-		(lib_name "T-FF_Preload_8")
+		(lib_name "T-FF_Preload_2")
 		(lib_id "MMC5:T-FF_Preload")
 		(at 356.87 187.96 0)
@@
 	)
 	(symbol
-		(lib_name "BUFFER_3")
+		(lib_name "BUFFER_2")
 		(lib_id "MMC5:BUFFER")
 		(at 345.44 153.67 0)
@@
 	)
 	(symbol
-		(lib_name "INVERT_15")
+		(lib_name "INVERT_17")
 		(lib_id "MMC5:INVERT")
 		(at 318.77 86.36 0)
@@
 	)
 	(symbol
-		(lib_name "NAND_2_30")
+		(lib_name "NAND_2_12")
 		(lib_id "MMC5:NAND_2")
 		(at 312.42 179.07 0)
@@
 	)
 	(symbol
+		(lib_name "BUFFER_1")
 		(lib_id "MMC5:BUFFER")
 		(at 271.78 184.15 0)
@@
 			)
 		)
-		(property "Value" "AOI_2"
+		(property "Value" "AOI_22"
 			(at 285.242 61.722 0)
 			(do_not_autoplace yes)
@@
 	)
 	(symbol
-		(lib_name "NAND_2_33")
+		(lib_name "NAND_2_7")
 		(lib_id "MMC5:NAND_2")
 		(at 300.99 173.99 0)
@@
 	)
 	(symbol
-		(lib_name "NAND_2_35")
+		(lib_name "NAND_2_14")
 		(lib_id "MMC5:NAND_2")
 		(at 312.42 165.1 0)
@@
 	)
 	(symbol
-		(lib_name "BUFFER_13")
 		(lib_id "MMC5:BUFFER")
 		(at 139.7 48.26 0)
@@
 	)
 	(symbol
-		(lib_name "NAND_2_34")
+		(lib_name "NAND_2_9")
 		(lib_id "MMC5:NAND_2")
 		(at 300.99 187.96 0)
@@
 	)
 	(symbol
-		(lib_name "NAND_2_13")
+		(lib_name "NAND_2_19")
 		(lib_id "MMC5:NAND_2")
 		(at 307.34 86.36 0)
@@
 	)
 	(symbol
-		(lib_name "NAND_2_2")
+		(lib_name "NAND_2_3")
 		(lib_id "MMC5:NAND_2")
 		(at 134.62 87.63 0)
@@
 	)
 	(symbol
-		(lib_name "INVERT_14")
+		(lib_name "INVERT_16")
 		(lib_id "MMC5:INVERT")
 		(at 318.77 95.25 0)
@@
 	)
 	(symbol
-		(lib_name "T-FF_Preload_10")
 		(lib_id "MMC5:T-FF_Preload")
 		(at 356.87 173.99 0)
@@
 	)
 	(symbol
-		(lib_name "INVERT_2")
+		(lib_name "INVERT_1")
 		(lib_id "MMC5:INVERT")
 		(at 193.04 138.43 0)
@@
 	)
 	(symbol
-		(lib_name "NAND_2_5")
 		(lib_id "MMC5:NAND_2")
 		(at 60.96 92.71 0)
@@
 	)
 	(symbol
-		(lib_name "INVERT_5")
+		(lib_name "INVERT_3")
 		(lib_id "MMC5:INVERT")
 		(at 135.89 72.39 0)
@@
 	)
 	(symbol
-		(lib_name "INVERT_6")
+		(lib_name "INVERT_8")
 		(lib_id "MMC5:INVERT")
 		(at 158.75 48.26 0)
@@
 	)
 	(symbol
-		(lib_name "INVERT_9")
+		(lib_name "INVERT_15")
 		(lib_id "MMC5:INVERT")
 		(at 269.24 60.96 0)
@@
 	)
 	(symbol
-		(lib_name "INVERT_10")
+		(lib_name "INVERT_7")
 		(lib_id "MMC5:INVERT")
 		(at 149.86 48.26 0)
@@
 	)
 	(symbol
-		(lib_name "INVERT_13")
+		(lib_name "INVERT_18")
 		(lib_id "MMC5:INVERT")
 		(at 318.77 104.14 0)
@@
 	)
 	(symbol
-		(lib_name "INVERT_1")
+		(lib_name "INVERT_2")
 		(lib_id "MMC5:INVERT")
 		(at 193.04 147.32 0)
@@
 	)
 	(symbol
+		(lib_name "INVERT_6")
 		(lib_id "MMC5:INVERT")
 		(at 193.04 129.54 0)
@@
 	)
 	(symbol
-		(lib_name "INVERT_31")
+		(lib_name "INVERT_14")
 		(lib_id "MMC5:INVERT")
 		(at 368.3 175.26 0)
@@
 	)
 	(symbol
-		(lib_name "T-FF_Preload_9")
+		(lib_name "T-FF_Preload_1")
 		(lib_id "MMC5:T-FF_Preload")
 		(at 356.87 160.02 0)
@@
 	)
 	(symbol
-		(lib_name "NAND_2_7")
+		(lib_name "NAND_2_13")
 		(lib_id "MMC5:NAND_2")
 		(at 344.17 52.07 0)
@@
 	)
 	(symbol
-		(lib_name "INVERT_11")
+		(lib_name "INVERT_9")
 		(lib_id "MMC5:INVERT")
 		(at 132.08 53.34 0)
@@
 	)
 	(symbol
-		(lib_name "INVERT_7")
+		(lib_name "INVERT_13")
 		(lib_id "MMC5:INVERT")
 		(at 344.17 63.5 0)
@@
 	)
 	(symbol
+		(lib_name "NAND_2_2")
 		(lib_id "MMC5:NAND_2")
 		(at 156.21 66.04 0)
@@
 	)
 	(symbol
-		(lib_name "NAND_2_3")
+		(lib_name "NAND_2_4")
 		(lib_id "MMC5:NAND_2")
 		(at 83.82 92.71 0)
@@
 	)
 	(symbol
-		(lib_name "NAND_2_29")
+		(lib_name "NAND_2_8")
 		(lib_id "MMC5:NAND_2")
 		(at 261.62 184.15 0)
@@
 	)
 	(symbol
-		(lib_name "INVERT_30")
+		(lib_name "INVERT_12")
 		(lib_id "MMC5:INVERT")
 		(at 368.3 161.29 0)
@@
 	)
 	(symbol
-		(lib_name "NAND_2_8")
+		(lib_name "NAND_2_15")
 		(lib_id "MMC5:NAND_2")
 		(at 332.74 63.5 0)
@@
 	)
 	(symbol
-		(lib_name "NAND_2_10")
+		(lib_name "NAND_2_17")
 		(lib_id "MMC5:NAND_2")
 		(at 294.64 81.28 0)
@@
 	)
 	(symbol
-		(lib_name "INVERT_32")
+		(lib_name "INVERT_11")
 		(lib_id "MMC5:INVERT")
 		(at 368.3 189.23 0)
@@
 	)
 	(symbol
-		(lib_name "INVERT_12")
 		(lib_id "MMC5:INVERT")
 		(at 123.19 53.34 0)
@@
 	)
 	(symbol
-		(lib_name "INVERT_4")
+		(lib_name "INVERT_5")
 		(lib_id "MMC5:INVERT")
 		(at 144.78 72.39 0)
@@
 	)
 	(symbol
-		(lib_name "NAND_2_9")
+		(lib_name "NAND_2_16")
 		(lib_id "MMC5:NAND_2")
 		(at 321.31 69.85 0)
@@
 	)
 	(symbol
-		(lib_name "NAND_2_37")
+		(lib_name "NAND_2_11")
 		(lib_id "MMC5:NAND_2")
 		(at 300.99 160.02 0)
@@
 	)
 	(symbol
-		(lib_name "INVERT_8")
+		(lib_name "INVERT_4")
 		(lib_id "MMC5:INVERT")
 		(at 102.87 44.45 0)
