File: Schematic (KiCAD)/exram_mode.kicad_sch (KiCad schematic)
At the start: 94 parts

Commit message: - Updated all of the various And-OR-Invert gates to have consistent names.  - Added the schematic for CL3 / SL3 GPIO pins.  There are no surprises revealed by this.  - Finished up the CPU address decoding tracing.  - Added one of the 'artifact' counters from the pulse channels
Parts:
- BK89: value OAI_2 -> OAI_21
Connections:
- net at BL100. (X): now also BL101. (X); no longer BL99. (/Q)
- net at BL90. (X): now also BL91. (X); no longer BL89. (/Q)
- net at BL93. (X): now also BL92. (X); no longer BN2. (X)
- net at BJ10. (X): now also BJ11. (/Q7); no longer BJ9. (X)
- net at BL88. (X): now also BL86. (X); no longer BL84. (X)
- net at BL92. (X): now also BL94. (X); no longer BL93. (X)
- net at BM9. (X): now also BM10. (X); no longer BM8. (X)
- net at BM10. (X): now also BL91. (X); no longer BM9. (X)
- net at BL84. (X): now also BL85. (X); no longer BL87. (X)
- net at BL103. (X): now also BJ39b. (X); no longer BL95. (X)
- net at BL85. (X): now also BL86. (X); no longer BL82. (X)
- net at BM3. (X): now also BM4. (X); no longer BM2. (X)
- net at BM4. (X): now also BM5. (X); no longer BM3. (X)
- net at BL106. (X): now also BL109. (/Q); no longer BL105. (X)
- new net: BL81. (X), BL87. (X)
- new net: BJ40. (Q9), BK78. (Q7), BK89. (X)
- new net: BK84. (X), BL102. (X), BL105. (X), BL107. (X), BN3. (X), BN4. (X)
- new net: BK83. (X), BK84. (X)
- new net: BK84. (X), BK86. (X)
- new net: BL108. (X), BL99. (/Q)
- new net: BL100. (X), BL99. (/Q)
- new net: BL93. (X), BL94. (X), BL98. (/Q)
- new net: BJ40. (Q9), BJ43. (X)
- new net: BK91. (X), BK93. (X)
- new net: BK77. (Q7), BK90. (X)
- new net: BK77. (Q7), BK78. (Q7) (x8)
- new net: BK79. (X), BK81. (X), BK82. (Q1)
- new net: BL89. (/Q), BL90. (X)
- new net: BK92. (X), BK93. (X)
- new net: BL93. (X), BN2. (X)
- new net: BJ7. (X), BJ9. (X)
- new net: BJ10. (X), BJ9. (X)
- new net: BJ32. (X), BJ33. (X), BJ34. (X), BJ35. (X), BJ36. (X), BJ37. (X), BJ38. (X), BJ39. (X), BJ39b. (X) (x2)
- new net: BL84. (X), BL88. (X)
- new net: BL88. (X), BM5. (X), BM6. (X)
- new net: BM8. (X), BM9. (X)
- new net: BK79. (X), BK82. (Q1), BL96. (X)
- new net: BL84. (X), BL87. (X)
- new net: BL104. (X), BL95. (X)
- new net: BL103. (X), BL95. (X)
- new net: BL82. (X), BL85. (X)
- new net: BL83. (X), BL84. (X)
- new net: BJ51. (X), BK96. (X)
- new net: BM2. (X), BM3. (X)
- new net: BK80. (X), BK82. (Q1)
- new net: BL105. (X), BL106. (X)
- new net: BL91. (X), BL92. (X)
- new net: BJ40. (Q9), BJ50. (X)
- new net: BJ40. (Q9), BJ46. (X)
- new net: BJ40. (Q9), BJ42. (X)
- new net: BJ40. (Q9), BJ44. (X)
- new net: BJ40. (Q9), BJ49. (X)
- new net: BJ40. (Q9), BJ45. (X)
- new net: BJ40. (Q9), BJ48. (X)
- new net: BJ40. (Q9), BJ47. (X)
- new net: BJ40. (Q9), BJ41. (X)
- new net: BK94. (X), BK95. (X)
Changed lines of the file:
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@@
 	)
 	(symbol
-		(lib_name "BIGBUF_2")
+		(lib_name "BIGBUF_1")
 		(lib_id "MMC5:BIGBUF")
 		(at 138.43 102.87 0)
@@
 	)
 	(symbol
-		(lib_name "OAI_2_2")
 		(lib_id "MMC5:OAI_2")
 		(at 237.49 151.13 0)
@@
 			)
 		)
-		(property "Value" "OAI_2"
+		(property "Value" "OAI_21"
 			(at 237.49 155.702 0)
 			(do_not_autoplace yes)
@@
 	)
 	(symbol
-		(lib_name "NAND_3_3")
 		(lib_id "MMC5:NAND_3")
 		(at 133.35 142.24 0)
@@
 	)
 	(symbol
-		(lib_name "D-FF_Reset_1")
 		(lib_id "MMC5:D-FF_Reset")
 		(at 105.41 167.64 0)
@@
 	)
 	(symbol
-		(lib_name "BUFFER_24")
+		(lib_name "BUFFER_3")
 		(lib_id "MMC5:BUFFER")
 		(at 48.26 224.79 0)
@@
 	)
 	(symbol
+		(lib_name "D-FF_Reset_1")
 		(lib_id "MMC5:D-FF_Reset")
 		(at 57.15 83.82 0)
@@
 	)
 	(symbol
-		(lib_name "NAND_2_9")
+		(lib_name "NAND_2_2")
 		(lib_id "MMC5:NAND_2")
 		(at 121.92 170.18 0)
@@
 	)
 	(symbol
-		(lib_name "BUFFER_10")
 		(lib_id "MMC5:BUFFER")
 		(at 109.22 43.18 0)
@@
 	)
 	(symbol
-		(lib_name "NAND_Mux_3_6")
+		(lib_name "NAND_Mux_3_2")
 		(lib_id "MMC5:NAND_Mux_3")
 		(at 314.96 121.92 0)
@@
 	)
 	(symbol
-		(lib_name "INVERT_9")
+		(lib_name "INVERT_3")
 		(lib_id "MMC5:INVERT")
 		(at 297.18 34.29 0)
@@
 	)
 	(symbol
-		(lib_name "BUFFER_23")
+		(lib_name "BUFFER_4")
 		(lib_id "MMC5:BUFFER")
 		(at 48.26 219.71 0)
@@
 	)
 	(symbol
-		(lib_name "NAND_2_2")
 		(lib_id "MMC5:NAND_2")
 		(at 97.79 50.8 0)
@@
 	)
 	(symbol
-		(lib_name "INVERT_1")
 		(lib_id "MMC5:INVERT")
 		(at 85.09 68.58 0)
@@
 	)
 	(symbol
-		(lib_name "BIGBUF_3")
+		(lib_name "BIGBUF_2")
 		(lib_id "MMC5:BIGBUF")
 		(at 58.42 96.52 0)
@@
 	)
 	(symbol
-		(lib_name "NAND_3_12")
+		(lib_name "NAND_3_2")
 		(lib_id "MMC5:NAND_3")
 		(at 59.69 252.73 0)
@@
 	)
 	(symbol
-		(lib_name "NAND_3_4")
+		(lib_name "NAND_3_1")
 		(lib_id "MMC5:NAND_3")
 		(at 121.92 142.24 0)
@@
 	)
 	(symbol
+		(lib_name "NAND_Mux_2_1")
 		(lib_id "MMC5:NAND_Mux_2")
 		(at 273.05 205.74 0)
@@
 	)
 	(symbol
-		(lib_name "NAND_2_6")
+		(lib_name "NAND_2_3")
 		(lib_id "MMC5:NAND_2")
 		(at 149.86 83.82 0)
@@
 	)
 	(symbol
-		(lib_name "BUFFER_9")
+		(lib_name "BUFFER_5")
 		(lib_id "MMC5:BUFFER")
 		(at 113.03 71.12 0)
@@
 	)
 	(symbol
-		(lib_name "INVERT_27")
+		(lib_name "INVERT_1")
 		(lib_id "MMC5:INVERT")
 		(at 50.8 257.81 0)
@@
 	)
 	(symbol
-		(lib_name "NOR_2_1")
 		(lib_id "MMC5:NOR_2")
 		(at 93.98 166.37 0)
@@
 	)
 	(symbol
-		(lib_name "BUFFER_25")
+		(lib_name "BUFFER_1")
 		(lib_id "MMC5:BUFFER")
 		(at 48.26 240.03 0)
@@
 	)
 	(symbol
-		(lib_name "BUFFER_26")
+		(lib_name "BUFFER_2")
 		(lib_id "MMC5:BUFFER")
 		(at 48.26 229.87 0)
@@
 	)
 	(symbol
-		(lib_name "BUFFER_22")
+		(lib_name "BUFFER_7")
 		(lib_id "MMC5:BUFFER")
 		(at 48.26 214.63 0)
@@
 	)
 	(symbol
-		(lib_name "BUFFER_30")
+		(lib_name "BUFFER_10")
 		(lib_id "MMC5:BUFFER")
 		(at 69.85 252.73 0)
@@
 	)
 	(symbol
-		(lib_name "BUFFER_8")
+		(lib_name "BUFFER_6")
 		(lib_id "MMC5:BUFFER")
 		(at 121.92 71.12 0)
@@
 	)
 	(symbol
+		(lib_name "INVERT_2")
 		(lib_id "MMC5:INVERT")
 		(at 86.36 52.07 0)
@@
 	)
 	(symbol
+		(lib_name "NOR_2_1")
 		(lib_id "MMC5:NOR_2")
 		(at 123.19 93.98 0)
@@
 	)
 	(symbol
-		(lib_name "NAND_3_1")
+		(lib_name "NAND_3_3")
 		(lib_id "MMC5:NAND_3")
 		(at 163.83 91.44 0)
@@
 	)
 	(symbol
-		(lib_name "NAND_2_11")
+		(lib_name "NAND_2_5")
 		(lib_id "MMC5:NAND_2")
 		(at 66.04 179.07 0)
@@
 	)
 	(symbol
-		(lib_name "NAND_Mux_2_1")
 		(lib_id "MMC5:NAND_Mux_2")
 		(at 273.05 213.36 0)
@@
 	)
 	(symbol
-		(lib_name "NAND_2_13")
+		(lib_name "NAND_2_12")
 		(lib_id "MMC5:NAND_2")
 		(at 285.75 44.45 0)
@@
 	)
 	(symbol
-		(lib_name "BUFFER_3")
+		(lib_name "BUFFER_9")
 		(lib_id "MMC5:BUFFER")
 		(at 166.37 71.12 0)
@@
 	)
 	(symbol
-		(lib_name "BUFFER_7")
+		(lib_name "BUFFER_8")
 		(lib_id "MMC5:BUFFER")
 		(at 130.81 71.12 0)
@@
 	)
 	(symbol
-		(lib_name "INVERT_5")
+		(lib_name "INVERT_7")
 		(lib_id "MMC5:INVERT")
 		(at 66.04 157.48 0)
@@
 	)
 	(symbol
+		(lib_name "NAND_3_5")
 		(lib_id "MMC5:NAND_3")
 		(at 93.98 71.12 0)
@@
 	)
 	(symbol
-		(lib_name "BUFFER_6")
+		(lib_name "BUFFER_17")
 		(lib_id "MMC5:BUFFER")
 		(at 139.7 71.12 0)
@@
 	)
 	(symbol
-		(lib_name "BIGBUF_1")
+		(lib_name "BIGBUF_3")
 		(lib_id "MMC5:BIGBUF")
 		(at 40.64 153.67 0)
@@
 	)
 	(symbol
+		(lib_name "NAND_Mux_3_4")
 		(lib_id "MMC5:NAND_Mux_3")
 		(at 314.96 50.8 0)
@@
 	)
 	(symbol
-		(lib_name "BUFFER_5")
+		(lib_name "BUFFER_14")
 		(lib_id "MMC5:BUFFER")
 		(at 148.59 71.12 0)
@@
 	)
 	(symbol
-		(lib_name "NAND_2_5")
+		(lib_name "NAND_2_10")
 		(lib_id "MMC5:NAND_2")
 		(at 71.12 81.28 0)
@@
 	)
 	(symbol
-		(lib_name "NAND_Mux_3_4")
+		(lib_name "NAND_Mux_3_7")
 		(lib_id "MMC5:NAND_Mux_3")
 		(at 314.96 91.44 0)
@@
 	)
 	(symbol
-		(lib_name "BUFFER_2")
+		(lib_name "BUFFER_15")
 		(lib_id "MMC5:BUFFER")
 		(at 175.26 71.12 0)
@@
 	)
 	(symbol
-		(lib_name "NAND_Mux_2_7")
+		(lib_name "NAND_Mux_2_6")
 		(lib_id "MMC5:NAND_Mux_2")
 		(at 273.05 259.08 0)
@@
 	)
 	(symbol
-		(lib_name "NAND_Mux_3_7")
+		(lib_name "NAND_Mux_3_3")
 		(lib_id "MMC5:NAND_Mux_3")
 		(at 314.96 111.76 0)
@@
 	)
 	(symbol
-		(lib_name "NAND_Mux_2_6")
+		(lib_name "NAND_Mux_2_7")
 		(lib_id "MMC5:NAND_Mux_2")
 		(at 273.05 251.46 0)
@@
 	)
 	(symbol
-		(lib_name "BUFFER_27")
+		(lib_name "BUFFER_20")
 		(lib_id "MMC5:BUFFER")
 		(at 48.26 234.95 0)
@@
 	)
 	(symbol
-		(lib_name "NAND_2_12")
+		(lib_name "NAND_2_13")
 		(lib_id "MMC5:NAND_2")
 		(at 237.49 182.88 0)
@@
 	)
 	(symbol
-		(lib_name "INVERT_4")
+		(lib_name "INVERT_5")
 		(lib_id "MMC5:INVERT")
 		(at 109.22 35.56 0)
@@
 	)
 	(symbol
-		(lib_name "NAND_3_5")
+		(lib_name "NAND_3_7")
 		(lib_id "MMC5:NAND_3")
 		(at 285.75 34.29 0)
@@
 	)
 	(symbol
-		(lib_name "INVERT_8")
+		(lib_name "INVERT_10")
 		(lib_id "MMC5:INVERT")
 		(at 224.79 203.2 0)
@@
 	)
 	(symbol
-		(lib_name "INVERT_3")
+		(lib_name "INVERT_6")
 		(lib_id "MMC5:INVERT")
 		(at 175.26 91.44 0)
@@
 	)
 	(symbol
-		(lib_name "NAND_Mux_3_1")
 		(lib_id "MMC5:NAND_Mux_3")
 		(at 314.96 60.96 0)
@@
 	)
 	(symbol
+		(lib_name "BUFFER_16")
 		(lib_id "MMC5:BUFFER")
 		(at 104.14 71.12 0)
@@
 	)
 	(symbol
-		(lib_name "NAND_2_3")
+		(lib_name "NAND_2_6")
 		(lib_id "MMC5:NAND_2")
 		(at 82.55 85.09 0)
@@
 	)
 	(symbol
+		(lib_name "NAND_2_9")
 		(lib_id "MMC5:NAND_2")
 		(at 97.79 43.18 0)
@@
 	)
 	(symbol
-		(lib_name "NAND_Mux_3_5")
+		(lib_name "NAND_Mux_3_6")
 		(lib_id "MMC5:NAND_Mux_3")
 		(at 314.96 101.6 0)
@@
 	)
 	(symbol
-		(lib_name "BUFFER_1")
+		(lib_name "BUFFER_19")
 		(lib_id "MMC5:BUFFER")
 		(at 184.15 71.12 0)
@@
 	)
 	(symbol
-		(lib_name "NAND_Mux_3_3")
+		(lib_name "NAND_Mux_3_5")
 		(lib_id "MMC5:NAND_Mux_3")
 		(at 314.96 71.12 0)
@@
 	)
 	(symbol
-		(lib_name "INVERT_6")
+		(lib_name "INVERT_4")
 		(lib_id "MMC5:INVERT")
 		(at 93.98 173.99 0)
@@
 	)
 	(symbol
-		(lib_name "INVERT_10")
+		(lib_name "INVERT_8")
 		(lib_id "MMC5:INVERT")
 		(at 297.18 21.59 0)
@@
 	)
 	(symbol
-		(lib_name "BUFFER_4")
+		(lib_name "BUFFER_18")
 		(lib_id "MMC5:BUFFER")
 		(at 157.48 71.12 0)
@@
 	)
 	(symbol
-		(lib_name "NAND_2_10")
+		(lib_name "NAND_2_8")
 		(lib_id "MMC5:NAND_2")
 		(at 82.55 173.99 0)
@@
 	)
 	(symbol
-		(lib_name "BUFFER_21")
+		(lib_name "BUFFER_13")
 		(lib_id "MMC5:BUFFER")
 		(at 48.26 209.55 0)
@@
 	)
 	(symbol
-		(lib_name "NAND_Mux_3_2")
+		(lib_name "NAND_Mux_3_1")
 		(lib_id "MMC5:NAND_Mux_3")
 		(at 314.96 81.28 0)
@@
 	)
 	(symbol
-		(lib_name "NAND_2_8")
+		(lib_name "NAND_2_11")
 		(lib_id "MMC5:NAND_2")
 		(at 121.92 123.19 0)
@@
 	)
 	(symbol
-		(lib_name "BUFFER_28")
+		(lib_name "BUFFER_12")
 		(lib_id "MMC5:BUFFER")
 		(at 48.26 245.11 0)
@@
 	)
 	(symbol
-		(lib_name "NAND_3_2")
+		(lib_name "NAND_3_4")
 		(lib_id "MMC5:NAND_3")
 		(at 121.92 132.08 0)
@@
 	)
 	(symbol
-		(lib_name "INVERT_7")
+		(lib_name "INVERT_9")
 		(lib_id "MMC5:INVERT")
 		(at 245.11 199.39 0)
