File: Schematic (KiCAD)/fill_mode.kicad_sch (KiCad schematic)
At the start: 12 parts

Commit message: - Updated all of the various And-OR-Invert gates to have consistent names.  - Added the schematic for CL3 / SL3 GPIO pins.  There are no surprises revealed by this.  - Finished up the CPU address decoding tracing.  - Added one of the 'artifact' counters from the pulse channels
Connections:
- new net: L10. (/Q7), L15. (X)
- new net: L10. (/Q7), L14. (X)
- new net: L10. (/Q7), L16. (X)
- new net: L10. (/Q7), L13. (X)
- new net: L10. (/Q7), L18. (X)
- new net: L10. (/Q7), L17. (X)
- new net: L10. (/Q7), L11. (X)
- new net: L10. (/Q7), L12. (X)
