File: Schematic (KiCAD)/mmc5a_timer.kicad_sch (KiCad schematic)
At the start: 204 parts

Commit message: Added the new MMC5A read-register bits in the schematic. Additional MMC5A tracing work.
Connections:
- net at TE41. (X): now also TE20. (X), TE40. (X)
- net at TC23. (X): now also TC12. (X), TC13. (X); no longer TC24. (X)
- net at TD25. (X): now also TD30. (/Q); no longer TD24. (X)
- net at TD30. (/Q): now also TD27. (X); no longer TD25. (X)
- net at TB35. (X): now also TB36. (X); no longer TB32. (/Q)
- net at TB36. (X): now also TB41. (/Q); no longer TB35. (X)
- net at TB10. (/Q): now also TB9. (X); no longer TB11. (X)
- net at TB13. (X): now also TB14. (X); no longer TB10. (/Q)
- net at TB5. (X): now also TB4. (X); no longer TB10. (/Q)
- net at TB9. (X): now also TB8. (X); no longer TB10. (/Q)
- net at TD7. (X): now also TD8. (/Q); no longer TD6. (X)
- net at TD19. (X): now also TD18. (X), TD20. (X)
- net at TC32. (X): now also TC33. (/Q); no longer TC31. (X)
- net at TE11. (X): now also TE8. (/Q); no longer TE12. (X)
- net at TE8. (/Q): now also TE9. (X); no longer TE11. (X)
- net at TE32. (X): now also TE20. (X), TE31. (X)
- net at TD31. (X): now also TD20. (X), TD32. (X); no longer TD30. (/Q)
- net at TE29. (X): now also TE30. (/Q); no longer TE28. (X)
- net at TB31. (X): now also TB32. (/Q); no longer TB30. (X)
- net at TD22. (X): now also TC1. (X), TD21. (X)
- net at TE30. (/Q): now also TE25. (X); no longer TE29. (X)
- net at TE33. (X): now also TE34. (X); no longer TE30. (/Q)
- net at TE34. (X): now also TE39. (/Q); no longer TE33. (X)
- net at TC6. (X): now also TC11. (/Q); no longer TC5. (X)
- net at TC11. (/Q): now also TC12. (X); no longer TC6. (X)
- net at TA29. (X): now also TA7. (X); no longer TA30. (X)
- net at TB27. (X): now also TB26. (X); no longer TB32. (/Q)
- net at TB26. (X): now also TB19. (/Q); no longer TB27. (X)
- net at TB23. (X): now also TB24. (X); no longer TB22. (X)
- net at TB24. (X): no longer TB23. (X)
- net at TC33. (/Q): now also TC28. (X); no longer TC32. (X)
- net at TC14. (X): now also TC11. (/Q); no longer TC15. (X)
- net at TD10. (X): now also TD20. (X), TD9. (X)
- net at TD39. (/Q): now also TD34. (X); no longer TD36. (X)
- net at TD29. (X): now also TD28. (X); no longer TD30. (/Q)
- net at TD33. (X): now also TD34. (X); no longer TD30. (/Q)
- net at TB20. (X): now also TB21. (X), TB22. (X); no longer TB19. (/Q)
- net at TE38. (X): now also TE37. (X); no longer TE39. (/Q)
- net at TC20. (/Q): now also TC19. (X); no longer TC27. (X)
- net at TC19. (X): now also TC18. (X); no longer TC20. (/Q)
- net at TB19. (/Q): now also TB16. (X); no longer TB14. (X)
- net at TB18. (X): now also TB17. (X); no longer TB19. (/Q)
- net at TB40. (X): now also TB39. (X); no longer TB41. (/Q)
- net at TE39. (/Q): now also TE40. (X)
- net at TC36. (X): now also TC37. (X); no longer TC33. (/Q)
- net at TC28. (X): now also TC27. (X); no longer TC33. (/Q)
- net at TE17. (/Q): now also TE12. (X); no longer TE16. (X)
- net at TE24. (X): now also TE25. (X); no longer TE17. (/Q)
- net at TC37. (X): now also TC42. (/Q); no longer TC36. (X)
- net at TC10. (X): now also TC9. (X); no longer TC11. (/Q)
- net at TB32. (/Q): now also TB29. (X); no longer TB31. (X)
- net at TA28. (X): now also TA27. (X); no longer TA16. (/Q)
- net at TE7. (X): now also TE6. (X); no longer TE8. (/Q)
- net at TD12. (X): now also TD11. (X); no longer TD17. (/Q)
- net at TD11. (X): now also TD8. (/Q); no longer TD12. (X)
- net at TD17. (/Q): now also TD16. (X); no longer TD14. (X)
- net at TD16. (X): now also TD15. (X); no longer TD17. (/Q)
- net at TA27. (X): now also TD42. (X); no longer TA28. (X)
- net at TB33. (X): now also TB22. (X), TB34. (X); no longer TB32. (/Q)
- net at TA10. (X), TA9. (X): now also TB1. (X)
- net at TE3. (X): now also TE2. (X); no longer TE8. (/Q)
- net at TD38. (X): now also TD37. (X); no longer TD39. (/Q)
- net at TC41. (X): now also TC42. (/Q); no longer TC40. (X)
- net at TC42. (/Q): no longer TC41. (X)
- new net: TC23. (X), TC34. (X), TC35. (X)
- new net: TC23. (X), TC24. (X)
- new net: TC23. (X), TC43. (X), TC44. (X)
- new net: TC21. (X), TC22. (X), TC23. (X)
- new net: TB6. (X), TB7. (X), TB8. (X)
- new net: TD24. (X), TD25. (X)
- new net: TB32. (/Q), TB35. (X)
- new net: TA16. (/Q), TA18. (X), TA19. (X)
- new net: TA17. (X), TA18. (X)
- new net: TB10. (/Q), TB11. (X)
- new net: TB10. (/Q), TB13. (X)
- new net: TB10. (/Q), TB5. (X)
- new net: TB10. (/Q), TB7. (X)
- new net: TA11. (X), TA12. (/Q)
- new net: TA11. (X), TF9. (X)
- new net: TD4. (X), TD5. (X), TD6. (X)
- new net: TD6. (X), TD7. (X)
- new net: TB22. (X), TB42. (X), TB43. (X)
- new net: TC38. (X), TC39. (X), TC42. (/Q)
- new net: TC31. (X), TC32. (X)
- new net: TC30. (X), TC31. (X)
- new net: TC2. (X), TC24. (X), TC25. (X)
- new net: TE11. (X), TE12. (X)
- new net: TD30. (/Q), TD31. (X)
- new net: TE21. (X), TE22. (X), TE42. (X)
- new net: TA23. (X), TA6. (X), TA7. (X)
- new net: TA23. (X), TE43. (X)
- new net: TA23. (X), TA29. (X), TE43. (X)
- new net: TE28. (X), TE29. (X)
- new net: TE27. (X), TE28. (X)
- new net: TB30. (X), TB31. (X)
- new net: TB28. (X), TB29. (X), TB30. (X)
- new net: TD2. (X), TD22. (X), TD23. (X)
- new net: TE26. (X), TE27. (X), TE30. (/Q)
- new net: TE30. (/Q), TE33. (X)
- new net: TC5. (X), TC6. (X)
- new net: TC16. (X), TC17. (X), TC20. (/Q)
- new net: TC17. (X), TC18. (X)
- new net: TE2. (X), TE22. (X), TE23. (X)
- new net: TE18. (X), TE19. (X), TE20. (X)
- new net: TE4. (X), TE5. (X), TE8. (/Q)
- new net: TA29. (X), TA30. (X)
- new net: TB27. (X), TB32. (/Q)
- new net: TB22. (X), TB23. (X)
- new net: TC14. (X), TC15. (X)
- new net: TA16. (/Q), TA21. (X), TA27. (X)
- new net: TD36. (X), TD39. (/Q)
- new net: TD35. (X), TD36. (X), TD37. (X)
- new net: TD29. (X), TD30. (/Q)
- new net: TD30. (/Q), TD33. (X)
- new net: TB19. (/Q), TB20. (X)
- new net: TE38. (X), TE39. (/Q)
- new net: TB11. (X), TB12. (X), TB22. (X)
- new net: TC11. (/Q), TC7. (X), TC8. (X)
- new net: TC8. (X), TC9. (X)
- new net: TB24. (X), TB25. (X), TB4. (X)
- new net: TC25. (X), TC26. (X), TC5. (X)
- new net: TC20. (/Q), TC27. (X)
- new net: TB14. (X), TB19. (/Q)
- new net: TB18. (X), TB19. (/Q)
- new net: TB40. (X), TB41. (/Q)
- new net: TB37. (X), TB38. (X), TB39. (X)
- new net: TB38. (X), TB41. (/Q)
- new net: TA3. (X), TA4. (X)
- new net: TE35. (X), TE36. (X), TE39. (/Q)
- new net: TC33. (/Q), TC36. (X)
- new net: TC29. (X), TC30. (X), TC33. (/Q)
- new net: TE16. (X), TE17. (/Q)
- new net: TE13. (X), TE14. (X), TE17. (/Q)
- new net: TE17. (/Q), TE24. (X)
- new net: TB15. (X), TB16. (X), TB17. (X)
- new net: TC10. (X), TC11. (/Q)
- new net: TA2. (/Q), TA3. (X)
- new net: TE14. (X), TE15. (X)
- new net: TA16. (/Q), TA28. (X)
- new net: TA15. (X), TA16. (/Q)
- new net: TC39. (X), TC40. (X)
- new net: TD26. (X), TD27. (X), TD28. (X)
- new net: TA5. (/Q), TA6. (X)
- new net: TE7. (X), TE8. (/Q)
- new net: TD12. (X), TD17. (/Q)
- new net: TD5. (X), TD8. (/Q)
- new net: TD14. (X), TD17. (/Q)
- new net: TD13. (X), TD14. (X), TD15. (X)
- new net: TB32. (/Q), TB33. (X)
- new net: TE10. (X), TE20. (X), TE9. (X)
- new net: TA10. (X), TA9. (X)
- new net: TE36. (X), TE37. (X)
- new net: TD42. (X), TD43. (X)
- new net: TD20. (X), TD40. (X), TD41. (X)
- new net: TE3. (X), TE8. (/Q)
- new net: TD38. (X), TD39. (/Q)
- new net: TC40. (X), TC41. (X)
- new net: TE5. (X), TE6. (X)
- now unconnected: TB24. (X), TC13. (X), TC22. (X), TC25. (X), TC25. (X), TC35. (X), TC42. (/Q), TC42. (/Q), TD32. (X), TE10. (X), TE19. (X), TE22. (X), TE22. (X)

Commit message: - Fixed the register read bit schematic errors noted by Joe in the Nesdev forum.
Connections:
- net at TE41. (X): now also TE20. (X), TE40. (X)
- net at TC23. (X): now also TC12. (X), TC13. (X); no longer TC24. (X)
- net at TD25. (X): now also TD30. (/Q); no longer TD24. (X)
- net at TD30. (/Q): now also TD27. (X); no longer TD25. (X)
- net at TB35. (X): now also TB36. (X); no longer TB32. (/Q)
- net at TB36. (X): now also TB41. (/Q); no longer TB35. (X)
- net at TB10. (/Q): now also TB9. (X); no longer TB11. (X)
- net at TB13. (X): now also TB14. (X); no longer TB10. (/Q)
- net at TB5. (X): now also TB4. (X); no longer TB10. (/Q)
- net at TB9. (X): now also TB8. (X); no longer TB10. (/Q)
- net at TD7. (X): now also TD8. (/Q); no longer TD6. (X)
- net at TD19. (X): now also TD18. (X), TD20. (X)
- net at TC32. (X): now also TC33. (/Q); no longer TC31. (X)
- net at TE11. (X): now also TE8. (/Q); no longer TE12. (X)
- net at TE8. (/Q): now also TE9. (X); no longer TE11. (X)
- net at TE32. (X): now also TE20. (X), TE31. (X)
- net at TD31. (X): now also TD20. (X), TD32. (X); no longer TD30. (/Q)
- net at TE29. (X): now also TE30. (/Q); no longer TE28. (X)
- net at TB31. (X): now also TB32. (/Q); no longer TB30. (X)
- net at TD22. (X): now also TC1. (X), TD21. (X)
- net at TE30. (/Q): now also TE25. (X); no longer TE29. (X)
- net at TE33. (X): now also TE34. (X); no longer TE30. (/Q)
- net at TE34. (X): now also TE39. (/Q); no longer TE33. (X)
- net at TC6. (X): now also TC11. (/Q); no longer TC5. (X)
- net at TC11. (/Q): now also TC12. (X); no longer TC6. (X)
- net at TA29. (X): now also TA7. (X); no longer TA30. (X)
- net at TB27. (X): now also TB26. (X); no longer TB32. (/Q)
- net at TB26. (X): now also TB19. (/Q); no longer TB27. (X)
- net at TB23. (X): now also TB24. (X); no longer TB22. (X)
- net at TB24. (X): no longer TB23. (X)
- net at TC33. (/Q): now also TC28. (X); no longer TC32. (X)
- net at TC14. (X): now also TC11. (/Q); no longer TC15. (X)
- net at TD10. (X): now also TD20. (X), TD9. (X)
- net at TD39. (/Q): now also TD34. (X); no longer TD36. (X)
- net at TD29. (X): now also TD28. (X); no longer TD30. (/Q)
- net at TD33. (X): now also TD34. (X); no longer TD30. (/Q)
- net at TB20. (X): now also TB21. (X), TB22. (X); no longer TB19. (/Q)
- net at TE38. (X): now also TE37. (X); no longer TE39. (/Q)
- net at TC20. (/Q): now also TC19. (X); no longer TC27. (X)
- net at TC19. (X): now also TC18. (X); no longer TC20. (/Q)
- net at TB19. (/Q): now also TB16. (X); no longer TB14. (X)
- net at TB18. (X): now also TB17. (X); no longer TB19. (/Q)
- net at TB40. (X): now also TB39. (X); no longer TB41. (/Q)
- net at TE39. (/Q): now also TE40. (X)
- net at TC36. (X): now also TC37. (X); no longer TC33. (/Q)
- net at TC28. (X): now also TC27. (X); no longer TC33. (/Q)
- net at TE17. (/Q): now also TE12. (X); no longer TE16. (X)
- net at TE24. (X): now also TE25. (X); no longer TE17. (/Q)
- net at TC37. (X): now also TC42. (/Q); no longer TC36. (X)
- net at TC10. (X): now also TC9. (X); no longer TC11. (/Q)
- net at TB32. (/Q): now also TB29. (X); no longer TB31. (X)
- net at TA28. (X): now also TA27. (X); no longer TA16. (/Q)
- net at TE7. (X): now also TE6. (X); no longer TE8. (/Q)
- net at TD12. (X): now also TD11. (X); no longer TD17. (/Q)
- net at TD11. (X): now also TD8. (/Q); no longer TD12. (X)
- net at TD17. (/Q): now also TD16. (X); no longer TD14. (X)
- net at TD16. (X): now also TD15. (X); no longer TD17. (/Q)
- net at TA27. (X): now also TD42. (X); no longer TA28. (X)
- net at TB33. (X): now also TB22. (X), TB34. (X); no longer TB32. (/Q)
- net at TA10. (X), TA9. (X): now also TB1. (X)
- net at TE3. (X): now also TE2. (X); no longer TE8. (/Q)
- net at TD38. (X): now also TD37. (X); no longer TD39. (/Q)
- net at TC41. (X): now also TC42. (/Q); no longer TC40. (X)
- net at TC42. (/Q): no longer TC41. (X)
- new net: TC23. (X), TC34. (X), TC35. (X)
- new net: TC23. (X), TC24. (X)
- new net: TC23. (X), TC43. (X), TC44. (X)
- new net: TC21. (X), TC22. (X), TC23. (X)
- new net: TB6. (X), TB7. (X), TB8. (X)
- new net: TD24. (X), TD25. (X)
- new net: TB32. (/Q), TB35. (X)
- new net: TA16. (/Q), TA18. (X), TA19. (X)
- new net: TA17. (X), TA18. (X)
- new net: TB10. (/Q), TB11. (X)
- new net: TB10. (/Q), TB13. (X)
- new net: TB10. (/Q), TB5. (X)
- new net: TB10. (/Q), TB7. (X)
- new net: TA11. (X), TA12. (/Q)
- new net: TA11. (X), TF9. (X)
- new net: TD4. (X), TD5. (X), TD6. (X)
- new net: TD6. (X), TD7. (X)
- new net: TB22. (X), TB42. (X), TB43. (X)
- new net: TC38. (X), TC39. (X), TC42. (/Q)
- new net: TC31. (X), TC32. (X)
- new net: TC30. (X), TC31. (X)
- new net: TC2. (X), TC24. (X), TC25. (X)
- new net: TE11. (X), TE12. (X)
- new net: TD30. (/Q), TD31. (X)
- new net: TE21. (X), TE22. (X), TE42. (X)
- new net: TA23. (X), TA6. (X), TA7. (X)
- new net: TA23. (X), TE43. (X)
- new net: TA23. (X), TA29. (X), TE43. (X)
- new net: TE28. (X), TE29. (X)
- new net: TE27. (X), TE28. (X)
- new net: TB30. (X), TB31. (X)
- new net: TB28. (X), TB29. (X), TB30. (X)
- new net: TD2. (X), TD22. (X), TD23. (X)
- new net: TE26. (X), TE27. (X), TE30. (/Q)
- new net: TE30. (/Q), TE33. (X)
- new net: TC5. (X), TC6. (X)
- new net: TC16. (X), TC17. (X), TC20. (/Q)
- new net: TC17. (X), TC18. (X)
- new net: TE2. (X), TE22. (X), TE23. (X)
- new net: TE18. (X), TE19. (X), TE20. (X)
- new net: TE4. (X), TE5. (X), TE8. (/Q)
- new net: TA29. (X), TA30. (X)
- new net: TB27. (X), TB32. (/Q)
- new net: TB22. (X), TB23. (X)
- new net: TC14. (X), TC15. (X)
- new net: TA16. (/Q), TA21. (X), TA27. (X)
- new net: TD36. (X), TD39. (/Q)
- new net: TD35. (X), TD36. (X), TD37. (X)
- new net: TD29. (X), TD30. (/Q)
- new net: TD30. (/Q), TD33. (X)
- new net: TB19. (/Q), TB20. (X)
- new net: TE38. (X), TE39. (/Q)
- new net: TB11. (X), TB12. (X), TB22. (X)
- new net: TC11. (/Q), TC7. (X), TC8. (X)
- new net: TC8. (X), TC9. (X)
- new net: TB24. (X), TB25. (X), TB4. (X)
- new net: TC25. (X), TC26. (X), TC5. (X)
- new net: TC20. (/Q), TC27. (X)
- new net: TB14. (X), TB19. (/Q)
- new net: TB18. (X), TB19. (/Q)
- new net: TB40. (X), TB41. (/Q)
- new net: TB37. (X), TB38. (X), TB39. (X)
- new net: TB38. (X), TB41. (/Q)
- new net: TA3. (X), TA4. (X)
- new net: TE35. (X), TE36. (X), TE39. (/Q)
- new net: TC33. (/Q), TC36. (X)
- new net: TC29. (X), TC30. (X), TC33. (/Q)
- new net: TE16. (X), TE17. (/Q)
- new net: TE13. (X), TE14. (X), TE17. (/Q)
- new net: TE17. (/Q), TE24. (X)
- new net: TB15. (X), TB16. (X), TB17. (X)
- new net: TC10. (X), TC11. (/Q)
- new net: TA2. (/Q), TA3. (X)
- new net: TE14. (X), TE15. (X)
- new net: TA16. (/Q), TA28. (X)
- new net: TA15. (X), TA16. (/Q)
- new net: TC39. (X), TC40. (X)
- new net: TD26. (X), TD27. (X), TD28. (X)
- new net: TA5. (/Q), TA6. (X)
- new net: TE7. (X), TE8. (/Q)
- new net: TD12. (X), TD17. (/Q)
- new net: TD5. (X), TD8. (/Q)
- new net: TD14. (X), TD17. (/Q)
- new net: TD13. (X), TD14. (X), TD15. (X)
- new net: TB32. (/Q), TB33. (X)
- new net: TE10. (X), TE20. (X), TE9. (X)
- new net: TA10. (X), TA9. (X)
- new net: TE36. (X), TE37. (X)
- new net: TD42. (X), TD43. (X)
- new net: TD20. (X), TD40. (X), TD41. (X)
- new net: TE3. (X), TE8. (/Q)
- new net: TD38. (X), TD39. (/Q)
- new net: TC40. (X), TC41. (X)
- new net: TE5. (X), TE6. (X)
- now unconnected: TB24. (X), TC13. (X), TC22. (X), TC25. (X), TC25. (X), TC35. (X), TC42. (/Q), TC42. (/Q), TD32. (X), TE10. (X), TE19. (X), TE22. (X), TE22. (X)

Commit message: - Updated all of the various And-OR-Invert gates to have consistent names.  - Added the schematic for CL3 / SL3 GPIO pins.  There are no surprises revealed by this.  - Finished up the CPU address decoding tracing.  - Added one of the 'artifact' counters from the pulse channels
Parts:
- removed TA1, TA8: BUFFER, symbol MMC5:BUFFER
Connections:
- net at TE41. (X): now also TE20. (X), TE40. (X)
- net at TC23. (X): now also TC12. (X), TC13. (X); no longer TC24. (X)
- net at TD25. (X): now also TD30. (/Q); no longer TD24. (X)
- net at TD30. (/Q): now also TD27. (X); no longer TD25. (X)
- net at TB35. (X): now also TB36. (X); no longer TB32. (/Q)
- net at TB36. (X): now also TB41. (/Q); no longer TB35. (X)
- net at TB10. (/Q): now also TB9. (X); no longer TB11. (X)
- net at TB13. (X): now also TB14. (X); no longer TB10. (/Q)
- net at TB5. (X): now also TB4. (X); no longer TB10. (/Q)
- net at TB9. (X): now also TB8. (X); no longer TB10. (/Q)
- net at TD7. (X): now also TD8. (/Q); no longer TD6. (X)
- net at TD19. (X): now also TD18. (X), TD20. (X)
- net at TC32. (X): now also TC33. (/Q); no longer TC31. (X)
- net at TE11. (X): now also TE8. (/Q); no longer TE12. (X)
- net at TE8. (/Q): now also TE9. (X); no longer TE11. (X)
- net at TE32. (X): now also TE20. (X), TE31. (X)
- net at TD31. (X): now also TD20. (X), TD32. (X); no longer TD30. (/Q)
- net at TE29. (X): now also TE30. (/Q); no longer TE28. (X)
- net at TB31. (X): now also TB32. (/Q); no longer TB30. (X)
- net at TD22. (X): now also TC1. (X), TD21. (X)
- net at TE30. (/Q): now also TE25. (X); no longer TE29. (X)
- net at TE33. (X): now also TE34. (X); no longer TE30. (/Q)
- net at TE34. (X): now also TE39. (/Q); no longer TE33. (X)
- net at TC6. (X): now also TC11. (/Q); no longer TC5. (X)
- net at TC11. (/Q): now also TC12. (X); no longer TC6. (X)
- net at TA29. (X): now also TA7. (X); no longer TA30. (X)
- net at TB27. (X): now also TB26. (X); no longer TB32. (/Q)
- net at TB26. (X): now also TB19. (/Q); no longer TB27. (X)
- net at TB23. (X): now also TB24. (X); no longer TB22. (X)
- net at TB24. (X): no longer TB23. (X)
- net at TC33. (/Q): now also TC28. (X); no longer TC32. (X)
- net at TC14. (X): now also TC11. (/Q); no longer TC15. (X)
- net at TD10. (X): now also TD20. (X), TD9. (X)
- net at TD39. (/Q): now also TD34. (X); no longer TD36. (X)
- net at TD29. (X): now also TD28. (X); no longer TD30. (/Q)
- net at TD33. (X): now also TD34. (X); no longer TD30. (/Q)
- net at TB20. (X): now also TB21. (X), TB22. (X); no longer TB19. (/Q)
- net at TE38. (X): now also TE37. (X); no longer TE39. (/Q)
- net at TC20. (/Q): now also TC19. (X); no longer TC27. (X)
- net at TC19. (X): now also TC18. (X); no longer TC20. (/Q)
- net at TB19. (/Q): now also TB16. (X); no longer TB14. (X)
- net at TB18. (X): now also TB17. (X); no longer TB19. (/Q)
- net at TB40. (X): now also TB39. (X); no longer TB41. (/Q)
- net at TE39. (/Q): now also TE40. (X)
- net at TC36. (X): now also TC37. (X); no longer TC33. (/Q)
- net at TC28. (X): now also TC27. (X); no longer TC33. (/Q)
- net at TE17. (/Q): now also TE12. (X); no longer TE16. (X)
- net at TE24. (X): now also TE25. (X); no longer TE17. (/Q)
- net at TC37. (X): now also TC42. (/Q); no longer TC36. (X)
- net at TC10. (X): now also TC9. (X); no longer TC11. (/Q)
- net at TB32. (/Q): now also TB29. (X); no longer TB31. (X)
- net at TA28. (X): now also TA27. (X); no longer TA16. (/Q)
- net at TE7. (X): now also TE6. (X); no longer TE8. (/Q)
- net at TD12. (X): now also TD11. (X); no longer TD17. (/Q)
- net at TD11. (X): now also TD8. (/Q); no longer TD12. (X)
- net at TD17. (/Q): now also TD16. (X); no longer TD14. (X)
- net at TD16. (X): now also TD15. (X); no longer TD17. (/Q)
- net at TA27. (X): now also TD42. (X); no longer TA28. (X)
- net at TB33. (X): now also TB22. (X), TB34. (X); no longer TB32. (/Q)
- net at TA10. (X), TA9. (X): now also TB1. (X)
- net at TE3. (X): now also TE2. (X); no longer TE8. (/Q)
- net at TD38. (X): now also TD37. (X); no longer TD39. (/Q)
- net at TC41. (X): now also TC42. (/Q); no longer TC40. (X)
- net at TC42. (/Q): no longer TC41. (X)
- new net: TC23. (X), TC34. (X), TC35. (X)
- new net: TC23. (X), TC24. (X)
- new net: TC23. (X), TC43. (X), TC44. (X)
- new net: TC21. (X), TC22. (X), TC23. (X)
- new net: TB6. (X), TB7. (X), TB8. (X)
- new net: TD24. (X), TD25. (X)
- new net: TB32. (/Q), TB35. (X)
- new net: TA16. (/Q), TA18. (X), TA19. (X)
- new net: TA17. (X), TA18. (X)
- new net: TB10. (/Q), TB11. (X)
- new net: TB10. (/Q), TB13. (X)
- new net: TB10. (/Q), TB5. (X)
- new net: TB10. (/Q), TB7. (X)
- new net: TA11. (X), TA12. (/Q)
- new net: TA11. (X), TF9. (X)
- new net: TD4. (X), TD5. (X), TD6. (X)
- new net: TD6. (X), TD7. (X)
- new net: TB22. (X), TB42. (X), TB43. (X)
- new net: TC38. (X), TC39. (X), TC42. (/Q)
- new net: TC31. (X), TC32. (X)
- new net: TC30. (X), TC31. (X)
- new net: TC2. (X), TC24. (X), TC25. (X)
- new net: TE11. (X), TE12. (X)
- new net: TD30. (/Q), TD31. (X)
- new net: TE21. (X), TE22. (X), TE42. (X)
- new net: TA23. (X), TA6. (X), TA7. (X)
- new net: TA23. (X), TE43. (X)
- new net: TA23. (X), TA29. (X), TE43. (X)
- new net: TE28. (X), TE29. (X)
- new net: TE27. (X), TE28. (X)
- new net: TB30. (X), TB31. (X)
- new net: TB28. (X), TB29. (X), TB30. (X)
- new net: TD2. (X), TD22. (X), TD23. (X)
- new net: TE26. (X), TE27. (X), TE30. (/Q)
- new net: TE30. (/Q), TE33. (X)
- new net: TC5. (X), TC6. (X)
- new net: TC16. (X), TC17. (X), TC20. (/Q)
- new net: TC17. (X), TC18. (X)
- new net: TE2. (X), TE22. (X), TE23. (X)
- new net: TE18. (X), TE19. (X), TE20. (X)
- new net: TE4. (X), TE5. (X), TE8. (/Q)
- new net: TA29. (X), TA30. (X)
- new net: TB27. (X), TB32. (/Q)
- new net: TB22. (X), TB23. (X)
- new net: TC14. (X), TC15. (X)
- new net: TA16. (/Q), TA21. (X), TA27. (X)
- new net: TD36. (X), TD39. (/Q)
- new net: TD35. (X), TD36. (X), TD37. (X)
- new net: TD29. (X), TD30. (/Q)
- new net: TD30. (/Q), TD33. (X)
- new net: TB19. (/Q), TB20. (X)
- new net: TE38. (X), TE39. (/Q)
- new net: TB11. (X), TB12. (X), TB22. (X)
- new net: TC11. (/Q), TC7. (X), TC8. (X)
- new net: TC8. (X), TC9. (X)
- new net: TB24. (X), TB25. (X), TB4. (X)
- new net: TC25. (X), TC26. (X), TC5. (X)
- new net: TC20. (/Q), TC27. (X)
- new net: TB14. (X), TB19. (/Q)
- new net: TB18. (X), TB19. (/Q)
- new net: TB40. (X), TB41. (/Q)
- new net: TB37. (X), TB38. (X), TB39. (X)
- new net: TB38. (X), TB41. (/Q)
- new net: TA3. (X), TA4. (X)
- new net: TE35. (X), TE36. (X), TE39. (/Q)
- new net: TC33. (/Q), TC36. (X)
- new net: TC29. (X), TC30. (X), TC33. (/Q)
- new net: TE16. (X), TE17. (/Q)
- new net: TE13. (X), TE14. (X), TE17. (/Q)
- new net: TE17. (/Q), TE24. (X)
- new net: TB15. (X), TB16. (X), TB17. (X)
- new net: TC10. (X), TC11. (/Q)
- new net: TA2. (/Q), TA3. (X)
- new net: TE14. (X), TE15. (X)
- new net: TA16. (/Q), TA28. (X)
- new net: TA15. (X), TA16. (/Q)
- new net: TC39. (X), TC40. (X)
- new net: TD26. (X), TD27. (X), TD28. (X)
- new net: TA5. (/Q), TA6. (X)
- new net: TE7. (X), TE8. (/Q)
- new net: TD12. (X), TD17. (/Q)
- new net: TD5. (X), TD8. (/Q)
- new net: TD14. (X), TD17. (/Q)
- new net: TD13. (X), TD14. (X), TD15. (X)
- new net: TB32. (/Q), TB33. (X)
- new net: TE10. (X), TE20. (X), TE9. (X)
- new net: TA10. (X), TA9. (X)
- new net: TE36. (X), TE37. (X)
- new net: TD42. (X), TD43. (X)
- new net: TD20. (X), TD40. (X), TD41. (X)
- new net: TE3. (X), TE8. (/Q)
- new net: TD38. (X), TD39. (/Q)
- new net: TC40. (X), TC41. (X)
- new net: TE5. (X), TE6. (X)
- now unconnected: TB24. (X), TC13. (X), TC22. (X), TC25. (X), TC25. (X), TC35. (X), TC42. (/Q), TC42. (/Q), TD32. (X), TE10. (X), TE19. (X), TE22. (X), TE22. (X)
