File: Schematic (KiCAD)/ppu_data_bus.kicad_sch (KiCad schematic)
At the start: 111 parts

Commit message: - Lots of additional comments and signal name improvements.  - "Don't know what this is yet but it is important" section of the pulse channels:    - I worked out the logic and it is a 4-bit binary up-counter with preload, made from gates and D-latches instead of T-flip-flops.    - It is extremely similar to the envelope counter, but takes twice the die space and much more traces.    - None of its outputs go anywhere else, so I believe that it has no actual function.    - It seems to be a previous attempt at making the envelope counter and it got disconnected and left in.    - Each pulse channel has its own copy and I moved both of them to the "Artifacts" sheet.    - The wasted space amounts to about half of one of the large columns on the left side of the die.  - A couple of "OAI2" cells that noted "unclear order": I determined the correct order of the inputs based on several others which were known.  - Deduced the purpose of the 2 separate methods of scanline detection:    - The one looking for 3 consecutive reads finds the start of a scanline.    - The one counting PPU /RD to find PPU cycle 336, finds the end of the scanline.    - I moved these beside each other on the same sheet for clarity.  - A66.5 Changed from Nand to Nor in order to make sense.  - Basic test mode:    - Pin 92: Active low, enables test mode.    - Pin 29: In test mode, it gives external control of "Scanline Start Detection", which is normally done with the familiar 3 matching PPU reads.  When not in test mode, the pin has no function.    - Pin 30: In test mode, it gives external control of "Scanline End Detection", which is normally done by counting PPU /RD to find PPU cycle 336.  It also gives control of "Pulse Length Clock" when in test mode.  When not in test mode, the pin has no function.    - Pin 98/SL3: In test mode, it gives external control of "Pulse Timer Clock".  Whether or not in test mode, this pin low makes the MMC5 pretend $5104 had not yet been written since reset, probably as a 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
Connections:
- net at BK24. (X): now also BK23. (X); no longer BK25. (X)
- net at BK23. (X): now also BL16. (X); no longer BK24. (X)
- net at BL14. (X): now also BL2. (X); no longer BK15. (X)
- net at BL45. (X): now also BL46. (X); no longer BL41. (X)
- net V-Split_Rendering{BL43}: now reaches BL41. (X)
- net V-Split_Rendering{BL43}: now also BH16. (X), BH25. (X), BH8. (X), BL29. (X), BL32. (X), BL36. (X); no longer BL42. (X)
- net at BH21. (X): now also BH12. (X), BH4. (X); no longer BH22. (X)
- net at BK8. (X): now also BK7. (X); no longer BK9. (X)
- net at BK7. (X): now also BK15. (X), BK23. (X), BK31. (X), BK43. (X); no longer BK8. (X)
- net at BH19. (X): now also BH14. (X), BH6. (X); no longer BH20. (X)
- net at BH11. (X): now also BH12. (X); no longer BH13. (X)
- net at BL19. (X): now also BL7. (X); no longer BK35. (X)
- net at BL35. (X): now also BL29. (X); no longer BL40. (X)
- net at BL12. (X): now also BK1. (X); no longer BK7. (X)
- net at S1. (X): now also BH20. (X), BH24. (X), BH27. (X); no longer S2. (X)
- net at BK31. (X): now also BK32. (X); no longer BL18. (X)
- net at BK32. (X): now also BK33. (X); no longer BK31. (X)
- net at BK36. (X): now also BK35. (X); no longer BK37. (X)
- net at BH18. (X): now also BH22. (X), BH27. (X); no longer BH17. (X)
- net at BK28. (X): now also BK27. (X); no longer BK29. (X)
- net at BH2. (X): now also BH3. (X); no longer BH1. (X)
- net at BH3. (X): now also BH6. (X); no longer BH2. (X)
- net at BL16. (X): now also BL4. (X); no longer BK23. (X)
- net at BK11. (X): now also BK12. (X); no longer BL13. (X)
- net at BK12. (X): now also BK13. (X); no longer BK11. (X)
- net at BH10. (X): now also BH11. (X); no longer BH9. (X)
- net at BL15. (X): now also BK19. (X); no longer BL3. (X)
- net at BL17. (X): now also BL5. (X); no longer BK27. (X)
- net at BL37. (X): now also BL38. (X), BL42. (X); no longer BL36. (X)
- net at BK20. (X): now also BK19. (X); no longer BK21. (X)
- removed net V-Split_Side_Latched{BL43}: BH16. (X), BH25. (X), BH8. (X), BL29. (X), BL32. (X), BL36. (X), BL41. (X)
- new net: BK24. (X), BK25. (X)
- new net: BL12. (X), BL13. (X), BL14. (X), BL15. (X), BL16. (X), BL17. (X), BL18. (X), BL19. (X), BL31. (X)
- new net: BK15. (X), BL14. (X)
- new net: BK10. (X), BK14. (X), BK18. (X), BK22. (X), BK26. (X), BK30. (X), BK34. (X), BK38. (X), BL39. (X)
- new net: BL41. (X), BL45. (X)
- new net: BL41. (X), BL42. (X)
- new net: BH21. (X), BH22. (X)
- new net: BK8. (X), BK9. (X)
- new net: BK4. (X), BK5. (X)
- new net: BK2. (X), BK5. (X)
- new net: BH19. (X), BH20. (X)
- new net: BK25. (X), BK26. (X)
- new net: BH13. (X), BH23. (X), BH5. (X)
- new net: BH11. (X), BH13. (X)
- new net: BK35. (X), BL19. (X)
- new net: BK10. (X), BK9. (X)
- new net: BL34. (X), BL35. (X), BL37. (X)
- new net: BL35. (X), BL40. (X)
- new net: BK7. (X), BL12. (X)
- new net: S1. (X), S2. (X)
- new net: BK15. (X), BK23. (X), BK31. (X), BK42. (X), BK7. (X)
- new net: BK31. (X), BL18. (X)
- new net: BK37. (X), BK38. (X)
- new net: BK36. (X), BK37. (X)
- new net: BH18. (X), BH20. (X), BH26. (X)
- new net: BH18. (X), BH20. (X), BH22. (X), BH24. (X), BH25. (X)
- new net: BH17. (X), BH18. (X)
- new net: BH15. (X), BH17. (X), BH7. (X)
- new net: BH11. (X), BH15. (X)
- new net: BK29. (X), BK30. (X)
- new net: BK28. (X), BK29. (X)
- new net: BK11. (X), BK19. (X), BK27. (X), BK35. (X), BK40. (X)
- new net: BK39. (X), BK40. (X), BK42. (X)
- new net: BH1. (X), BH2. (X)
- new net: BK11. (X), BK19. (X), BK27. (X), BK35. (X), BK41. (X)
- new net: BK11. (X), BL13. (X)
- new net: BK21. (X), BK22. (X)
- new net: BK13. (X), BK14. (X)
- new net: BH10. (X), BH9. (X)
- new net: BL28. (X), BL29. (X), BL37. (X)
- new net: BL15. (X), BL3. (X)
- new net: BK27. (X), BL17. (X)
- new net: BK41. (X), BK43. (X), BK44. (X)
- new net: BL36. (X), BL37. (X)
- new net: BK20. (X), BK21. (X)
- new net: BK33. (X), BK34. (X)
- new net: BH11. (X), BH16. (X)
- new net: BH3. (X), BH5. (X)
- new net: BH3. (X), BH8. (X)
- new net: BH3. (X), BH4. (X)
- new net: BH3. (X), BH7. (X)
- new net: BK17. (X), BK18. (X)
- new net: BH11. (X), BH14. (X)
Changed lines of the file:
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@@
 		)
 	)
-	(global_label "V-Split_Side_Latched{BL43}"
+	(global_label "V-Split_Rendering{BL43}"
 		(shape input)
 		(at 179.07 21.59 180)
@@
 		)
 		(property "Intersheetrefs" "${INTERSHEET_REFS}"
-			(at 149.294 21.59 0)
+			(at 152.2573 21.59 0)
 			(effects
 				(font

Commit message: I fixed 2 errors in the letterless MMC5 tracing:
1. BK5 is a NAND-4 gate.  It was thought to be NAND-3 before.
2.  BL83 and BL96 signals got swapped here before.  They actually cross each other:

BL83 = "PPU_RW_Mode_%0x_Access"
BL96 = "+ExRAM_Mode_$0x"

This propagated out to several changes in the schematic.
Parts:
- removed BK5: NAND_3, symbol MMC5:NAND_3
- added BK5: NAND_4, symbol MMC5:NAND_4
Connections:
- net PPU_RW_Mode_%0x_Access{BL48} is gone; now on net +ExRAM_Mode_$0x{BL48}: BL42. (X)
- net +PPU_A13_B{BK6}: now also BK5. (X)
- net +PPU_RD_A{BJ1}: now also BK5. (X)
- net at BK24. (X): now also BK23. (X); no longer BK25. (X)
- net at BK23. (X): now also BL16. (X); no longer BK24. (X)
- net at BL14. (X): now also BL2. (X); no longer BK15. (X)
- net at BL45. (X): now also BL46. (X); no longer BL41. (X)
- net +ExRAM_Mode_$0x{BL48}: now reaches BL42. (X)
- net +ExRAM_Mode_$0x{BL48}: no longer BL41. (X)
- net at BH21. (X): now also BH12. (X), BH4. (X); no longer BH22. (X)
- net at BK8. (X): now also BK7. (X); no longer BK9. (X)
- net at BK7. (X): now also BK15. (X), BK23. (X), BK31. (X), BK43. (X); no longer BK8. (X)
- net at BH19. (X): now also BH14. (X), BH6. (X); no longer BH20. (X)
- net at BH11. (X): now also BH12. (X); no longer BH13. (X)
- net at BL19. (X): now also BL7. (X); no longer BK35. (X)
- net at BL35. (X): now also BL29. (X); no longer BL40. (X)
- net at BL12. (X): now also BK1. (X); no longer BK7. (X)
- net at S1. (X): now also BH20. (X), BH24. (X), BH27. (X); no longer S2. (X)
- net at BK31. (X): now also BK32. (X); no longer BL18. (X)
- net at BK32. (X): now also BK33. (X); no longer BK31. (X)
- net at BK36. (X): now also BK35. (X); no longer BK37. (X)
- net at BH18. (X): now also BH22. (X), BH27. (X); no longer BH17. (X)
- net at BK28. (X): now also BK27. (X); no longer BK29. (X)
- net at BH2. (X): now also BH3. (X); no longer BH1. (X)
- net at BH3. (X): now also BH6. (X); no longer BH2. (X)
- net at BL16. (X): now also BL4. (X); no longer BK23. (X)
- net at BK11. (X): now also BK12. (X); no longer BL13. (X)
- net at BK12. (X): now also BK13. (X); no longer BK11. (X)
- net at BH10. (X): now also BH11. (X); no longer BH9. (X)
- net at BL15. (X): now also BK19. (X); no longer BL3. (X)
- net at BL17. (X): now also BL5. (X); no longer BK27. (X)
- net at BL37. (X): now also BL38. (X), BL42. (X); no longer BL36. (X)
- net at BK20. (X): now also BK19. (X); no longer BK21. (X)
- new net: BK24. (X), BK25. (X)
- new net: BL12. (X), BL13. (X), BL14. (X), BL15. (X), BL16. (X), BL17. (X), BL18. (X), BL19. (X), BL31. (X)
- new net: BK15. (X), BL14. (X)
- new net: BK10. (X), BK14. (X), BK18. (X), BK22. (X), BK26. (X), BK30. (X), BK34. (X), BK38. (X), BL39. (X)
- new net: BL41. (X), BL45. (X)
- new net: BL41. (X), BL42. (X)
- new net: BH21. (X), BH22. (X)
- new net: BK8. (X), BK9. (X)
- new net: BH19. (X), BH20. (X)
- new net: BK25. (X), BK26. (X)
- new net: BH13. (X), BH23. (X), BH5. (X)
- new net: BH11. (X), BH13. (X)
- new net: BK35. (X), BL19. (X)
- new net: BK10. (X), BK9. (X)
- new net: BL34. (X), BL35. (X), BL37. (X)
- new net: BL35. (X), BL40. (X)
- new net: BK7. (X), BL12. (X)
- new net: S1. (X), S2. (X)
- new net: BK15. (X), BK23. (X), BK31. (X), BK42. (X), BK7. (X)
- new net: BK31. (X), BL18. (X)
- new net: BK37. (X), BK38. (X)
- new net: BK36. (X), BK37. (X)
- new net: BH18. (X), BH20. (X), BH26. (X)
- new net: BH18. (X), BH20. (X), BH22. (X), BH24. (X), BH25. (X)
- new net: BH17. (X), BH18. (X)
- new net: BH15. (X), BH17. (X), BH7. (X)
- new net: BH11. (X), BH15. (X)
- new net: BK29. (X), BK30. (X)
- new net: BK28. (X), BK29. (X)
- new net: BK11. (X), BK19. (X), BK27. (X), BK35. (X), BK40. (X)
- new net: BK39. (X), BK40. (X), BK42. (X)
- new net: BH1. (X), BH2. (X)
- new net: BK11. (X), BK19. (X), BK27. (X), BK35. (X), BK41. (X)
- new net: BK11. (X), BL13. (X)
- new net: BK21. (X), BK22. (X)
- new net: BK13. (X), BK14. (X)
- new net: BH10. (X), BH9. (X)
- new net: BK4. (X), BK5. (X)
- new net: BK2. (X), BK5. (X)
- new net: BL28. (X), BL29. (X), BL37. (X)
- new net: BL15. (X), BL3. (X)
- new net: BK27. (X), BL17. (X)
- new net: BK41. (X), BK43. (X), BK44. (X)
- new net: BL36. (X), BL37. (X)
- new net: BK20. (X), BK21. (X)
- new net: BK33. (X), BK34. (X)
- new net: BH11. (X), BH16. (X)
- new net: BH3. (X), BH5. (X)
- new net: BH3. (X), BH8. (X)
- new net: BH3. (X), BH4. (X)
- new net: BH3. (X), BH7. (X)
- new net: BK17. (X), BK18. (X)
- new net: BH11. (X), BH14. (X)
- new net /PPU_A12_B{BK3}: BK5. (X)
Other:
- moved on the sheet: BK2
Changed lines of the file:
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@@
 	(wire
 		(pts
-			(xy 372.11 214.63) (xy 372.11 215.9)
+			(xy 372.11 213.36) (xy 372.11 214.63)
 		)
 		(stroke
@@
 		)
 	)
-	(global_label "PPU_RW_Mode_%0x_Access{BL48}"
+	(global_label "+ExRAM_Mode_$0x{BL48}"
 		(shape input)
 		(at 161.29 72.39 180)
@@
 		)
 		(property "Intersheetrefs" "${INTERSHEET_REFS}"
-			(at 126.4944 72.39 0)
+			(at 134.1145 72.39 0)
 			(effects
 				(font
@@
 		)
 	)
+	(global_label "{slash}PPU_A12_B{BK3}"
+		(shape input)
+		(at 372.11 222.25 180)
+		(fields_autoplaced yes)
+		(effects
+			(font
+				(size 1.27 1.27)
+			)
+			(justify right)
+		)
+		(property "Intersheetrefs" "${INTERSHEET_REFS}"
+			(at 351.7681 222.25 0)
+			(effects
+				(font
+					(size 1.27 1.27)
+				)
+				(justify right)
+				(hide yes)
+			)
+		)
+	)
 	(global_label "PPU_D0_OUT_PIN"
 		(shape output)
@@
 	(global_label "CIRAM_CE_PIN{A9}"
 		(shape input)
-		(at 363.22 214.63 180)
+		(at 363.22 213.36 180)
 		(fields_autoplaced yes)
 		(effects
@@
 		)
 		(property "Intersheetrefs" "${INTERSHEET_REFS}"
-			(at 342.999 214.63 0)
+			(at 342.999 213.36 0)
 			(effects
 				(font
@@
 	(global_label "+PPU_A13_B{BK6}"
 		(shape input)
-		(at 372.11 220.98 180)
+		(at 372.11 219.71 180)
 		(fields_autoplaced yes)
 		(effects
@@
 		)
 		(property "Intersheetrefs" "${INTERSHEET_REFS}"
-			(at 351.5262 220.98 0)
+			(at 351.5262 219.71 0)
 			(effects
 				(font
@@
 	(global_label "+PPU_RD_A{BJ1}"
 		(shape input)
-		(at 372.11 218.44 180)
+		(at 372.11 217.17 180)
 		(fields_autoplaced yes)
 		(effects
@@
 		)
 		(property "Intersheetrefs" "${INTERSHEET_REFS}"
-			(at 352.9776 218.44 0)
+			(at 352.9776 217.17 0)
 			(effects
 				(font
@@
 	)
 	(symbol
-		(lib_name "NAND_3_8")
-		(lib_id "MMC5:NAND_3")
-		(at 377.19 218.44 0)
-		(unit 1)
-		(exclude_from_sim no)
-		(in_bom yes)
-		(on_board yes)
-		(dnp no)
-		(fields_autoplaced yes)
-		(property "Reference" "BK5"
-			(at 377.19 213.614 0)
-			(do_not_autoplace yes)
-			(effects
-				(font
-					(size 1.27 1.27)
-				)
-				(justify top)
-			)
-		)
-		(property "Value" "NAND_3"
-			(at 377.19 218.44 0)
-			(do_not_autoplace yes)
-			(effects
-				(font
-					(size 0.635 0.635)
-				)
-			)
-		)
-		(property "Footprint" ""
-			(at 377.19 218.44 0)
-			(effects
-				(font
-					(size 1.27 1.27)
-				)
-				(hide yes)
-			)
-		)
-		(property "Datasheet" ""
-			(at 377.19 218.44 0)
-			(effects
-				(font
-					(size 1.27 1.27)
-				)
-				(hide yes)
-			)
-		)
-		(property "Description" ""
-			(at 377.19 218.44 0)
-			(effects
-				(font
-					(size 1.27 1.27)
-				)
-				(hide yes)
-			)
-		)
-		(pin ""
-		)
-		(pin ""
-		)
-		(pin ""
-		)
-		(pin ""
-		)
-		(instances
-			(project "MMC5"
-				(path "/46093bf6-f83e-4237-9ece-7350a682aff0/4e6a5c22-b922-467f-8545-4eb558480830"
-					(reference "BK5")
-					(unit 1)
-				)
-			)
-		)
-	)
-	(symbol
 		(lib_name "INVERT_12")
 		(lib_id "MMC5:INVERT")
@@
 	)
 	(symbol
+		(lib_name "NAND_4_1")
+		(lib_id "MMC5:NAND_4")
+		(at 377.19 218.44 0)
+		(unit 1)
+		(exclude_from_sim no)
+		(in_bom yes)
+		(on_board yes)
+		(dnp no)
+		(fields_autoplaced yes)
+		(property "Reference" "BK5"
+			(at 377.19 214.122 0)
+			(do_not_autoplace yes)
+			(effects
+				(font
+					(size 1.27 1.27)
+				)
+				(justify top)
+			)
+		)
+		(property "Value" "NAND_4"
+			(at 377.19 218.44 0)
+			(do_not_autoplace yes)
+			(effects
+				(font
+					(size 0.635 0.635)
+				)
+			)
+		)
+		(property "Footprint" ""
+			(at 377.19 218.44 0)
+			(effects
+				(font
+					(size 1.27 1.27)
+				)
+				(hide yes)
+			)
+		)
+		(property "Datasheet" ""
+			(at 377.19 218.44 0)
+			(effects
+				(font
+					(size 1.27 1.27)
+				)
+				(hide yes)
+			)
+		)
+		(property "Description" ""
+			(at 377.19 218.44 0)
+			(effects
+				(font
+					(size 1.27 1.27)
+				)
+				(hide yes)
+			)
+		)
+		(pin ""
+		)
+		(pin ""
+		)
+		(pin ""
+		)
+		(pin ""
+		)
+		(pin ""
+		)
+		(instances
+			(project ""
+				(path "/46093bf6-f83e-4237-9ece-7350a682aff0/4e6a5c22-b922-467f-8545-4eb558480830"
+					(reference "BK5")
+					(unit 1)
+				)
+			)
+		)
+	)
+	(symbol
 		(lib_name "INVERT_14")
 		(lib_id "MMC5:INVERT")
@@
 		(lib_name "BUFFER_8")
 		(lib_id "MMC5:BUFFER")
-		(at 367.03 214.63 0)
+		(at 367.03 213.36 0)
 		(unit 1)
 		(exclude_from_sim no)
@@
 		(fields_autoplaced yes)
 		(property "Reference" "BK2"
-			(at 367.03 211.328 0)
+			(at 367.03 210.058 0)
 			(do_not_autoplace yes)
 			(effects
@@
 		)
 		(property "Value" "BUFFER"
-			(at 369.824 215.9 0)
+			(at 369.824 214.63 0)
 			(do_not_autoplace yes)
 			(effects
@@
 		)
 		(property "Footprint" ""
-			(at 367.03 214.63 0)
+			(at 367.03 213.36 0)
 			(effects
 				(font
@@
 		)
 		(property "Datasheet" ""
-			(at 367.03 214.63 0)
+			(at 367.03 213.36 0)
 			(effects
 				(font
@@
 		)
 		(property "Description" ""
-			(at 367.03 214.63 0)
+			(at 367.03 213.36 0)
 			(effects
 				(font
