File: Schematic (KiCAD)/ppu_fetch_counting.kicad_sch (KiCad schematic)
At the start: 29 parts, among them M1 10x 2to1 Multiplexer

Commit message: - Lots of additional comments and signal name improvements.  - "Don't know what this is yet but it is important" section of the pulse channels:    - I worked out the logic and it is a 4-bit binary up-counter with preload, made from gates and D-latches instead of T-flip-flops.    - It is extremely similar to the envelope counter, but takes twice the die space and much more traces.    - None of its outputs go anywhere else, so I believe that it has no actual function.    - It seems to be a previous attempt at making the envelope counter and it got disconnected and left in.    - Each pulse channel has its own copy and I moved both of them to the "Artifacts" sheet.    - The wasted space amounts to about half of one of the large columns on the left side of the die.  - A couple of "OAI2" cells that noted "unclear order": I determined the correct order of the inputs based on several others which were known.  - Deduced the purpose of the 2 separate methods of scanline detection:    - The one looking for 3 consecutive reads finds the start of a scanline.    - The one counting PPU /RD to find PPU cycle 336, finds the end of the scanline.    - I moved these beside each other on the same sheet for clarity.  - A66.5 Changed from Nand to Nor in order to make sense.  - Basic test mode:    - Pin 92: Active low, enables test mode.    - Pin 29: In test mode, it gives external control of "Scanline Start Detection", which is normally done with the familiar 3 matching PPU reads.  When not in test mode, the pin has no function.    - Pin 30: In test mode, it gives external control of "Scanline End Detection", which is normally done by counting PPU /RD to find PPU cycle 336.  It also gives control of "Pulse Length Clock" when in test mode.  When not in test mode, the pin has no function.    - Pin 98/SL3: In test mode, it gives external control of "Pulse Timer Clock".  Whether or not in test mode, this pin low makes the MMC5 pretend $5104 had not yet been written since reset, probably as a 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
Parts:
- removed R5: JK-FF Reset, symbol MMC5:JK-FF_Reset
- added P1, S5, S6, X1: INVERT, symbol MMC5:INVERT
- added P2: NOR_2, symbol MMC5:NOR_2
- added R5: D-FF-SR, symbol MMC5:D-FF-SR
- added X2: NAND_2, symbol MMC5:NAND_2
Connections:
- net Increment_PPU_Fetch_Count{S6} is gone; now on net /Scanline_Start_Detected{R2}: S8. (/Q)
- net /New_Scanline_Detected{R2} is gone; now on net /Scanline_Start_Detected{R2}: R11. (X), R13. (X), S12. (/Q), S20. (/Q), S8. (/Q)
- net +PPU_Fetch_Counter.6{S17}: now also S16. (X)
- net /PPU_Fetch_Counter.6{S27}: no longer S16. (X)
- net /Reset_Detect{R14}: now also R5. (/Q)
- net /Scanline_Start_Detected{R2}: now reaches S12. (/Q), S8. (/Q)
- net /Scanline_Start_Detected{R2}: now also R5. (/Q); no longer S10. (X)
- net at S7. (X): now also R9. (X); no longer S8. (/Q)
- net at S19. (X): now also R12. (X); no longer S20. (/Q)
- net at S11. (X): now also R10. (X); no longer S12. (/Q)
- net at S14. (X): now also R11. (X); no longer S15. (/Q)
- removed net V-Split_Scanline_Detected_Internal{R8}: R10. (X), R11. (X), R12. (X), R13. (X), R9. (X)
- new net: S10. (X), S12. (/Q), S8. (/Q)
- new net: R5. (/Q), S16. (X)
- new net: P2. (X), R5. (/Q)
- new net: S22. (X), S23. (/Q), S26. (/Q), S27. (/Q), S28. (/Q)
- new net: P1. (X), S5. (X)
- new net: P1. (X), P2. (X)
- new net: S5. (X), S6. (X)
- new net: S7. (X), S8. (/Q)
- new net: S19. (X), S20. (/Q)
- new net: S12. (/Q), S13. (X), S15. (/Q)
- new net: S11. (X), S12. (/Q)
- new net: S14. (X), S15. (/Q)
- new net: S20. (/Q), S21. (X), S23. (/Q)
- new net: X1. (X), X2. (X)
- new net +In_Frame{Z21}: X2. (X)
- new net +PPU_RD_B{X3}: X2. (X)
- new net Increment_Scanline_Fetch_Count{S6}: R5. (/Q), S6. (X), S8. (/Q)
- new net Scanline_End_Detected_Internal{R8}: R10. (X), R11. (X), R12. (X), R13. (X), R9. (X)
- new net /Any_PPU_Fetch_While_In_Frame{X1}: P2. (X), X1. (X)
Other:
- note added: "0=count 1=don't count"
- note added: "I am guessing this is any PPU fetch excluding sprites"
- note added: "I am not sure if this is NAND 8 or NOR 8. Counter.6: unclear if + or /"
- note added: "Value (None of these numbers make sense.) NOR=> +180 (/.6=+244) NAND=> /75 (/.6=/11)"
- note removed: "I think this may be a NAND 8 instead of NOR."
- note removed: "This Flip-Flop is unknown and J & K are complete guesses. May need swapping or inverting J & K and Q & /Q."
- note removed: "Value 244 or 11"
- moved on the sheet: S16

Commit message: - Improved "Identification of Cells" document for NAND, NOR, and XNOR/XOR gates.  - Gate S16 is a NAND-8 gate; it was shown as NOR-8 before.
Parts:
- removed S16: NOR_8, symbol MMC5:NOR_8
- added S16: NAND_8, symbol MMC5:NAND_8
Connections:
- net +PPU_Fetch_Counter.0{S10}: now also S16. (X)
- net +PPU_Fetch_Counter.1{S12}: now also S16. (X)
- net +PPU_Fetch_Counter.3{S21}: now also S16. (X)
- net +PPU_Fetch_Counter.6{S17}: now also S16. (X)
- net /PPU_Fetch_Counter.2{S15}: now also S16. (X)
- net /PPU_Fetch_Counter.4{S23}: now also S16. (X)
- net /PPU_Fetch_Counter.5{S26}: now also S16. (X)
- net /PPU_Fetch_Counter.7{S28}: now also S16. (X)
- net at P1. (X): now also P2. (X); no longer S5. (X)
- net at S7. (X): now also R9. (X); no longer S8. (/Q)
- net at S19. (X): now also R12. (X); no longer S20. (/Q)
- net at S11. (X): now also R10. (X); no longer S12. (/Q)
- net at S14. (X): now also R11. (X); no longer S15. (/Q)
- new net: S10. (X), S12. (/Q), S8. (/Q)
- new net: R5. (/Q), S16. (X)
- new net: P2. (X), R5. (/Q)
- new net: S22. (X), S23. (/Q), S26. (/Q), S27. (/Q), S28. (/Q)
- new net: P1. (X), S5. (X)
- new net: S7. (X), S8. (/Q)
- new net: S19. (X), S20. (/Q)
- new net: S12. (/Q), S13. (X), S15. (/Q)
- new net: S11. (X), S12. (/Q)
- new net: S14. (X), S15. (/Q)
- new net: S20. (/Q), S21. (X), S23. (/Q)
- new net: X1. (X), X2. (X)
Other:
- note added: "Counter.6: unclear if + or /"
- note added: "Value (None of these numbers make sense.) NAND=> /75 (/.6=/11)"
- note removed: "I am not sure if this is NAND 8 or NOR 8. Counter.6: unclear if + or /"
- note removed: "Value (None of these numbers make sense.) NOR=> +180 (/.6=+244) NAND=> /75 (/.6=/11)"
Changed lines of the file:
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@@
 	(generator_version "9.0")
 	(paper "USLedger")
-	(text "I am not sure if this is\nNAND 8 or NOR 8.\n\nCounter.6: unclear if + or /"
+	(text "Counter.6: unclear if + or /"
 		(exclude_from_sim no)
 		(at 80.518 189.992 0)
@@
 		)
 	)
-	(text "Value (None of these numbers make sense.)\nNOR=> +180 (/.6=+244)\nNAND=> /75 (/.6=/11)"
+	(text "Value (None of these numbers make sense.)\nNAND=> /75 (/.6=/11)"
 		(exclude_from_sim no)
 		(at 90.932 170.434 0)
@@
 	)
 	(symbol
-		(lib_id "MMC5:NOR_8")
-		(at 86.36 173.99 0)
-		(unit 1)
-		(exclude_from_sim no)
-		(in_bom yes)
-		(on_board yes)
-		(dnp no)
-		(fields_autoplaced yes)
-		(property "Reference" "S16"
-			(at 86.36 169.672 0)
-			(do_not_autoplace yes)
-			(effects
-				(font
-					(size 1.27 1.27)
-				)
-				(justify top)
-			)
-		)
-		(property "Value" "NOR_8"
-			(at 86.36 173.99 0)
-			(do_not_autoplace yes)
-			(effects
-				(font
-					(size 0.635 0.635)
-				)
-			)
-		)
-		(property "Footprint" ""
-			(at 86.36 173.99 0)
-			(effects
-				(font
-					(size 1.27 1.27)
-				)
-				(hide yes)
-			)
-		)
-		(property "Datasheet" ""
-			(at 86.36 173.99 0)
-			(effects
-				(font
-					(size 1.27 1.27)
-				)
-				(hide yes)
-			)
-		)
-		(property "Description" ""
-			(at 86.36 173.99 0)
-			(effects
-				(font
-					(size 1.27 1.27)
-				)
-				(hide yes)
-			)
-		)
-		(pin ""
-		)
-		(pin ""
-		)
-		(pin ""
-		)
-		(pin ""
-		)
-		(pin ""
-		)
-		(pin ""
-		)
-		(pin ""
-		)
-		(pin ""
-		)
-		(pin ""
-		)
-		(instances
-			(project ""
-				(path "/46093bf6-f83e-4237-9ece-7350a682aff0/e44f8884-f3b7-4888-9ab5-cb34742c183f"
-					(reference "S16")
-					(unit 1)
-				)
-			)
-		)
-	)
-	(symbol
 		(lib_id "MMC5:T-FF_Reset")
 		(at 93.98 62.23 0)
@@
 					(unit 1)
 				)
+			)
+		)
+	)
+	(symbol
+		(lib_id "MMC5:NAND_8")
+		(at 86.36 173.99 0)
+		(unit 1)
+		(exclude_from_sim no)
+		(in_bom yes)
+		(on_board yes)
+		(dnp no)
+		(fields_autoplaced yes)
+		(property "Reference" "S16"
+			(at 86.36 169.672 0)
+			(do_not_autoplace yes)
+			(effects
+				(font
+					(size 1.27 1.27)
+				)
+				(justify top)
+			)
+		)
+		(property "Value" "NAND_8"
+			(at 86.36 173.99 0)
+			(do_not_autoplace yes)
+			(effects
+				(font
+					(size 0.635 0.635)
+				)
+			)
+		)
+		(property "Footprint" ""
+			(at 86.36 173.99 0)
+			(effects
+				(font
+					(size 1.27 1.27)
+				)
+				(hide yes)
+			)
+		)
+		(property "Datasheet" ""
+			(at 86.36 173.99 0)
+			(effects
+				(font
+					(size 1.27 1.27)
+				)
+				(hide yes)
+			)
+		)
+		(property "Description" ""
+			(at 86.36 173.99 0)
+			(effects
+				(font
+					(size 1.27 1.27)
+				)
+				(hide yes)
+			)
+		)
+		(pin ""
+		)
+		(pin ""
+		)
+		(pin ""
+		)
+		(pin ""
+		)
+		(pin ""
+		)
+		(pin ""
+		)
+		(pin ""
+		)
+		(pin ""
+		)
+		(pin ""
+		)
+		(instances
+			(project ""
+				(path "/46093bf6-f83e-4237-9ece-7350a682aff0/e44f8884-f3b7-4888-9ab5-cb34742c183f"
+					(reference "S16")
+					(unit 1)
+				)

Commit message: Schematic and SVG Updates
Connections:
- net at P1. (X): now also P2. (X); no longer S5. (X)
- net at S7. (X): now also R9. (X); no longer S8. (/Q)
- net at S19. (X): now also R12. (X); no longer S20. (/Q)
- net at S11. (X): now also R10. (X); no longer S12. (/Q)
- net at S14. (X): now also R11. (X); no longer S15. (/Q)
- removed net +PPU_Fetch_Counter.1{S12}: S12. (/Q), S16. (X)
- new net: S10. (X), S12. (/Q), S8. (/Q)
- new net: R5. (/Q), S16. (X)
- new net: P2. (X), R5. (/Q)
- new net: S22. (X), S23. (/Q), S26. (/Q), S27. (/Q), S28. (/Q)
- new net: P1. (X), S5. (X)
- new net: S7. (X), S8. (/Q)
- new net: S19. (X), S20. (/Q)
- new net: S11. (X), S12. (/Q)
- new net: S14. (X), S15. (/Q)
- new net: S20. (/Q), S21. (X), S23. (/Q)
- new net: X1. (X), X2. (X)
- new net /PPU_Fetch_Counter.1{S12}: S12. (/Q), S13. (X), S15. (/Q), S16. (X)
Other:
- note added: "Value (None of these numbers make sense.) NAND=> /73 (/.6=/9)"
- note removed: "Value (None of these numbers make sense.) NAND=> /75 (/.6=/11)"
Changed lines of the file:
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@@
 		)
 	)
-	(text "Value (None of these numbers make sense.)\nNAND=> /75 (/.6=/11)"
+	(text "Value (None of these numbers make sense.)\nNAND=> /73 (/.6=/9)"
 		(exclude_from_sim no)
 		(at 90.932 170.434 0)
@@
 	)
 	(junction
+		(at 100.33 53.34)
+		(diameter 0)
+		(color 0 0 0 0)
+	)
+	(junction
 		(at 175.26 175.26)
 		(diameter 0)
@@
 	(wire
 		(pts
+			(xy 100.33 53.34) (xy 100.33 49.53)
+		)
+		(stroke
+			(width 0)
+			(type default)
+		)
+	)
+	(wire
+		(pts
 			(xy 121.92 179.07) (xy 123.19 179.07)
 		)
@@
 	(wire
 		(pts
+			(xy 100.33 53.34) (xy 109.22 53.34)
+		)
+		(stroke
+			(width 0)
+			(type default)
+		)
+	)
+	(wire
+		(pts
 			(xy 100.33 109.22) (xy 100.33 111.76)
 		)
@@
 	(wire
 		(pts
-			(xy 109.22 45.72) (xy 100.33 45.72)
-		)
-		(stroke
-			(width 0)
-			(type default)
-		)
-	)
-	(wire
-		(pts
 			(xy 87.63 97.79) (xy 100.33 97.79)
 		)
@@
 	(wire
 		(pts
-			(xy 100.33 45.72) (xy 100.33 46.99)
-		)
-		(stroke
-			(width 0)
-			(type default)
-		)
-	)
-	(wire
-		(pts
 			(xy 87.63 107.95) (xy 87.63 97.79)
 		)
@@
 	(wire
 		(pts
-			(xy 100.33 55.88) (xy 100.33 49.53)
+			(xy 100.33 55.88) (xy 100.33 53.34)
 		)
 		(stroke
@@
 		)
 	)
-	(global_label "+PPU_Fetch_Counter.1{S12}"
+	(global_label "{slash}PPU_Fetch_Counter.1{S12}"
 		(shape input)
 		(at 81.28 167.64 180)
@@
 		)
 		(property "Intersheetrefs" "${INTERSHEET_REFS}"
-			(at 111.2375 167.64 0)
-			(effects
-				(font
-					(size 1.27 1.27)
-				)
-				(justify left)
+			(at 51.5644 167.64 0)
+			(effects
+				(font
+					(size 1.27 1.27)
+				)
+				(justify right)
 				(hide yes)
 			)
@@
 		)
 	)
-	(global_label "+PPU_Fetch_Counter.1{S12}"
+	(global_label "{slash}PPU_Fetch_Counter.1{S12}"
 		(shape output)
-		(at 109.22 45.72 0)
+		(at 109.22 53.34 0)
 		(fields_autoplaced yes)
 		(effects
@@
 		)
 		(property "Intersheetrefs" "${INTERSHEET_REFS}"
-			(at 139.1775 45.72 0)
-			(effects
-				(font
+			(at 138.9356 53.34 0)
+			(effects
+				(font

Commit message: Tracing and schematic updates.  - Added timer to schematic.  - Added all items from artifacts sheet to the MMC5A trace.
Connections:
- net +PPU_RD_B{X3} is gone; now on net /PPU_RD_B{X3}: X2. (X)
- net 1? is gone; now on net PPU_Fetch_Mux_9{M1}: M1. (Y10)
- net 1: now also M1. (Y10)
- net at P1. (X): now also P2. (X); no longer S5. (X)
- net at S7. (X): now also R9. (X); no longer S8. (/Q)
- net at S19. (X): now also R12. (X); no longer S20. (/Q)
- net at S11. (X): now also R10. (X); no longer S12. (/Q)
- net at S14. (X): now also R11. (X); no longer S15. (/Q)
- net /PPU_RD_B{X3}: now reaches X2. (X)
- net /PPU_RD_B{X3}: no longer X1. (X)
- new net: S10. (X), S12. (/Q), S8. (/Q)
- new net: R5. (/Q), S16. (X)
- new net: P2. (X), R5. (/Q)
- new net: S22. (X), S23. (/Q), S26. (/Q), S27. (/Q), S28. (/Q)
- new net: P1. (X), S5. (X)
- new net: S7. (X), S8. (/Q)
- new net: S19. (X), S20. (/Q)
- new net: S11. (X), S12. (/Q)
- new net: S14. (X), S15. (/Q)
- new net: S20. (/Q), S21. (X), S23. (/Q)
- new net: X1. (X), X2. (X)
Other:
- note added: "The output of this mux is the ExRAM address for the data to be substituted for the PPU. See sheet 14."
Changed lines of the file:
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@@
+		)
+	)
+	(text "The output of this mux is the\nExRAM address for the data to\nbe substituted for the PPU.\n\nSee sheet 14."
+		(exclude_from_sim no)
+		(at 273.304 73.152 0)
+		(effects
+			(font
+				(size 1.27 1.27)
+			)
+			(justify left)
 		)
 	)
@@
 		)
 	)
+	(global_label "1"
+		(shape input)
+		(at 232.41 113.03 180)
+		(fields_autoplaced yes)
+		(effects
+			(font
+				(size 1.27 1.27)
+			)
+			(justify right)
+		)
+		(property "Intersheetrefs" "${INTERSHEET_REFS}"
+			(at 228.2153 113.03 0)
+			(effects
+				(font
+					(size 1.27 1.27)
+				)
+				(justify right)
+				(hide yes)
+			)
+		)
+	)
 	(global_label "PPU_Fetch_Mux_9{M1}"
 		(shape output)
@@
 		)
 	)
-	(global_label "1?"
+	(global_label "1"
 		(shape input)
 		(at 232.41 93.98 180)
@@
 		)
 		(property "Intersheetrefs" "${INTERSHEET_REFS}"
-			(at 227.1267 93.98 0)
+			(at 228.2153 93.98 0)
 			(effects
 				(font
@@
 		)
 	)
-	(global_label "1?"
-		(shape input)
-		(at 232.41 106.68 180)
-		(fields_autoplaced yes)
-		(effects
-			(font
-				(size 1.27 1.27)
-			)
-			(justify right)
-		)
-		(property "Intersheetrefs" "${INTERSHEET_REFS}"
-			(at 227.1267 106.68 0)
-			(effects
-				(font
-					(size 1.27 1.27)
-				)
-				(justify right)
-				(hide yes)
-			)
-		)
-	)
-	(global_label "1?"
-		(shape input)
-		(at 232.41 113.03 180)
-		(fields_autoplaced yes)
-		(effects
-			(font
-				(size 1.27 1.27)
-			)
-			(justify right)
-		)
-		(property "Intersheetrefs" "${INTERSHEET_REFS}"
-			(at 227.1267 113.03 0)
-			(effects
-				(font
-					(size 1.27 1.27)
-				)
-				(justify right)
-				(hide yes)
-			)
-		)
-	)
 	(global_label "PPU_Fetch_Mux_2{M1}"
 		(shape output)
@@
 		)
 	)
-	(global_label "1?"
-		(shape input)
-		(at 232.41 100.33 180)
-		(fields_autoplaced yes)
-		(effects
-			(font
-				(size 1.27 1.27)
-			)
-			(justify right)
-		)
-		(property "Intersheetrefs" "${INTERSHEET_REFS}"
-			(at 227.1267 100.33 0)
-			(effects
-				(font
-					(size 1.27 1.27)
-				)
-				(justify right)
-				(hide yes)
-			)
-		)
-	)
 	(global_label "1"
 		(shape input)
@@
 		)
 	)
-	(global_label "+PPU_RD_B{X3}"
+	(global_label "{slash}PPU_RD_B{X3}"
 		(shape input)
 		(at 116.84 163.83 180)
@@
 		)
 		(property "Intersheetrefs" "${INTERSHEET_REFS}"
-			(at 98.5543 163.83 0)
+			(at 98.7962 163.83 0)
 			(effects
 				(font
@@
 				(hide yes)
 			)
+		)
+	)
+	(global_label "1"
+		(shape input)
+		(at 232.41 100.33 180)
+		(fields_autoplaced yes)
+		(effects
+			(font
+				(size 1.27 1.27)
+			)
+			(justify right)
+		)
+		(property "Intersheetrefs" "${INTERSHEET_REFS}"
+			(at 228.2153 100.33 0)
+			(effects
+				(font
+					(size 1.27 1.27)
+				)
+				(justify right)
+				(hide yes)
+			)
+		)
+	)
+	(global_label "1"
+		(shape input)
+		(at 232.41 106.68 180)
+		(fields_autoplaced yes)
+		(effects
+			(font
+				(size 1.27 1.27)
+			)
+			(justify right)
+		)
+		(property "Intersheetrefs" "${INTERSHEET_REFS}"
+			(at 228.2153 106.68 0)
+			(effects
+				(font
+					(size 1.27 1.27)
+				)
+				(justify right)
+				(hide yes)
+			)

Commit message: - Updated all of the various And-OR-Invert gates to have consistent names.  - Added the schematic for CL3 / SL3 GPIO pins.  There are no surprises revealed by this.  - Finished up the CPU address decoding tracing.  - Added one of the 'artifact' counters from the pulse channels
Connections:
- net at P1. (X): now also P2. (X); no longer S5. (X)
- net at S7. (X): now also R9. (X); no longer S8. (/Q)
- net at S19. (X): now also R12. (X); no longer S20. (/Q)
- net at S11. (X): now also R10. (X); no longer S12. (/Q)
- net at S14. (X): now also R11. (X); no longer S15. (/Q)
- new net: S10. (X), S12. (/Q), S8. (/Q)
- new net: R5. (/Q), S16. (X)
- new net: P2. (X), R5. (/Q)
- new net: S22. (X), S23. (/Q), S26. (/Q), S27. (/Q), S28. (/Q)
- new net: P1. (X), S5. (X)
- new net: S7. (X), S8. (/Q)
- new net: S19. (X), S20. (/Q)
- new net: S11. (X), S12. (/Q)
- new net: S14. (X), S15. (/Q)
- new net: S20. (/Q), S21. (X), S23. (/Q)
- new net: X1. (X), X2. (X)
