File: Schematic (KiCAD)/scanline_detection.kicad_sch (KiCad schematic)
At the start: 102 parts, among them M2 NAND_2, M3 BIGBUF, P3 INVERT, P4 INVERT, T5 BUFFER, X12 D-FF Reset, X13 NAND_2, X14 BUFFER, X16 INVERT, X17 NAND_2, X26 INVERT, X27 D-FF No Reset, X28 INVERT, X4 NAND_2, X5 D-FF No Reset, X6 NAND_4, X7 INVERT, X8 Reg 2 DFF-No-Reset N, X9 NAND_2, Y1 BUFFER, Y10 XNOR_2, Y13 XNOR_2, Y15 NOR_2, Y17 XNOR_2, Y2,7,9,14,16,21,23,28 Reg 8 D-Latch, Y20 XNOR_2, Y22 NAND_4, Y24 XNOR_2, Y27 XNOR_2, Y29 NOR_2, Y3 XNOR_2, Y30 INVERT, Y31 D-FF Reset, Y32 INVERT, Y6 XNOR_2, Y8 NAND_4

Commit message: Tracing and schematic updates.  - Added timer to schematic.  - Added all items from artifacts sheet to the MMC5A trace.
Connections:
- net +PPU_RD_B{AB4} is gone; now on net /PPU_RD_B{AB4}: AB10. (/Q), AB13. (/Q), AB16. (/Q), AB19. (/Q), AB22. (/Q), AB6. (/Q), AB7. (/Q)
- net +PPU_RD_B{AC1} is gone; now on net /PPU_RD_B{AC1}: AC2. (Q1)
- net +PPU_RD_B{AC7} is gone; now on net /PPU_RD_B{AC7}: AC12. (/Q), AC15. (/Q), AC18. (/Q), AC21. (/Q), AC24. (/Q), AC27. (/Q), AC9. (/Q)
- net /PPU_RD_B{W1} is gone; now on net +PPU_RD_B{W1}: AB2(a). (X), AB2. (Q2)
- net at X7. (X): now also Z23. (/Q); no longer X6. (X)
- net at X13. (X): now also X12. (/Q); no longer X14. (X)
- net at X9. (X): now also Z24. (X); no longer X8. (/Q1)
- net /PPU_RD_B{AB4}: now reaches AB6. (/Q)
- net /PPU_RD_B{AB4}: no longer AA9. (X)
- net at AA10. (X): now also AA13. (X); no longer AA9. (X)
- net at AA16. (X): now also AA14. (X); no longer AA17. (X)
- net at Z2-Z18. (/Q7): now also Y3. (X); no longer Z19. (X)
- net at R7. (X): now also R8. (X); no longer R6. (X)
- net at Y29. (X): now also Y31. (/Q); no longer Y30. (X)
- net at Y15. (X): now also Y22. (X); no longer Y29. (X)
- net at Y17. (X): now also Y22. (X); no longer Y2,7,9,14,16,21,23,28. (Q7)
- net at Y24. (X): now also Y22. (X); no longer Y2,7,9,14,16,21,23,28. (Q7)
- net at Y20. (X): now also Y22. (X); no longer Y2,7,9,14,16,21,23,28. (Q7)
- net at Y6. (X): now also Y8. (X); no longer Y2,7,9,14,16,21,23,28. (Q7)
- net at Y13. (X): now also Y8. (X); no longer Y2,7,9,14,16,21,23,28. (Q7)
- net at Y10. (X): now also Y8. (X); no longer Y2,7,9,14,16,21,23,28. (Q7)
- net at Y3. (X): now also Y8. (X); no longer Y2,7,9,14,16,21,23,28. (Q7)
- net at Y27. (X): now also Y22. (X); no longer Y2,7,9,14,16,21,23,28. (Q7)
- net at AA20. (X): now also AA16. (X); no longer AA21. (X)
- net /PPU_RD_B{AC7}: now reaches AC15. (/Q)
- net at X17. (X): now also Z20. (X); no longer M2. (X)
- net at N39. (X): now also N38. (X); no longer M2. (X)
- net /PPU_RD_B{AC1}: now reaches AC2. (Q1)
- net /PPU_RD_B{AC1}: no longer AC6. (X)
- net at AA19. (X): now also AB18. (X); no longer AA22. (X)
- net at AA15. (X): now also AB17. (X); no longer AA11. (X)
- net at X26. (X): now also Y31. (/Q); no longer X17. (X)
- net at Y8. (X): now also Y15. (X); no longer Y6. (X)
- net at AA5. (X): now also AA15. (X); no longer AA10. (X)
- net +PPU_RD_B{W1}: now reaches AB2. (Q2)
- net +PPU_RD_B{W1}: no longer AA5. (X)
- net at AA2. (X): now also AB1. (X); no longer AA3. (X)
- net at AB1. (X): now also AB2(a). (X); no longer AA2. (X)
- new net: X4. (X), X5. (/Q)
- new net: X16. (X), X4. (X)
- new net: X5. (/Q), X6. (X)
- new net: X6. (X), X7. (X)
- new net: X13. (X), X14. (X)
- new net: X13. (X), Y31. (/Q), Y32. (X)
- new net: P4. (X), R1. (X)
- new net: AA1. (X), AA2. (X), R1. (X) (x2)
- new net: P3. (X), R1. (X)
- new net: X8. (/Q1), X9. (X) (x2)
- new net: AA9. (X), AB6. (/Q)
- new net: AA10. (X), AA9. (X)
- new net: AA17. (X), AB16. (/Q)
- new net: AA16. (X), AA17. (X)
- new net: Z19. (X), Z2-Z18. (/Q7)
- new net: R6. (X), R7. (X)
- new net: Y29. (X), Y30. (X)
- new net: Y15. (X), Y29. (X)
- new net: Y1. (X), Y2,7,9,14,16,21,23,28. (Q7)
- new net: Y17. (X), Y2,7,9,14,16,21,23,28. (Q7)
- new net: Y2,7,9,14,16,21,23,28. (Q7), Y24. (X)
- new net: Y2,7,9,14,16,21,23,28. (Q7), Y20. (X)
- new net: Y2,7,9,14,16,21,23,28. (Q7), Y6. (X)
- new net: Y13. (X), Y2,7,9,14,16,21,23,28. (Q7)
- new net: Y10. (X), Y2,7,9,14,16,21,23,28. (Q7)
- new net: Y2,7,9,14,16,21,23,28. (Q7), Y3. (X)
- new net: Y2,7,9,14,16,21,23,28. (Q7), Y27. (X)
- new net: AA20. (X), AA21. (X)
- new net: AA21. (X), AB22. (/Q)
- new net: AA7. (X), AB10. (/Q), AB13. (/Q), AB16. (/Q), AB19. (/Q), AB22. (/Q), AB6. (/Q), AB7. (/Q)
- new net: AB3. (X), AC12. (/Q), AC15. (/Q), AC18. (/Q), AC21. (/Q), AC24. (/Q), AC27. (/Q), AC9. (/Q)
- new net: AB11. (X), AC15. (/Q)
- new net: AA12. (X), AB7. (/Q)
- new net: M2. (X), X17. (X)
- new net: M2. (X), N39. (X)
- new net: Y17. (X), Z2-Z18. (/Q7), Z22. (X)
- new net: Y24. (X), Z2-Z18. (/Q7), Z22. (X)
- new net: Y20. (X), Z2-Z18. (/Q7), Z22. (X)
- new net: Y27. (X), Z2-Z18. (/Q7), Z22. (X)
- new net: Y6. (X), Z2-Z18. (/Q7)
- new net: Y13. (X), Z2-Z18. (/Q7)
- new net: Y10. (X), Z2-Z18. (/Q7)
- new net: Z1. (X), Z2-Z18. (/Q7)
- new net: AA10. (X), AA12. (X)
- new net: AA22. (X), AC27. (/Q)
- new net: AA11. (X), AC12. (/Q)
- new net: AC2. (Q1), AC6. (X) (x2)
- new net: AA19. (X), AA22. (X)
- new net: AA11. (X), AA15. (X)
- new net: AA18. (X), AB19. (/Q)
- new net: AA16. (X), AA18. (X)
- new net: X17. (X), X26. (X)
- new net: AA10. (X), AA5. (X)
- new net: AA5. (X), AB2. (Q2)
- new net: AA19. (X), AA5. (X)
- new net: AA16. (X), AA5. (X)
- new net: AA10. (X), AA8. (X)
- new net: AA2. (X), AA3. (X)
- new net: AA2. (X), AA4. (X)
- new net: Z24. (X), Z25. (X)
- new net: AA8. (X), AC9. (/Q)
- new net: M3. (X), N38. (X)
- new net: AB1. (X), AB2. (Q2) (x3)
- new net: AA13. (X), AB10. (/Q)
- new net: AB17. (X), AC21. (/Q)
- new net: N16. (X), N9. (X)
- new net: AA15. (X), AB12. (X)
- new net: AB12. (X), AC18. (/Q)
- new net: X27. (/Q), X28. (X)
- new net: AB18. (X), AC24. (/Q)
- new net: AA14. (X), AB13. (/Q)
- new net: AA15. (X), AB11. (X)
Other:
- note added: "This signal likely needs to be active hi."
- note added: "This signal likely needs to be active low."
Changed lines of the file:
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@@
 		)
 	)
+	(text "This signal likely needs\nto be active hi."
+		(exclude_from_sim no)
+		(at 351.536 117.094 0)
+		(effects
+			(font
+				(size 1.27 1.27)
+			)
+		)
+	)
 	(text "External Scanline End"
 		(exclude_from_sim no)
@@
 		)
 	)
+	(text "This signal likely needs\nto be active low."
+		(exclude_from_sim no)
+		(at 339.344 91.694 0)
+		(effects
+			(font
+				(size 1.27 1.27)
+			)
+		)
+	)
 	(text "/IRQ"
 		(exclude_from_sim no)
@@
 		)
 	)
-	(global_label "+PPU_RD_B{AC7}"
+	(global_label "{slash}PPU_RD_B{AC7}"
 		(shape input)
 		(at 54.61 138.43 180)
@@
 		)
 		(property "Intersheetrefs" "${INTERSHEET_REFS}"
-			(at 35.1752 138.43 0)
+			(at 35.4171 138.43 0)
 			(effects
 				(font
@@
 		)
 	)
-	(global_label "+PPU_RD_B{AC1}"
+	(global_label "{slash}PPU_RD_B{AC1}"
 		(shape input)
 		(at 162.56 76.2 180)
@@
 		)
 		(property "Intersheetrefs" "${INTERSHEET_REFS}"
-			(at 143.1252 76.2 0)
+			(at 143.3671 76.2 0)
 			(effects
 				(font
@@
 		)
 	)
-	(global_label "{slash}PPU_RD_B{W1}"
+	(global_label "+PPU_RD_B{W1}"
 		(shape input)
 		(at 161.29 54.61 180)
@@
 		)
 		(property "Intersheetrefs" "${INTERSHEET_REFS}"
-			(at 143.0043 54.61 0)
+			(at 142.7624 54.61 0)
 			(effects
 				(font
@@
 		)
 	)
-	(global_label "+PPU_RD_B{AB4}"
+	(global_label "{slash}PPU_RD_B{AB4}"
 		(shape input)
 		(at 54.61 115.57 180)
@@
 		)
 		(property "Intersheetrefs" "${INTERSHEET_REFS}"
-			(at 35.1752 115.57 0)
+			(at 35.4171 115.57 0)
 			(effects
 				(font

Commit message: - Updated all of the various And-OR-Invert gates to have consistent names.  - Added the schematic for CL3 / SL3 GPIO pins.  There are no surprises revealed by this.  - Finished up the CPU address decoding tracing.  - Added one of the 'artifact' counters from the pulse channels
Parts:
- AA2, R1: value AOI_2 -> AOI_22
Connections:
- net at X7. (X): now also Z23. (/Q); no longer X6. (X)
- net at X13. (X): now also X12. (/Q); no longer X14. (X)
- net at X9. (X): now also Z24. (X); no longer X8. (/Q1)
- net at AA10. (X): now also AA13. (X); no longer AA9. (X)
- net at AA16. (X): now also AA14. (X); no longer AA17. (X)
- net at Z2-Z18. (/Q7): now also Y3. (X); no longer Z19. (X)
- net at R7. (X): now also R8. (X); no longer R6. (X)
- net at Y29. (X): now also Y31. (/Q); no longer Y30. (X)
- net at Y15. (X): now also Y22. (X); no longer Y29. (X)
- net at Y17. (X): now also Y22. (X); no longer Y2,7,9,14,16,21,23,28. (Q7)
- net at Y24. (X): now also Y22. (X); no longer Y2,7,9,14,16,21,23,28. (Q7)
- net at Y20. (X): now also Y22. (X); no longer Y2,7,9,14,16,21,23,28. (Q7)
- net at Y6. (X): now also Y8. (X); no longer Y2,7,9,14,16,21,23,28. (Q7)
- net at Y13. (X): now also Y8. (X); no longer Y2,7,9,14,16,21,23,28. (Q7)
- net at Y10. (X): now also Y8. (X); no longer Y2,7,9,14,16,21,23,28. (Q7)
- net at Y3. (X): now also Y8. (X); no longer Y2,7,9,14,16,21,23,28. (Q7)
- net at Y27. (X): now also Y22. (X); no longer Y2,7,9,14,16,21,23,28. (Q7)
- net at AA20. (X): now also AA16. (X); no longer AA21. (X)
- net at X17. (X): now also Z20. (X); no longer M2. (X)
- net at N39. (X): now also N38. (X); no longer M2. (X)
- net at AA19. (X): now also AB18. (X); no longer AA22. (X)
- net at AA15. (X): now also AB17. (X); no longer AA11. (X)
- net at X26. (X): now also Y31. (/Q); no longer X17. (X)
- net at Y8. (X): now also Y15. (X); no longer Y6. (X)
- net at AA5. (X): now also AA15. (X); no longer AA10. (X)
- net at AA2. (X): now also AB1. (X); no longer AA3. (X)
- net at AB1. (X): now also AB2(a). (X); no longer AA2. (X)
- new net: X4. (X), X5. (/Q)
- new net: X16. (X), X4. (X)
- new net: X5. (/Q), X6. (X)
- new net: X6. (X), X7. (X)
- new net: X13. (X), X14. (X)
- new net: X13. (X), Y31. (/Q), Y32. (X)
- new net: P4. (X), R1. (X)
- new net: AA1. (X), AA2. (X), R1. (X) (x2)
- new net: P3. (X), R1. (X)
- new net: X8. (/Q1), X9. (X) (x2)
- new net: AA9. (X), AB6. (/Q)
- new net: AA10. (X), AA9. (X)
- new net: AA17. (X), AB16. (/Q)
- new net: AA16. (X), AA17. (X)
- new net: Z19. (X), Z2-Z18. (/Q7)
- new net: R6. (X), R7. (X)
- new net: Y29. (X), Y30. (X)
- new net: Y15. (X), Y29. (X)
- new net: Y1. (X), Y2,7,9,14,16,21,23,28. (Q7)
- new net: Y17. (X), Y2,7,9,14,16,21,23,28. (Q7)
- new net: Y2,7,9,14,16,21,23,28. (Q7), Y24. (X)
- new net: Y2,7,9,14,16,21,23,28. (Q7), Y20. (X)
- new net: Y2,7,9,14,16,21,23,28. (Q7), Y6. (X)
- new net: Y13. (X), Y2,7,9,14,16,21,23,28. (Q7)
- new net: Y10. (X), Y2,7,9,14,16,21,23,28. (Q7)
- new net: Y2,7,9,14,16,21,23,28. (Q7), Y3. (X)
- new net: Y2,7,9,14,16,21,23,28. (Q7), Y27. (X)
- new net: AA20. (X), AA21. (X)
- new net: AA21. (X), AB22. (/Q)
- new net: AA7. (X), AB10. (/Q), AB13. (/Q), AB16. (/Q), AB19. (/Q), AB22. (/Q), AB6. (/Q), AB7. (/Q)
- new net: AB3. (X), AC12. (/Q), AC15. (/Q), AC18. (/Q), AC21. (/Q), AC24. (/Q), AC27. (/Q), AC9. (/Q)
- new net: AB11. (X), AC15. (/Q)
- new net: AA12. (X), AB7. (/Q)
- new net: M2. (X), X17. (X)
- new net: M2. (X), N39. (X)
- new net: Y17. (X), Z2-Z18. (/Q7), Z22. (X)
- new net: Y24. (X), Z2-Z18. (/Q7), Z22. (X)
- new net: Y20. (X), Z2-Z18. (/Q7), Z22. (X)
- new net: Y27. (X), Z2-Z18. (/Q7), Z22. (X)
- new net: Y6. (X), Z2-Z18. (/Q7)
- new net: Y13. (X), Z2-Z18. (/Q7)
- new net: Y10. (X), Z2-Z18. (/Q7)
- new net: Z1. (X), Z2-Z18. (/Q7)
- new net: AA10. (X), AA12. (X)
- new net: AA22. (X), AC27. (/Q)
- new net: AA11. (X), AC12. (/Q)
- new net: AC2. (Q1), AC6. (X) (x2)
- new net: AA19. (X), AA22. (X)
- new net: AA11. (X), AA15. (X)
- new net: AA18. (X), AB19. (/Q)
- new net: AA16. (X), AA18. (X)
- new net: X17. (X), X26. (X)
- new net: AA10. (X), AA5. (X)
- new net: AA5. (X), AB2. (Q2)
- new net: AA19. (X), AA5. (X)
- new net: AA16. (X), AA5. (X)
- new net: AA10. (X), AA8. (X)
- new net: AA2. (X), AA3. (X)
- new net: AA2. (X), AA4. (X)
- new net: Z24. (X), Z25. (X)
- new net: AA8. (X), AC9. (/Q)
- new net: M3. (X), N38. (X)
- new net: AB1. (X), AB2. (Q2) (x3)
- new net: AA13. (X), AB10. (/Q)
- new net: AB17. (X), AC21. (/Q)
- new net: N16. (X), N9. (X)
- new net: AA15. (X), AB12. (X)
- new net: AB12. (X), AC18. (/Q)
- new net: X27. (/Q), X28. (X)
- new net: AB18. (X), AC24. (/Q)
- new net: AA14. (X), AB13. (/Q)
- new net: AA15. (X), AB11. (X)
